File: hardware/ETH1CFGEN1/ETH1CFGEN1.kicad_sch (KiCad schematic)
At the start: 0 parts

Commit message: Development
Other:
- added sheet Power (Power.kicad_sch)
- added sheet Waveform DAC (WaveformDAC.kicad_sch)
Changed lines of the file:
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@@
+    )
+  )
+  (sheet (at 134.62 121.285) (size 33.655 26.67) (fields_autoplaced)
+    (stroke (width 0.1524) (type solid))
+    (fill (color 0 0 0 0.0000))
+    (property "Sheetname" "Power" (at 134.62 120.5734 0)
+      (effects (font (size 1.27 1.27)) (justify left bottom))
+    )
+    (property "Sheetfile" "Power.kicad_sch" (at 134.62 148.5396 0)
+      (effects (font (size 1.27 1.27)) (justify left top))
+    )
+    (instances
+      (project "ETH1CFGEN1"
+        (path "/44bc1157-6d68-4ab3-afc0-b8d9f089cc50" (page "7"))
+      )
+    )
+  )
+  (sheet (at 70.485 33.02) (size 59.055 26.035) (fields_autoplaced)
+    (stroke (width 0.1524) (type solid))
+    (fill (color 0 0 0 0.0000))
+    (property "Sheetname" "Waveform DAC" (at 70.485 32.3084 0)
+      (effects (font (size 1.27 1.27)) (justify left bottom))
+    )
+    (property "Sheetfile" "WaveformDAC.kicad_sch" (at 70.485 59.6396 0)
+      (effects (font (size 1.27 1.27)) (justify left top))
+    )
+    (instances
+      (project "ETH1CFGEN1"
+        (path "/44bc1157-6d68-4ab3-afc0-b8d9f089cc50" (page "6"))
+      )
     )
   )

Commit message: Development
Other:
- sheet Waveform DAC ports: added SET_ARB_FLTR1, SET_ARB_FLTR2, SET_SIN_FLTR1, SET_SIN_FLTR2, SINE_ARB, SQUARE, SQ_COMP_EN, V_AMPL, V_DTY_CYCL, V_NULL_SINE, WFDAC[0..13], WFD_FPGA_50MHZ; removed none
Changed lines of the file:
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@@
     )
   )
-  (sheet (at 70.485 33.02) (size 59.055 26.035) (fields_autoplaced)
+  (sheet (at 79.375 31.75) (size 50.165 26.67) (fields_autoplaced)
     (stroke (width 0.1524) (type solid))
     (fill (color 0 0 0 0.0000))
-    (property "Sheetname" "Waveform DAC" (at 70.485 32.3084 0)
+    (property "Sheetname" "Waveform DAC" (at 79.375 31.0384 0)
       (effects (font (size 1.27 1.27)) (justify left bottom))
     )
-    (property "Sheetfile" "WaveformDAC.kicad_sch" (at 70.485 59.6396 0)
+    (property "Sheetfile" "WaveformDAC.kicad_sch" (at 79.375 59.0046 0)
       (effects (font (size 1.27 1.27)) (justify left top))
     )
+    (pin "SET_SIN_FLTR2" input (at 79.375 48.26 180)
+      (effects (font (size 1.27 1.27)) (justify left))
+    )
+    (pin "V_NULL_SINE" input (at 79.375 37.465 180)
+      (effects (font (size 1.27 1.27)) (justify left))
+    )
+    (pin "SET_ARB_FLTR2" input (at 79.375 50.165 180)
+      (effects (font (size 1.27 1.27)) (justify left))
+    )
+    (pin "SQUARE" output (at 79.375 40.64 180)
+      (effects (font (size 1.27 1.27)) (justify left))
+    )
+    (pin "SINE_ARB" output (at 129.54 36.83 0)
+      (effects (font (size 1.27 1.27)) (justify right))
+    )
+    (pin "WFDAC[0..13]" bidirectional (at 79.375 44.45 180)
+      (effects (font (size 1.27 1.27)) (justify left))
+    )
+    (pin "SET_SIN_FLTR1" input (at 79.375 52.07 180)
+      (effects (font (size 1.27 1.27)) (justify left))
+    )
+    (pin "SET_ARB_FLTR1" input (at 79.375 53.975 180)
+      (effects (font (size 1.27 1.27)) (justify left))
+    )
+    (pin "V_DTY_CYCL" input (at 79.375 46.355 180)
+      (effects (font (size 1.27 1.27)) (justify left))
+    )
+    (pin "SQ_COMP_EN" input (at 79.375 42.545 180)
+      (effects (font (size 1.27 1.27)) (justify left))
+    )
+    (pin "WFD_FPGA_50MHZ" output (at 79.375 34.925 180)
+      (effects (font (size 1.27 1.27)) (justify left))
+    )
+    (pin "V_AMPL" input (at 129.54 41.275 0)
+      (effects (font (size 1.27 1.27)) (justify right))
+    )
     (instances
