File: hardware/ETH1CFGEN1/FPGA.kicad_sch (KiCad schematic)
At the start: 0 parts

Commit message: Development
Parts:
- added C501, C502, C503, C504, C505, C507, C508, C509, C510, C511, C512, C514, C515, C516, C517, C518, C519, C520, C521, C522, C523, C524, C525, C526, C527, C528, C529: 0.1u, symbol Device:C
- added C506, C513: 10u, symbol Device:C
- added D501: BLUE, symbol Device:LED
- added J501: Conn_01x06, symbol Connector_Generic:Conn_01x06
- added J502: Conn_02x07_Odd_Even, symbol Connector_Generic:Conn_02x07_Odd_Even
- added R501, R502, R509: 10k, symbol Device:R
- added R503: 2k2, symbol Device:R
- added R504, R508: 4k7, symbol Device:R
- added R505: 1k, symbol Device:R
- added R506: 27, symbol Device:R
- added R507: 1K, symbol Device:R
- added U503: XC6SLX9-TQG144, symbol FPGA_Xilinx_Spartan6:XC6SLX9-TQG144
- added U504: W25Q64JV, Package_SO:SOIC-8_5.23x5.23mm_P1.27mm, symbol Memory_Flash:W25Q32JVSS
- added U?: TLV1117LV33DCYR, symbol Regulator_Linear:TLV1117-15
- added U?: TLV1117LV12DCYR, symbol Regulator_Linear:TLV1117-15
- added X501: ASFL1-100.000MHZ-L-T, symbol Oscillator:SG-5032CBN
Connections:
- new net: D501.1 (K), R507.2
- new net: R505.2, X501.1 (~{ST})
- new net: R506.1, X501.3 (OUT)
- new net +5VD: C503.1, U?.3 (VI)
- new net CMPCS_B_2: R509.1, U503.72 (CMPCS_B_2)
- new net DONE_2: R507.1, U503.71 (DONE_2)
- new net FLASH_HOLD: R501.2, U504.7 (IO3)
- new net FLASH_INIT_B: R504.2, U503.39 (IO_L65P_INIT_B_2)
- new net FLASH_SCK: U503.70 (IO_L1P_CCLK_2), U504.6 (CLK)
- new net FLASH_SI: U504.5 (DI(IO0))
- new net FLASH_SO: U504.2 (DO(IO1))
- new net FLASH_WP: R502.2, U504.3 (IO2)
- new net FLASH_nCS: R503.2, U503.38 (IO_L65N_CSO_B_2), U504.1 (~{CS})
- new net FPGA_1V2: C513.1, C515.1, C523.1, C524.1, C525.1, C526.1, C527.1, U503.128 (VCCINT), U503.19 (VCCINT), U503.28 (VCCINT), U503.52 (VCCINT), U503.89 (VCCINT), U?.2 (VO)
- new net FPGA_3V3: C501.1, C502.1, C504.1, C505.1, C506.1, C507.1, C508.1, C509.1, C510.1, C511.1, C512.1, C514.1, C516.1, C517.1, C518.1, C519.1, C520.1, C521.1, C522.1, C528.1, C529.1, D501.2 (A), J501.1 (Pin_1), J502.2 (Pin_2), R501.1, R502.1, R503.1, R504.1, R505.1, R508.2, R509.2, U503.103 (VCCO_1), U503.122 (VCCO_0), U503.125 (VCCO_0), U503.129 (VCCAUX), U503.135 (VCCO_0), U503.18 (VCCO_3), U503.20 (VCCAUX), U503.31 (VCCO_3), U503.36 (VCCAUX), U503.4 (VCCO_3), U503.42 (VCCO_2), U503.53 (VCCAUX), U503.63 (VCCO_2), U503.69 (IO_L1N_M0_CMPMISO_2), U503.76 (VCCO_1), U503.86 (VCCO_1), U503.90 (VCCAUX), U504.8 (VCC), U?.2 (VO), U?.3 (VI), X501.4 (VCC)
- new net FPGA_CLK_100MHZ: R506.2
- new net FPGA_TCK: J501.3 (Pin_3), J502.6 (Pin_6), U503.109 (TCK)
- new net FPGA_TDI: J501.5 (Pin_5), J502.10 (Pin_10), U503.110 (TDI)
- new net FPGA_TDO: J501.4 (Pin_4), J502.8 (Pin_8), U503.106 (TDO)
- new net FPGA_TMS: J501.2 (Pin_2), J502.4 (Pin_4), U503.107 (TMS)
- new net GNDD: C501.2, C502.2, C503.2, C504.2, C505.2, C506.2, C507.2, C508.2, C509.2, C510.2, C511.2, C512.2, C513.2, C514.2, C515.2, C516.2, C517.2, C518.2, C519.2, C520.2, C521.2, C522.2, C523.2, C524.2, C525.2, C526.2, C527.2, C528.2, C529.2, J501.6 (Pin_6), J502.11 (Pin_11), J502.13 (Pin_13), J502.3 (Pin_3), J502.5 (Pin_5), J502.7 (Pin_7), J502.9 (Pin_9), U503.108 (GND), U503.113 (GND), U503.13 (GND), U503.130 (GND), U503.136 (GND), U503.25 (GND), U503.3 (GND), U503.49 (GND), U503.54 (GND), U503.60 (IO_L13P_M1_2), U503.68 (GND), U503.73 (SUSPEND), U503.77 (GND), U503.91 (GND), U503.96 (GND), U504.4 (GND), U?.1 (GND), U?.1 (GND), X501.2 (GND)
- new net PROG_B_2: R508.1, U503.37 (PROGRAM_B_2)
- no-connect marks 0 -> 3

Commit message: Development
Changed lines of the file:
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@@
   )
   (symbol (lib_id "ETH1CFGEN1:FGPA_3V3") (at 196.85 200.025 0) (unit 1)
-    (in_bom yes) (on_board yes) (dnp no) (fields_autoplaced)
+    (in_bom yes) (on_board yes) (dnp no)
     (property "Reference" "#PWR0514" (at 196.85 203.835 0)
       (effects (font (size 1.27 1.27)) hide)
     )
-    (property "Value" "FPGA_3V3" (at 196.85 194.945 0)
+    (property "Value" "FPGA_3V3" (at 196.85 195.58 0)
       (effects (font (size 1.27 1.27)))
     )
