File: hardware/ETH1CFGEN1/FPGA.kicad_sch (KiCad schematic)
At the start: 46 parts, among them J201 Conn_01x06, J202 Conn_02x07_Odd_Even, U201 TLV1117LV33DCYR, U202 TLV1117LV12DCYR, U203 XC6SLX9-3TQG144I, U204 W25Q64JV, X201 ASFL1-100.000MHZ-L-T

Commit message: Development
Parts:
- removed J201: Conn_01x06, Connector_PinHeader_2.54mm:PinHeader_1x06_P2.54mm_Vertical, symbol Connector_Generic:Conn_01x06
Changed lines of the file:
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@@
 (kicad_sch (version 20230121) (generator eeschema)
   (paper "A3")
+  (title_block
+    (date "2023-07-12")
+    (rev "1.1")
+  )
   (junction (at 156.21 156.21) (diameter 0) (color 0 0 0 0)
   )
@@
     (stroke (width 0) (type default))
   )
-  (wire (pts (xy 335.28 239.395) (xy 335.28 240.665))
-    (stroke (width 0) (type default))
-  )
   (wire (pts (xy 359.41 236.855) (xy 360.045 236.855))
     (stroke (width 0) (type default))
@@
     (stroke (width 0) (type default))
   )
-  (wire (pts (xy 334.01 231.775) (xy 346.075 231.775))
-    (stroke (width 0) (type default))
-  )
   (wire (pts (xy 236.855 276.225) (xy 236.855 276.86))
     (stroke (width 0) (type default))
@@
     (stroke (width 0) (type default))
   )
-  (wire (pts (xy 334.01 234.315) (xy 346.075 234.315))
-    (stroke (width 0) (type default))
-  )
   (wire (pts (xy 118.745 238.76) (xy 118.745 240.03))
     (stroke (width 0) (type default))
   )
-  (wire (pts (xy 334.01 229.235) (xy 346.075 229.235))
-    (stroke (width 0) (type default))
-  )
   (wire (pts (xy 104.14 140.97) (xy 104.14 138.43))
     (stroke (width 0) (type default))
@@
     (stroke (width 0) (type default))
   )
-  (wire (pts (xy 334.01 236.855) (xy 346.075 236.855))
-    (stroke (width 0) (type default))
-  )
   (wire (pts (xy 252.73 29.21) (xy 252.73 28.575))
     (stroke (width 0) (type default))
@@
     (stroke (width 0) (type default))
   )
-  (wire (pts (xy 335.28 226.695) (xy 335.28 224.79))
-    (stroke (width 0) (type default))
-  )
   (wire (pts (xy 106.045 229.87) (xy 118.745 229.87))
     (stroke (width 0) (type default))
@@
     (stroke (width 0) (type default))
   )
-  (wire (pts (xy 334.01 226.695) (xy 335.28 226.695))
-    (stroke (width 0) (type default))
-  )
   (wire (pts (xy 359.41 239.395) (xy 359.41 240.665))
     (stroke (width 0) (type default))
@@
     (stroke (width 0) (type default))
   )
-  (wire (pts (xy 334.01 239.395) (xy 335.28 239.395))
-    (stroke (width 0) (type default))
-  )
   (wire (pts (xy 156.21 158.75) (xy 155.575 158.75))
     (stroke (width 0) (type default))
@@
     (effects (font (size 1.27 1.27)) (justify left bottom))
   )
-  (label "FPGA_TDO" (at 346.075 234.315 180) (fields_autoplaced)
-    (effects (font (size 1.27 1.27)) (justify right bottom))
-  )
   (label "FLASH_SCK" (at 230.505 49.53 0) (fields_autoplaced)
     (effects (font (size 1.27 1.27)) (justify left bottom))
@@
     (effects (font (size 1.27 1.27)) (justify right bottom))
   )
-  (label "FPGA_TDI" (at 346.075 236.855 180) (fields_autoplaced)
-    (effects (font (size 1.27 1.27)) (justify right bottom))
-  )
   (label "FLASH_INIT_B" (at 230.505 110.49 0) (fields_autoplaced)
     (effects (font (size 1.27 1.27)) (justify left bottom))
@@
     (effects (font (size 1.27 1.27)) (justify right bottom))
   )
-  (label "FPGA_TMS" (at 346.075 229.235 180) (fields_autoplaced)
-    (effects (font (size 1.27 1.27)) (justify right bottom))
-  )
   (label "FLASH_nCS" (at 230.505 113.03 0) (fields_autoplaced)
     (effects (font (size 1.27 1.27)) (justify left bottom))
@@
     (effects (font (size 1.27 1.27)) (justify left bottom))
   )
-  (label "FPGA_TCK" (at 346.075 231.775 180) (fields_autoplaced)
-    (effects (font (size 1.27 1.27)) (justify right bottom))
-  )
   (label "CMPCS_B_2" (at 342.9 164.465 180) (fields_autoplaced)
     (effects (font (size 1.27 1.27)) (justify right bottom))
@@
       (project "ETH1CFGEN1"
         (path "/44bc1157-6d68-4ab3-afc0-b8d9f089cc50/341f5c61-297e-4a23-a6a5-42e392eadbed"
-          (reference "#PWR0736") (unit 1)
+          (reference "#PWR0734") (unit 1)
         )
       )
@@
       (project "ETH1CFGEN1"
         (path "/44bc1157-6d68-4ab3-afc0-b8d9f089cc50/341f5c61-297e-4a23-a6a5-42e392eadbed"
-          (reference "#PWR0735") (unit 1)
+          (reference "#PWR0733") (unit 1)
         )
       )
@@
     )
   )
-  (symbol (lib_id "Connector_Generic:Conn_01x06") (at 328.93 231.775 0) (mirror y) (unit 1)
-    (in_bom yes) (on_board yes) (dnp no)
-    (property "Reference" "J201" (at 326.39 231.775 0)
-      (effects (font (size 1.27 1.27)) (justify left))
-    )
-    (property "Value" "Conn_01x06" (at 326.39 234.315 0)
-      (effects (font (size 1.27 1.27)) (justify left))
-    )
-    (property "Footprint" "Connector_PinHeader_2.54mm:PinHeader_1x06_P2.54mm_Vertical" (at 328.93 231.775 0)
-      (effects (font (size 1.27 1.27)) hide)
-    )
-    (property "Datasheet" "~" (at 328.93 231.775 0)
-      (effects (font (size 1.27 1.27)) hide)
-    )
-    (pin "1")
-    (pin "2")
-    (pin "3")
-    (pin "4")
-    (pin "5")
-    (pin "6")
-    (instances
-      (project "ETH1CFGEN1B"
-        (path "/3dceb0a1-97ad-435d-a235-e3839b959163/95cc2f98-d767-47b4-8dfd-bb0285571db4"
-          (reference "J201") (unit 1)
-        )
-      )
-      (project "ETH1CFGEN1"
-        (path "/44bc1157-6d68-4ab3-afc0-b8d9f089cc50/341f5c61-297e-4a23-a6a5-42e392eadbed"
-          (reference "J701") (unit 1)
-        )
-      )
-    )
-  )
   (symbol (lib_id "Device:C") (at 118.745 234.95 0) (unit 1)
     (in_bom yes) (on_board yes) (dnp no) (fields_autoplaced)
@@
       (project "ETH1CFGEN1"
         (path "/44bc1157-6d68-4ab3-afc0-b8d9f089cc50/341f5c61-297e-4a23-a6a5-42e392eadbed"
-          (reference "J702") (unit 1)
+          (reference "J701") (unit 1)
         )
       )
@@
       (project "ETH1CFGEN1"
         (path "/44bc1157-6d68-4ab3-afc0-b8d9f089cc50/341f5c61-297e-4a23-a6a5-42e392eadbed"
-          (reference "#PWR0734") (unit 1)
+          (reference "#PWR0732") (unit 1)
         )
       )
@@
     )
   )
-  (symbol (lib_id "power:GNDD") (at 335.28 240.665 0) (unit 1)
-    (in_bom yes) (on_board yes) (dnp no) (fields_autoplaced)
-    (property "Reference" "#PWR0233" (at 335.28 247.015 0)
-      (effects (font (size 1.27 1.27)) hide)
-    )
-    (property "Value" "GNDD" (at 335.28 244.475 0)
-      (effects (font (size 1.27 1.27)))
-    )
-    (property "Footprint" "" (at 335.28 240.665 0)
-      (effects (font (size 1.27 1.27)) hide)
-    )
-    (property "Datasheet" "" (at 335.28 240.665 0)
-      (effects (font (size 1.27 1.27)) hide)
-    )
-    (pin "1")
-    (instances
-      (project "ETH1CFGEN1B"
-        (path "/3dceb0a1-97ad-435d-a235-e3839b959163/95cc2f98-d767-47b4-8dfd-bb0285571db4"
-          (reference "#PWR0233") (unit 1)
-        )
-      )
-      (project "ETH1CFGEN1"
-        (path "/44bc1157-6d68-4ab3-afc0-b8d9f089cc50/341f5c61-297e-4a23-a6a5-42e392eadbed"
-          (reference "#PWR0733") (unit 1)
-        )
-      )
-    )
-  )
   (symbol (lib_id "Device:C") (at 27.94 272.415 0) (unit 1)
     (in_bom yes) (on_board yes) (dnp no)
@@
     )
   )
-  (symbol (lib_id "ETH1CFGEN1:FGPA_3V3") (at 335.28 224.79 0) (unit 1)
-    (in_bom yes) (on_board yes) (dnp no)
-    (property "Reference" "#PWR0232" (at 335.28 228.6 0)
-      (effects (font (size 1.27 1.27)) hide)
-    )
-    (property "Value" "FPGA_3V3" (at 335.28 220.98 0)
-      (effects (font (size 1.27 1.27)))
-    )
-    (property "Footprint" "" (at 335.28 224.79 0)
-      (effects (font (size 1.27 1.27)) hide)
-    )
-    (property "Datasheet" "" (at 335.28 224.79 0)
-      (effects (font (size 1.27 1.27)) hide)
-    )
-    (pin "1")
-    (instances
-      (project "ETH1CFGEN1B"
-        (path "/3dceb0a1-97ad-435d-a235-e3839b959163/95cc2f98-d767-47b4-8dfd-bb0285571db4"
-          (reference "#PWR0232") (unit 1)
-        )
-      )
-      (project "ETH1CFGEN1"
-        (path "/44bc1157-6d68-4ab3-afc0-b8d9f089cc50/341f5c61-297e-4a23-a6a5-42e392eadbed"
-          (reference "#PWR0732") (unit 1)
-        )
-      )
-    )
-  )
   (symbol (lib_id "power:GNDD") (at 359.41 240.665 0) (unit 1)
     (in_bom yes) (on_board yes) (dnp no) (fields_autoplaced)
@@
       (project "ETH1CFGEN1"
         (path "/44bc1157-6d68-4ab3-afc0-b8d9f089cc50/341f5c61-297e-4a23-a6a5-42e392eadbed"
-          (reference "#PWR0737") (unit 1)
+          (reference "#PWR0735") (unit 1)
         )
       )
@@
       (project "ETH1CFGEN1"
         (path "/44bc1157-6d68-4ab3-afc0-b8d9f089cc50/341f5c61-297e-4a23-a6a5-42e392eadbed"
-          (reference "#PWR0738") (unit 1)
+          (reference "#PWR0736") (unit 1)
         )
       )

Commit message: PCB design
Parts:
- removed J202: Conn_02x07_Odd_Even, symbol Connector_Generic:Conn_02x07_Odd_Even
- added J701: Conn_02x05_Odd_Even, Connector_PinHeader_2.54mm:PinHeader_2x05_P2.54mm_Vertical, symbol Connector_Generic:Conn_02x05_Odd_Even
- X201: footprint (none) -> Crystal:Crystal_SMD_5032-4Pin_5.0x3.2mm
Connections:
- net FPGA_3V3: now also J701.2 (Pin_2)
- net FPGA_TCK: now also J701.6 (Pin_6)
- net FPGA_TDI: now also J701.10 (Pin_10)
- net FPGA_TDO: now also J701.8 (Pin_8)
- net FPGA_TMS: now also J701.4 (Pin_4)
- net GNDD: now also J701.1 (Pin_1), J701.3 (Pin_3), J701.5 (Pin_5), J701.7 (Pin_7), J701.9 (Pin_9)
- no-connect marks 3 -> 0

Commit message: PCB design
Connections:
- net WFDAC6: now reaches U203.10 (IO_L50P_3)
- net WFDAC7: now reaches U203.11 (IO_L49N_3)
- net WFDAC8: now reaches U203.12 (IO_L49P_3)
- net WFDAC9: now reaches U203.14 (IO_L44N_GCLK20_3)
- net WFDAC10: now reaches U203.15 (IO_L44P_GCLK21_3)
- net WFDAC11: now reaches U203.16 (IO_L43N_GCLK22_IRDY2_3)
- net WFDAC12: now reaches U203.17 (IO_L43P_GCLK23_3)
- net WFDAC0: now reaches U203.2 (IO_L83P_3)
- net WFDAC13: now reaches U203.21 (IO_L42N_GCLK24_3)
- net WFDAC1: now reaches U203.5 (IO_L52N_3)
- net WFDAC2: now reaches U203.6 (IO_L52P_3)
- net WFDAC3: now reaches U203.7 (IO_L51N_3)
- net WFDAC4: now reaches U203.8 (IO_L51P_3)
- net WFDAC5: now reaches U203.9 (IO_L50N_3)
- no-connect marks 0 -> 1

Commit message: PCB design
Connections:
- net FPGA_CLK_100MHZ: now also U203.134 (IO_L34P_GCLK19_0)
- net MCU_SPI_NSS: now reaches U203.101 (IO_L32N_1)
- net MCU_SPI_MOSI: now reaches U203.102 (IO_L32P_1)
- net MCU_SPI_MISO: now reaches U203.104 (IO_L1N_VREF_1)
- net MCU_SPI_CLK: now reaches U203.105 (IO_L1P_1)
Changed lines of the file:
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@@
-    (stroke (width 0) (type default))
-  )
-  (wire (pts (xy 379.095 71.12) (xy 380.365 71.12))
     (stroke (width 0) (type default))
   )
@@
     (stroke (width 0) (type default))
   )
-  (wire (pts (xy 380.365 76.2) (xy 379.095 76.2))
-    (stroke (width 0) (type default))
-  )
   (wire (pts (xy 81.28 229.87) (xy 81.28 231.14))
     (stroke (width 0) (type default))
@@
     (stroke (width 0) (type default))
   )
+  (wire (pts (xy 182.245 49.53) (xy 180.975 49.53))
+    (stroke (width 0) (type default))
+  )
   (wire (pts (xy 156.21 163.83) (xy 155.575 163.83))
     (stroke (width 0) (type default))
@@
     (stroke (width 0) (type default))
   )
+  (wire (pts (xy 182.245 57.15) (xy 180.975 57.15))
+    (stroke (width 0) (type default))
+  )
   (wire (pts (xy 236.855 276.225) (xy 236.855 276.86))
     (stroke (width 0) (type default))
@@
     (stroke (width 0) (type default))
   )
+  (wire (pts (xy 180.975 54.61) (xy 182.245 54.61))
+    (stroke (width 0) (type default))
+  )
   (wire (pts (xy 39.37 229.87) (xy 32.385 229.87))
     (stroke (width 0) (type default))
@@
     (stroke (width 0) (type default))
   )
+  (wire (pts (xy 182.245 52.07) (xy 180.975 52.07))
+    (stroke (width 0) (type default))
+  )
   (bus (pts (xy 36.195 205.74) (xy 36.195 203.2))
     (stroke (width 0) (type default))
@@
     (stroke (width 0) (type default))
   )
-  (wire (pts (xy 380.365 68.58) (xy 379.095 68.58))
-    (stroke (width 0) (type default))
-  )
   (wire (pts (xy 27.94 276.225) (xy 27.94 276.86))
     (stroke (width 0) (type default))
@@
     (stroke (width 0) (type default))
   )
-  (wire (pts (xy 380.365 73.66) (xy 379.095 73.66))
+  (wire (pts (xy 79.375 69.85) (xy 61.595 69.85))
     (stroke (width 0) (type default))
   )
@@
     (effects (font (size 1.27 1.27)) (justify right bottom))
   )
+  (label "FPGA_CLK_100MHZ" (at 61.595 69.85 0) (fields_autoplaced)
+    (effects (font (size 1.27 1.27)) (justify left bottom))
+  )
   (label "FLASH_INIT_B" (at 230.505 110.49 0) (fields_autoplaced)
     (effects (font (size 1.27 1.27)) (justify left bottom))
@@
     (effects (font (size 1.27 1.27)) (justify right bottom))
   )
-  (hierarchical_label "MCU_SPI2_MISO" (shape output) (at 380.365 68.58 0) (fields_autoplaced)
-    (effects (font (size 1.27 1.27)) (justify left))
-  )
-  (hierarchical_label "MCU_SPI2_CS" (shape input) (at 380.365 73.66 0) (fields_autoplaced)
+  (hierarchical_label "MCU_SPI_NSS" (shape input) (at 182.245 57.15 0) (fields_autoplaced)
     (effects (font (size 1.27 1.27)) (justify left))
   )
@@
     (effects (font (size 1.27 1.27)) (justify right))
   )
-  (hierarchical_label "MCU_SPI2_MOSI" (shape input) (at 380.365 71.12 0) (fields_autoplaced)
+  (hierarchical_label "MCU_SPI_CLK" (shape input) (at 182.245 49.53 0) (fields_autoplaced)
     (effects (font (size 1.27 1.27)) (justify left))
   )
-  (hierarchical_label "MCU_SPI2_CLK" (shape input) (at 380.365 76.2 0) (fields_autoplaced)
+  (hierarchical_label "MCU_SPI_MOSI" (shape input) (at 182.245 54.61 0) (fields_autoplaced)
     (effects (font (size 1.27 1.27)) (justify left))
   )
+  (hierarchical_label "MCU_SPI_MISO" (shape output) (at 182.245 52.07 0) (fields_autoplaced)
+    (effects (font (size 1.27 1.27)) (justify left))
+  )

Commit message: Schematic and PCB design
Connections:
- net MCU_GPIO1: now reaches U203.100 (IO_L33P_1)
- net SDRAM_A9: now reaches U203.114 (IO_L65N_SCP2_0)
- net SDRAM_A8: now reaches U203.115 (IO_L65P_SCP3_0)
- net SDRAM_A7: now reaches U203.116 (IO_L64N_SCP4_0)
- net SDRAM_A6: now reaches U203.117 (IO_L64P_SCP5_0)
- net SDRAM_A5: now reaches U203.118 (IO_L63N_SCP6_0)
- net SDRAM_~{WE}: now reaches U203.119 (IO_L63P_SCP7_0)
- net SDRAM_IO7: now reaches U203.120 (IO_L62N_VREF_0)
- net SDRAM_IO6: now reaches U203.121 (IO_L62P_0)
- net SDRAM_IO5: now reaches U203.123 (IO_L37N_GCLK12_0)
- net SDRAM_IO4: now reaches U203.124 (IO_L37P_GCLK13_0)
- net SDRAM_IO3: now reaches U203.126 (IO_L36N_GCLK14_0)
- net SDRAM_IO2: now reaches U203.127 (IO_L36P_GCLK15_0)
- net SDRAM_IO1: now reaches U203.131 (IO_L35N_GCLK16_0)
- net SDRAM_IO0: now reaches U203.132 (IO_L35P_GCLK17_0)
- net SDRAM_~{CE}: now reaches U203.133 (IO_L34N_GCLK18_0)
- net SDRAM_A4: now reaches U203.137 (IO_L4N_0)
- net SDRAM_A3: now reaches U203.138 (IO_L4P_0)
- net SDRAM_A2: now reaches U203.139 (IO_L3N_0)
- net SDRAM_A1: now reaches U203.140 (IO_L3P_0)
- net SDRAM_A0: now reaches U203.141 (IO_L2N_0)
- net MCU_GPIO2: now reaches U203.99 (IO_L33N_1)
- net SDRAM_A17: now reaches U203.43 (IO_L62N_D6_2)
- net SDRAM_A16: now reaches U203.44 (IO_L62P_D5_2)
- net SDRAM_A15: now reaches U203.45 (IO_L49N_D4_2)
- net SDRAM_~{OE}: now reaches U203.46 (IO_L49P_D3_2)
- net SDRAM_~{UB}: now reaches U203.47 (IO_L48N_RDWR_B_VREF_2)
- net SDRAM_~{LB}: now reaches U203.48 (IO_L48P_D7_2)
- net SDRAM_IO15: now reaches U203.50 (IO_L31N_GCLK30_D15_2)
- net SDRAM_IO14: now reaches U203.51 (IO_L31P_GCLK31_D14_2)
- net SDRAM_IO13: now reaches U203.55 (IO_L30N_GCLK0_USERCCLK_2)
- net SDRAM_IO12: now reaches U203.56 (IO_L30P_GCLK1_D13_2)
- net SDRAM_IO11: now reaches U203.57 (IO_L14N_D12_2)
- net SDRAM_IO10: now reaches U203.58 (IO_L14P_D11_2)
- net SDRAM_IO9: now reaches U203.59 (IO_L13N_D10_2)
- net SDRAM_IO8: now reaches U203.61 (IO_L12N_D2_MISO3_2)
- net SDRAM_A14: now reaches U203.62 (IO_L12P_D1_MISO2_2)
- net SDRAM_A13: now reaches U203.64 (IO_L3N_MOSI_CSI_B_MISO0_2)
- net SDRAM_A12: now reaches U203.65 (IO_L3P_D0_DIN_MISO_MISO1_2)
- net SDRAM_A11: now reaches U203.66 (IO_L2N_CMPMOSI_2)
- net SDRAM_A10: now reaches U203.67 (IO_L2P_CMPCLK_2)
Other:
- moved on the sheet: D201, R204, R207, R208, R209, U203A, U203B, U203C, U203D

Commit message: FPGA code
Connections:
- net SQ_AMPL_CLK: now reaches U203.81 (IO_L46P_1)
- net SQ_AMPL_LE: now reaches U203.82 (IO_L45N_1)
- net SQ_AMPL_DATA: now reaches U203.83 (IO_L45P_1)
- net MSEL0: now reaches U203.92 (IO_L41N_GCLK8_1)
- net MSEL2: now reaches U203.93 (IO_L41P_GCLK9_IRDY1_1)
- net MSEL1: now reaches U203.94 (IO_L40N_GCLK10_1)
- net ADC_DATA: now reaches U203.95 (IO_L40P_GCLK11_1)
- net ADC_CLK: now reaches U203.97 (IO_L34N_1)
- net ADC_CONV: now reaches U203.98 (IO_L34P_1)
- net WFD_FPGA_50MHZ: now reaches U203.23 (IO_L41N_GCLK26_3)
- net DAC_nLDAC: now reaches U203.24 (IO_L41P_GCLK27_3)
- net DAC_nSYNC: now reaches U203.26 (IO_L37N_3)
- net DAC_nCLR: now reaches U203.27 (IO_L37P_3)
- net DAC_DIN: now reaches U203.29 (IO_L36N_3)
- net DAC_SCLK: now reaches U203.30 (IO_L36P_3)
- net SQ_COMP_EN: now reaches U203.33 (IO_L2P_3)
- net SET_SIN-ARB_FLTR2: now reaches U203.34 (IO_L1N_VREF_3)
- net SET_SIN-ARB_FLTR1: now reaches U203.35 (IO_L1P_3)
Other:
- moved on the sheet: R204, U203A, U203B
