File: hardware/ETH1CFGEN1/Power.kicad_sch (KiCad schematic)
At the start: 0 parts

Commit message: Development
Parts:
- added C701, C702: 10u/50V, Capacitor_SMD:C_1206_3216Metric_Pad1.42x1.75mm_HandSolder, symbol Device:C
- added C703, C704, C711, C712, C713, C714, C715, C716: 4u7/50V, Capacitor_SMD:C_1206_3216Metric_Pad1.42x1.75mm_HandSolder, symbol Device:C
- added C705, C706: 1u, Capacitor_SMD:C_0603_1608Metric_Pad1.05x0.95mm_HandSolder, symbol Device:C
- added C707, C708: 1u/HC, Capacitor_SMD:C_1206_3216Metric_Pad1.42x1.75mm_HandSolder, symbol Device:C
- added C709, C710: 4p7, Capacitor_SMD:C_0603_1608Metric_Pad1.05x0.95mm_HandSolder, symbol Device:C
- added D701, D702: PMEG6010EP,115, Diode_SMD:D_SOD-128, symbol Device:D_Schottky
- added L701, L702: 74489440068, ETH1CLCR1:74489440068, symbol ETH1CLCR1:74489440068
- added R701, R703, R705, R707: 1M, Resistor_SMD:R_0603_1608Metric_Pad1.05x0.95mm_HandSolder, symbol Device:R
- added R702, R704: 287k, Resistor_SMD:R_0603_1608Metric_Pad1.05x0.95mm_HandSolder, symbol Device:R
- added R706: 97k6, Resistor_SMD:R_0603_1608Metric_Pad1.05x0.95mm_HandSolder, symbol Device:R
- added R708: 46k4, Resistor_SMD:R_0603_1608Metric_Pad1.05x0.95mm_HandSolder, symbol Device:R
- added U701, U702: LT8330_S6, Package_TO_SOT_SMD:TSOT-23-6_HandSoldering, symbol ETH1CLCR1:LT8330_S6
- added U703: MC7815BD2TG, Package_TO_SOT_SMD:TO-263-2, symbol Regulator_Linear:L7815
- added U704: MC7915BD2TG, Package_TO_SOT_SMD:TO-263-2, symbol Regulator_Linear:MC79M15_TO252
Connections:
- new net: C708.1, D701.2 (A), L702.2
- new net: C709.1, C711.1, C713.1, D702.1 (K), R705.1, U703.1 (IN)
- new net: C710.1, C712.1, C714.1, L702.3, R707.1, U704.2 (VI)
- new net: C707.1, D702.2 (A), L701.2
- new net: R701.2, R702.1, U701.4 (EN/UVLO)
- new net: C708.2, L702.4, U702.1 (SW)
- new net: C710.2, R707.2, R708.1, U702.3 (FBX)
- new net: R703.2, R704.1, U702.4 (EN/UVLO)
- new net: C706.1, U702.5 (INTVCC)
- new net: C707.2, L701.4, U701.1 (SW)
- new net: C709.2, R705.2, R706.1, U701.3 (FBX)
- new net: C705.1, U701.5 (INTVCC)
- new net +15V: C715.1, U703.3 (OUT)
- new net +24VF: C701.1, C702.1, C703.1, C704.1, L701.1, L702.1, R701.1, R703.1, U701.6 (VIN), U702.6 (VIN)
- new net -15V: C716.1, U704.3 (VO)
- new net DGNDF: D701.1 (K), L701.3
- new net GNDA: C701.2, C702.2, C703.2, C704.2, C705.2, C706.2, C711.2, C712.2, C713.2, C714.2, C715.2, C716.2, R702.2, R704.2, R706.2, R708.2, U701.2 (GND), U702.2 (GND), U703.2 (GND), U704.1 (GND)
