File: hardware/ETH1CFGEN1/Power.kicad_sch (KiCad schematic)
At the start: 89 parts, among them Q601 IRFR5410, U601 TSR1-2450, U602 LT8330ES6#TRMPBF, U603 LT8330ES6#TRMPBF, U604 TSR1-2433, U605 MAX5902AAEUT+T, U606 MC7815BD2TR4G, U607 MC7915ACD2TG, U608 LT8330ES6#TRMPBF, U609 LT8330ES6#TRMPBF, U610 THL15-2415WI, U611 MC7805CD2TG, U612 L7905CD2T-TR

Commit message: PCB design
Parts:
- added C309 (x4): 22u/35V, Capacitor_Tantalum_SMD:CP_EIA-7343-31_Kemet-D_Pad2.25x2.55mm_HandSolder, symbol Device:C_Polarized
Connections:
- net +15V: now also C309.1
- net +5V: now also C309.1
- net -15V: now also C309.2
- net -5V: now also C309.2
- net GNDA: now also C309.1, C309.1, C309.2, C309.2
Other:
- moved on the sheet: C602, C603, C605, C606, C608, C609, C611, C612, C615, C616, C617, C618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

Commit message: PCB design
Changed lines of the file:
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@@
       (effects (font (size 1.27 1.27)) hide)
     )
-    (property "Value" "+3.3V" (at 250.19 256.794 0)
+    (property "Value" "+3.3V" (at 250.19 256.54 0)
       (effects (font (size 1.27 1.27)))
     )
@@
       (effects (font (size 1.27 1.27)) hide)
     )
-    (property "Value" "+5VD" (at 262.255 255.905 0)
+    (property "Value" "+5VD" (at 262.255 256.54 0)
       (effects (font (size 1.27 1.27)))
     )
@@
         (path "/44bc1157-6d68-4ab3-afc0-b8d9f089cc50/61e965c1-e946-4500-a63b-fb711a3a2ae7"
           (reference "#PWR0606") (unit 1)
-        )
-      )
-    )
-  )
-  (symbol (lib_id "power:PWR_FLAG") (at 236.22 260.35 0) (unit 1)
-    (in_bom yes) (on_board yes) (dnp no)
-    (property "Reference" "#FLG0605" (at 236.22 258.445 0)
-      (effects (font (size 1.27 1.27)) hide)
-    )
-    (property "Value" "PWR_FLAG" (at 236.22 256.54 0)
-      (effects (font (size 1.27 1.27)))
-    )
-    (property "Footprint" "" (at 236.22 260.35 0)
-      (effects (font (size 1.27 1.27)) hide)
-    )
-    (property "Datasheet" "~" (at 236.22 260.35 0)
-      (effects (font (size 1.27 1.27)) hide)
-    )
-    (pin "1")
-    (instances
-      (project "ETH1CFGEN1"
-        (path "/44bc1157-6d68-4ab3-afc0-b8d9f089cc50/61e965c1-e946-4500-a63b-fb711a3a2ae7"
-          (reference "#FLG0605") (unit 1)
-        )
-      )
-      (project "ETH1CLCR1"
-        (path "/da26c521-26ba-46a0-91ab-131d1ff07c76/00000000-0000-0000-0000-00005dec0296"
-          (reference "#FLG01502") (unit 1)
         )
       )
@@
         )
       )
-    )
-  )
-  (symbol (lib_id "power:GNDD") (at 236.22 260.35 0) (unit 1)
-    (in_bom yes) (on_board yes) (dnp no) (fields_autoplaced)
-    (property "Reference" "#PWR0626" (at 236.22 266.7 0)
-      (effects (font (size 1.27 1.27)) hide)
-    )
-    (property "Value" "GNDD" (at 236.22 264.795 0)
-      (effects (font (size 1.27 1.27)))
-    )
-    (property "Footprint" "" (at 236.22 260.35 0)
-      (effects (font (size 1.27 1.27)) hide)
-    )
-    (property "Datasheet" "" (at 236.22 260.35 0)
-      (effects (font (size 1.27 1.27)) hide)
-    )
-    (pin "1")
-    (instances
-      (project "ETH1CFGEN1"
-        (path "/44bc1157-6d68-4ab3-afc0-b8d9f089cc50/61e965c1-e946-4500-a63b-fb711a3a2ae7"
-          (reference "#PWR0626") (unit 1)
-        )
-      )

Commit message: Schematic and PCB design
Parts:
- renumbered C605 to C604, C606 to C605, C611 to C610, C612 to C611, C615 to C614, C616 to C615, C623 to C625, C624 to C626, C625 to C627, C626 to C628, C627 to C629, C628 to C630, C629 to C631, C630 to C632, C631 to C633, C632 to C634, C633 to C635, C634 to C636, C635 to C637, C636 to C638, C637 to C639, C638 to C640, C639 to C641, C640 to C642, C641 to C643, C642 to C644, R606 to R605, R607 to R606, R608 to R607, R609 to R608, R605 to R609
