File: hardware/ETH1CFGEN1/WaveformDAC.kicad_sch (KiCad schematic)
At the start: 13 parts, among them K601 G6SU-2F-DC3, U601 AD9744, U602 TL072, X1 SG5032CAN 50.000000M-TJGA3

Commit message: Development
Parts:
- removed R605: 1k, symbol Device:R
- added C603, C605, C606, C612, C617, C641, C644, C645, C651, C665, C666: 0.1u, symbol Device:C
- added C604, C607, C608, C620, C625, C626, C650, C652, C657: 10u, symbol Device:C
- added C609: 22u, symbol Device:C
- added C610, C611, C661, C662, C675, C677: 100p, symbol Device:C
- added C613, C614, C618, C619, C631, C632, C642, C643, C658, C659, C682: 33p, symbol Device:C
- added C615, C616: 30p, symbol Device:C
- added C621, C622, C627, C628, C633, C634, C655, C656: 56p, symbol Device:C
- added C623, C624: 3p3, symbol Device:C
- added C629, C630: 120p, symbol Device:C
- added C635, C636, C683: 150p, symbol Device:C
- added C637, C638: 62p, symbol Device:C
- added C639, C640: 8p2, symbol Device:C
- added C646, C647: 130p, symbol Device:C
- added C648, C649: 330p, symbol Device:C
- added C653, C654, C681: 15p, symbol Device:C
- added C660, C671: 0.22u, symbol Device:C
- added C663, C664: 5p6, symbol Device:C
- added C667, C668, C680: 47p, symbol Device:C
- added C669, C670: 22u, symbol Device:C_Polarized
- added C672, C673: 22p, symbol Device:C
- added C674, C678, C679: 10p, symbol Device:C
- added C676: 1p, symbol Device:C
- added D601: BAS40-04, Package_TO_SOT_SMD:SOT-23, symbol Diode:BAS40-04
- added FB601, FB602, FB603, FB604, FB605, FB606, FB607, FB608: KMZ1608SHR102ATD25, symbol Device:FerriteBead_Small
- added K602: G6SU-2F-DC3, symbol Relay:G6SU-2
- added L601, L602, L603, L604, L605, L606: 470n, symbol Device:L
- added L607, L608: 680n, symbol Device:L
- added L609, L610: 560n, symbol Device:L
- added L611, L612: 910n, symbol Device:L
- added L613, L614: 750n, symbol Device:L
- added L615, L616: 1u, symbol Device:L
- added L617: 1u2, symbol Device:L
- added L618: 100n, symbol Device:L
- added Q601: MMBT5087LT1G, symbol Device:Q_PNP_BEC
- added R607, R614: 1k, symbol Device:R
- added R608: 2k, symbol Device:R
- added R609, R613: 69, symbol Device:R
- added R610, R611: 261, symbol Device:R
- added R612: 21k5, symbol Device:R
- added R615, R616, R619, R622, R625: 100, symbol Device:R
- added R617, R623, R627: 10k, symbol Device:R
- added R618, R626: 1k78, symbol Device:R
- added R620, R621: 511, symbol Device:R
- added R624: 21R5, symbol Device:R
- added R628, R635: 51R1, symbol Device:R
- added R629, R630: 200, symbol Device:R
- added R631, R634: 100k, symbol Device:R
- added R632, R633: 953, symbol Device:R
- added R636: 34R8, symbol Device:R
- added R637: 196, symbol Device:R
- added U603: LT1016CS8, symbol Comparator:AD8561
- added U604: THS3001CD, Package_SO:SOIC-8_3.9x4.9mm_P1.27mm, symbol ETH1CFGEN1:THS3001CD
- U602: value TL072 -> TL072CD
- renumbered R604 to R602, R602 to R603, R603 to R604, R606 to R605, R607 to R606
Connections:
- net GND is gone; now on net GNDA: X1.2 (GND)
- net +15V: now also FB603.1, FB604.1; no longer U602.8 (V+)
- net +3.3V: now also FB601.1, FB602.1
- net -15V: now also FB605.1, FB606.1; no longer U602.4 (V-)
- net GNDA: now also C603.2, C604.2, C605.2, C606.2, C607.2, C608.2, C609.2, C612.2, C613.2, C614.1, C615.2, C616.1, C617.2, C620.2, C621.2, C622.1, C623.2, C624.1, C625.2, C626.2, C627.2, C628.1, C629.2, C630.1, C633.2, C634.1, C635.2, C636.1, C637.2, C638.1, C639.2, C640.1, C641.2, C644.2, C645.2, C646.2, C647.1, C648.2, C649.1, C650.2, C652.2, C653.2, C654.1, C655.2, C656.1, C657.2, C660.2, C661.2, C662.1, C663.2, C664.1, C665.2, C666.2, C667.2, C668.1, C669.2, C670.2, C671.2, C672.2, C673.1, C678.1, C679.2, C680.2, C681.2, C682.2, C683.2, D601.1, L615.2, L616.1, R608.1, R615.2, R616.1, R620.2, R621.1, R632.2, U603.6 (GND)
- net GNDD: now also C610.2, C611.1, C675.2, C677.1
- net +3V3_WFD1: now reaches U601.16 (REFLO)
- net +3V3_WFD1: now also U601.24 (AVDD), C605.1, C609.1, D601.2, FB602.2
- net V_AMPL: now reaches U601.17 (REFIO)
- net V_AMPL: now also R602.1, D601.3
- net at U601.18 (FS_ADJ): now also R608.2
- net at C601.1, U601.21 (IOUTB): now also K601.9, R613.1
- net at C602.1, U601.22 (IOUTA): now also K601.4, R609.1
- net at U601.25 (MODE): now also R607.1
- net +3V3_WFD2: now reaches U601.27 (DVDD)
- net +3V3_WFD2: now also C603.1, C604.1, C608.1, FB601.2, R607.2
- net at R605.2: now also Q601.1 (B)
- net at U602.1: now also C651.2, R623.2, R624.1
- net at U602.2 (-): now also R617.2, R623.1
- net at U602.3 (+): now also C660.1, R614.2
- net SET_SIN_FLTR1: now reaches K601.1
- net SET_SIN_FLTR1: now also C611.2
- net at K601.10: now also C616.2, C624.2, L604.1
- net SET_ARB_FLTR1: now reaches K601.12
- net SET_ARB_FLTR1: now also C610.1
- net at K601.3: now also C615.1, C623.1, L603.1
- net at K601.5: now also C613.1, C618.1, L601.1
- net at K601.8: now also C614.2, C619.1, L602.1
- net at R606.2: now also Q601.2 (E), R611.2, R612.1
- new net: C668.2, C673.2, L616.2, R621.2, R622.1
- new net: C674.1, C680.1, L617.1, U603.2 (+)
- new net: C674.2, C676.1, R625.2, R627.1, U603.3 (-)
- new net: C679.1, K602.9, R630.1
- new net: R630.2, R633.1, R634.1, U604.2 (-)
- new net: R629.2, R631.2, R632.1, U604.3 (+)
- new net: C648.1, C655.1, K602.5, L611.2, R615.1, R618.1
- new net: R633.2, R634.2, R636.1, R637.1, U604.6
- new net: C618.2, C621.1, C627.1, C631.1, L601.2, L605.1
- new net: C658.2, C661.1, C663.1, K602.3, L613.2, R619.1, R626.1
- new net: C667.1, C672.1, L615.1, R619.2, R620.1
- new net: C631.2, C633.1, C637.1, C642.1, L605.2, L609.1
- new net: C630.2, L604.2, L608.1
- new net: C649.2, C656.2, K602.8, L612.2, R616.2, R618.2
- new net: C607.1, R610.2, R611.1
- new net: C636.2, C640.2, L608.2, L612.1
- new net: C642.2, C646.1, C653.1, C658.1, L609.2, L613.1
- new net: C671.1, R624.2, R625.1
- new net: C629.1, L603.2, L607.1
- new net: C681.1, L617.2, R637.2
- new net: C619.2, C622.2, C628.2, C632.1, L602.2, L606.1
- new net: C659.2, C662.2, C664.2, K602.10, L614.2, R622.2, R626.2
- new net: C676.2, R627.2, R628.1, R628.2, U603.8 (~{Q})
- new net: C632.2, C634.2, C638.2, C643.1, L606.2, L610.1
- new net: C635.1, C639.1, L607.2, L611.1
- new net: C606.1, R609.2, R610.1, R613.2
- new net: R635.1, U603.7 (Q)
- new net: C643.2, C647.2, C654.2, C659.1, L610.2, L614.1
- new net: C682.1, L618.1, R636.2
- new net: C678.2, K602.4, R629.1
- new net +15V_WFD1: C617.1, C625.1, FB604.2, R612.2, U602.8 (V+)
- new net +15V_WFD2: C612.1, C620.1, C626.1, FB603.2, U604.7 (V+)
- new net +2V5: R617.1
- new net +5V: FB607.1
- new net +5V_WFD: C665.1, C669.1, FB607.2, U603.1 (V+)
- new net -15V_WFD1: C645.1, C652.1, FB606.2, Q601.3 (C), U602.4 (V-)
- new net -15V_WFD2: C641.1, C650.1, C657.1, FB605.2, U604.4 (V-)
- new net -5V: FB608.1
- new net -5V_WFD: C666.1, C670.1, FB608.2, U603.4 (V-)
- new net SET_ARB_FLTR2: C675.1, K602.1
- new net SET_SIN_FLTR2: C677.2, K602.12
- new net SINE_ARB: C683.1, L618.2
- new net SQUARE: R635.2
- new net SQ_COMP_EN: U603.5 (LATCH)
- new net V_DTY_CYCL: C644.1, C651.1, R614.1
- new net V_NULL_SINE: R631.1
Other:
- moved on the sheet: C601, C602, K601, R1, R602, R603, R604, R605, R606, U601, U602A, U602B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
