File: hardware/ETH1CFGEN1/WaveformDAC.kicad_sch (KiCad schematic)
At the start: 153 parts, among them K301 G6SU-2F-DC3, K302 G6SU-2F-DC3, Q301 MMBT5087LT1G, U301 TL072CDT, U302 AD9744, U303 LT1016CS8, U304 THS3001IDG, X1 SG5032CAN 50.000000M-TJGA3

Commit message: Development
Parts:
- removed C309, C367, C368: 22u, symbol Device:C_Polarized
- added C309 (x3): 22u, Capacitor_Tantalum_SMD:CP_EIA-7343-31_Kemet-D_Pad2.25x2.55mm_HandSolder, symbol Device:C_Polarized
- K301, K302: footprint (none) -> Relay_SMD:Relay_DPDT_Omron_G6SK-2F
- L301, L302, L303, L304, L305, L306, L307, L308, L309, L310, L311, L312, L313, L314, L315, L316, L317, L318: footprint (none) -> Inductor_SMD:L_0603_1608Metric_Pad1.05x0.95mm_HandSolder
- Q301: footprint (none) -> Package_TO_SOT_SMD:SOT-23
Connections:
- net +3V3_WFD1: now also C309.1
- net +5V_WFD: now also C309.1
- net -5V_WFD: now also C309.2
- net GNDA: now also C309.1, C309.2, C309.2

Commit message: PCB design
Parts:
- removed C303, C305, C312, C317, C341, C344, C363, C364: 100n, Capacitor_SMD:C_0603_1608Metric_Pad1.08x0.95mm_HandSolder, symbol Device:C
- removed C304, C308, C324, C325, C354, C355: 10u, Capacitor_SMD:C_1206_3216Metric_Pad1.33x1.80mm_HandSolder, symbol Device:C
- removed C309 (x3): 22u, Capacitor_Tantalum_SMD:CP_EIA-7343-31_Kemet-D_Pad2.25x2.55mm_HandSolder, symbol Device:C_Polarized
- removed FB301, FB302, FB303, FB304, FB305, FB306, FB307, FB308: KMZ1608SHR102ATD25, Inductor_SMD:L_0603_1608Metric_Pad1.05x0.95mm_HandSolder, symbol Device:FerriteBead_Small
- L301, L302, L303, L304, L305, L306, L307, L308, L309, L310, L311, L312, L313, L314, L315, L316, L317, L318: footprint Inductor_SMD:L_0603_1608Metric_Pad1.05x0.95mm_HandSolder -> Inductor_SMD:L_0805_2012Metric_Pad1.15x1.40mm_HandSolder
Connections:
- net +15V_WFD1 is gone; now on net +15V: R312.2, U301.8 (V+)
- net +15V_WFD2 is gone; now on net +15V: U304.7 (V+)
- net +3V3_WFD2 is gone; now on net +3.3V: R307.2, U302.27 (DVDD)
- net +5V_WFD is gone; now on net +5V: U303.1 (V+)
- net -15V_WFD1 is gone; now on net -15V: Q301.3 (C), U301.4 (V-)
- net -15V_WFD2 is gone; now on net -15V: U304.4 (V-), U304.9 (THR)
- net -5V_WFD is gone; now on net -5V: U303.4 (V-)
- net +3.3V: now also D301.2, U302.24 (AVDD)
- net +3V3_WFD1: no longer D301.2, U302.24 (AVDD)
- net at R327.2, R328.2, U303.8 (~{Q}): no longer C374.2, R328.1
- new net: C374.2, R328.1
Other:
- moved on the sheet: C306, C307, R313, R327

Commit message: PCB design
Parts:
- C330, C331: value 33p -> 56p
- C342, C343: value 33p -> 39p
- C356, C357: value 33p -> 5p6
Connections:
- net +3V3_WFD1 is gone; now on net +3.3V: U302.16 (REFLO)
Changed lines of the file:
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@@
   )
   (symbol (lib_id "Device:L") (at 274.32 59.055 0) (unit 1)
-    (in_bom yes) (on_board yes) (dnp no) (fields_autoplaced)
-    (property "Reference" "L316" (at 275.59 57.785 0)
+    (in_bom yes) (on_board yes) (dnp no)
+    (property "Reference" "L316" (at 274.955 57.785 0)
       (effects (font (size 1.27 1.27)) (justify left))
     )
@@
   (symbol (lib_id "Device:C") (at 283.21 59.055 0) (unit 1)
     (in_bom yes) (on_board yes) (dnp no)
-    (property "Reference" "C366" (at 287.02 57.785 0)
+    (property "Reference" "C366" (at 286.385 57.785 0)
       (effects (font (size 1.27 1.27)) (justify left))
     )
@@
   )
   (symbol (lib_id "Device:L") (at 274.32 50.165 0) (unit 1)
-    (in_bom yes) (on_board yes) (dnp no) (fields_autoplaced)
-    (property "Reference" "L315" (at 275.59 48.895 0)
+    (in_bom yes) (on_board yes) (dnp no)
+    (property "Reference" "L315" (at 274.955 48.895 0)
       (effects (font (size 1.27 1.27)) (justify left))
     )
@@
   (symbol (lib_id "Device:C") (at 187.325 78.74 90) (unit 1)
     (in_bom yes) (on_board yes) (dnp no) (fields_autoplaced)
-    (property "Reference" "C331" (at 187.325 71.755 90)
+    (property "Reference" "C331" (at 187.325 71.12 90)
       (effects (font (size 1.27 1.27)))
     )
-    (property "Value" "33p" (at 187.325 74.295 90)
+    (property "Value" "56p" (at 187.325 73.66 90)
       (effects (font (size 1.27 1.27)))
     )
@@
     )
   )
+  (symbol (lib_id "power:+3.3V") (at 41.275 126.365 90) (unit 1)
+    (in_bom yes) (on_board yes) (dnp no) (fields_autoplaced)
+    (property "Reference" "#PWR01142" (at 45.085 126.365 0)
+      (effects (font (size 1.27 1.27)) hide)
+    )
+    (property "Value" "+3.3V" (at 38.1 126.365 90)
+      (effects (font (size 1.27 1.27)) (justify left))
+    )
+    (property "Footprint" "" (at 41.275 126.365 0)
+      (effects (font (size 1.27 1.27)) hide)
+    )
+    (property "Datasheet" "" (at 41.275 126.365 0)
+      (effects (font (size 1.27 1.27)) hide)
+    )
+    (pin "1")
+    (instances
+      (project "ETH1CFGEN1"
+        (path "/44bc1157-6d68-4ab3-afc0-b8d9f089cc50/210fcfe0-f423-48d7-8524-4d1604eac601"
+          (reference "#PWR01142") (unit 1)
+        )
+      )
+    )
+  )
   (symbol (lib_id "Device:R") (at 79.375 66.04 180) (unit 1)
     (in_bom yes) (on_board yes) (dnp no) (fields_autoplaced)
@@
     )
   )
-  (symbol (lib_id "ETH1CFGEN1:+3V3_WFD1") (at 41.275 126.365 90) (unit 1)
-    (in_bom yes) (on_board yes) (dnp no)
-    (property "Reference" "#PWR0307" (at 45.085 126.365 0)
-      (effects (font (size 1.27 1.27)) hide)
-    )
-    (property "Value" "+3V3_WFD1" (at 33.02 126.365 90)
-      (effects (font (size 1.27 1.27)))
-    )
-    (property "Footprint" "" (at 41.275 126.365 0)
-      (effects (font (size 1.27 1.27)) hide)
-    )
-    (property "Datasheet" "" (at 41.275 126.365 0)
-      (effects (font (size 1.27 1.27)) hide)
-    )
-    (pin "1")
-    (instances
-      (project "ETH1CFGEN1B"
-        (path "/3dceb0a1-97ad-435d-a235-e3839b959163/4a966eb3-1da9-4a67-ba6c-e557098bb995"
-          (reference "#PWR0307") (unit 1)
-        )
-      )
-      (project "ETH1CFGEN1"
-        (path "/44bc1157-6d68-4ab3-afc0-b8d9f089cc50/210fcfe0-f423-48d7-8524-4d1604eac601"
-          (reference "#PWR01107") (unit 1)
-        )
-      )
-    )
-  )
   (symbol (lib_id "Device:L") (at 215.9 92.71 90) (unit 1)
     (in_bom yes) (on_board yes) (dnp no)
@@
   (symbol (lib_id "Device:C") (at 212.09 78.74 90) (unit 1)
     (in_bom yes) (on_board yes) (dnp no) (fields_autoplaced)
-    (property "Reference" "C343" (at 212.09 71.755 90)
+    (property "Reference" "C343" (at 212.09 71.12 90)
       (effects (font (size 1.27 1.27)))
     )
-    (property "Value" "33p" (at 212.09 74.295 90)
+    (property "Value" "39p" (at 212.09 73.66 90)
       (effects (font (size 1.27 1.27)))
     )
@@
   (symbol (lib_id "Device:C") (at 283.21 50.165 0) (unit 1)
     (in_bom yes) (on_board yes) (dnp no)
-    (property "Reference" "C365" (at 287.02 48.895 0)
+    (property "Reference" "C365" (at 286.385 48.895 0)
       (effects (font (size 1.27 1.27)) (justify left))
     )
@@
   )
   (symbol (lib_id "Device:R") (at 266.065 50.165 0) (unit 1)
-    (in_bom yes) (on_board yes) (dnp no) (fields_autoplaced)
-    (property "Reference" "R320" (at 268.605 48.895 0)
+    (in_bom yes) (on_board yes) (dnp no)
+    (property "Reference" "R320" (at 267.97 48.895 0)
       (effects (font (size 1.27 1.27)) (justify left))
     )
@@
   )
   (symbol (lib_id "Device:R") (at 266.065 59.055 0) (unit 1)
-    (in_bom yes) (on_board yes) (dnp no) (fields_autoplaced)
-    (property "Reference" "R321" (at 268.605 57.785 0)
+    (in_bom yes) (on_board yes) (dnp no)
+    (property "Reference" "R321" (at 267.97 57.785 0)
       (effects (font (size 1.27 1.27)) (justify left))
     )
@@
   )
   (symbol (lib_id "Device:R") (at 305.435 54.61 0) (unit 1)
-    (in_bom yes) (on_board yes) (dnp no) (fields_autoplaced)
-    (property "Reference" "R326" (at 307.975 53.34 0)
+    (in_bom yes) (on_board yes) (dnp no)
+    (property "Reference" "R326" (at 307.34 53.34 0)
       (effects (font (size 1.27 1.27)) (justify left))
     )
-    (property "Value" "1k78" (at 307.975 55.88 0)
+    (property "Value" "1k78" (at 307.34 55.88 0)
       (effects (font (size 1.27 1.27)) (justify left))
     )
@@
   (symbol (lib_id "Device:C") (at 236.855 78.74 90) (unit 1)
     (in_bom yes) (on_board yes) (dnp no) (fields_autoplaced)
-    (property "Reference" "C357" (at 236.855 71.755 90)
+    (property "Reference" "C357" (at 236.855 71.12 90)
       (effects (font (size 1.27 1.27)))
     )
-    (property "Value" "33p" (at 236.855 74.295 90)
+    (property "Value" "5p6" (at 236.855 73.66 90)
       (effects (font (size 1.27 1.27)))
     )
@@
       (effects (font (size 1.27 1.27)))
     )
-    (property "Value" "33p" (at 187.325 29.21 90)
+    (property "Value" "56p" (at 187.325 29.21 90)
       (effects (font (size 1.27 1.27)))
     )
@@
       (effects (font (size 1.27 1.27)))
     )
-    (property "Value" "33p" (at 212.09 29.21 90)
+    (property "Value" "39p" (at 212.09 29.21 90)
       (effects (font (size 1.27 1.27)))
     )
@@
       (effects (font (size 1.27 1.27)))
     )
-    (property "Value" "33p" (at 236.855 29.21 90)
+    (property "Value" "5p6" (at 236.855 29.21 90)
       (effects (font (size 1.27 1.27)))
     )

Commit message: PCB design
Parts:
- removed C310, C311, C373, C375: 100p, Capacitor_SMD:C_0603_1608Metric_Pad1.08x0.95mm_HandSolder, symbol Device:C
- removed K301, K302: G6SU-2F-DC3, Relay_SMD:Relay_DPDT_Omron_G6SK-2F, symbol Relay:G6SU-2
- added D1102, D1103: 1N4148W, Diode_SMD:D_SOD-123, symbol Diode:1N4148W
- added K1101, K1102: G6S-2F-DC5, Relay_SMD:Relay_DPDT_Omron_G6SK-2F, symbol Relay:G6S-2
- added Q1102, Q1103: BC847, Package_TO_SOT_SMD:SOT-23, symbol Transistor_BJT:BC847
- added R307 (x2): 1k, Resistor_SMD:R_0603_1608Metric_Pad0.98x0.95mm_HandSolder, symbol Device:R
Connections:
- net GNDD: now also Q1102.2 (E), Q1103.2 (E)
- net at C301.1, R313.1, U302.21 (IOUTB): now also K1101.9
- net at C302.1, R309.1, U302.22 (IOUTA): now also K1101.4
- net at C377.1, R330.1: now also K1102.9
- net at C347.1, C352.1, L311.2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: now also K1102.5
- net at C315.1, C322.1, L303.1: now also K1101.3
- net at C356.2, C359.1, C361.1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: now also K1102.3
- net at C316.2, C323.2, L304.1: now also K1101.10
- net at C348.2, C353.2, L312.2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: now also K1102.8
- net at C357.2, C360.2, C362.2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: now also K1102.10
- net at C313.1, C318.1, L301.1: now also K1101.5
- net at C376.2, R329.1: now also K1102.4
- net at C314.2, C319.1, L302.1: now also K1101.8
- new net: Q1103.1 (B), R307.1
- new net: D1103.2 (A), K1102.12, Q1103.3 (C)
- new net: D1102.2 (A), K1101.12, Q1102.3 (C)
- new net: Q1102.1 (B), R307.1
- new net +5VD: D1102.1 (K), D1103.1 (K), K1101.1, K1102.1
- new net SET_SIN-ARB_FLTR1: R307.2
- new net SET_SIN-ARB_FLTR2: R307.2
