File: hardware/ETH1CFGEN1/ETH1CFGEN1.kicad_pcb (KiCad board)
At the start: 4 copper layers, 160 x 100 mm, 505 parts, among them J201 Conn_02x01, J202 20021111-00010T4LF, J501 C64AC, J701 Conn_01x06, K501 HE3621A0510, K502 HE3621A0510, K503 HE3621A0510, K504 HE3621A0510, K505 HE3621A0510, K506 HE3621A0510, Q1301 2N7002, Q601 IRFR5410, U1101 TL072CDT, U1102 AD9744, U1103 LT1016CS8, U1104 THS3001IDG, U1201 AD706ARZ, U1202 AD706ARZ, U1203 AD706ARZ, U1204 AD1851RZ, U1205 AD8180ARZ, U1206 AD8009AR, U1207 AD8009AR, U1304 THS3001IDG, U1305 THS3001IDG, U1306 THS3001IDG, U1307 THS3001IDG, U201 HDC1080, U202 STM32F746ZG, U203 24LC08B-E/MS, U301 LAN8742, U302 LC03-3.3BTG, U303 LC03-3.3BTG, U401 TXB0104PW, U402 ADuM5402, U403 74AC125, U501 ULN2003AIPWR, U601 TSR1-2450, U602 LT8330ES6#TRMPBF, U603 LT8330ES6#TRMPBF, U604 TSR1-2433, U605 MAX5902AAEUT+T, U606 MC7815BD2TR4G, U607 MC7915ACD2TG, U608 LT8330ES6#TRMPBF, U609 LT8330ES6#TRMPBF, U610 THL15-2415WI, U611 MC7805CD2TG, U612 L7905CD2T-TR, U701 TLV1117LV33DCYR, U702 TLV1117LV12DCYR, U703 XC6SLX9-3TQG144I, U704 W25Q64JV, U801 TL074HIPWR, U802 TL074HIPWR, U803 TLA2528IRTER, X1101 SG5032CAN 50.000000M-TJGA3, Y201 NX5032GA-16.000M, Y301 NX5032GA-25.000000MHZ-LN-CD-1

Commit message: Development
Parts:
- removed J701: Conn_01x06, Connector_PinHeader_2.54mm:PinHeader_1x06_P2.54mm_Vertical
- added C1001: 100n, Capacitor_SMD:C_0603_1608Metric_Pad1.08x0.95mm_HandSolder, F.Cu at (36.9, -15.8)
- added C1002: 22u, Capacitor_Tantalum_SMD:CP_EIA-7343-31_Kemet-D_Pad2.25x2.55mm_HandSolder, F.Cu at (36.9, -13.3)
- added C1003: 10u, Capacitor_SMD:C_1206_3216Metric_Pad1.33x1.80mm_HandSolder, F.Cu at (36.9, -10.8)
- added C1004: 470p, Capacitor_SMD:C_0603_1608Metric_Pad1.08x0.95mm_HandSolder, F.Cu at (36.9, -8.25)
- added C1005: 330p, Capacitor_SMD:C_0603_1608Metric_Pad1.08x0.95mm_HandSolder, F.Cu at (36.9, -5.74)
- added C1006: 220p, Capacitor_SMD:C_0603_1608Metric_Pad1.08x0.95mm_HandSolder, F.Cu at (36.9, -3.23)
- added C1007: 10u, Capacitor_SMD:C_1206_3216Metric_Pad1.33x1.80mm_HandSolder, F.Cu at (36.9, -0.72)
- added C1008: 1000p, Capacitor_SMD:C_0603_1608Metric_Pad1.08x0.95mm_HandSolder, F.Cu at (121.1, -42.3)
- added C1009: 150p, Capacitor_SMD:C_0603_1608Metric_Pad1.08x0.95mm_HandSolder, F.Cu at (41.2, -15.8)
- added C1010: 4700p, Capacitor_SMD:C_0603_1608Metric_Pad1.08x0.95mm_HandSolder, F.Cu at (123.2, -46.9)
- added C1011: 2u2, Capacitor_SMD:C_1206_3216Metric_Pad1.33x1.80mm_HandSolder, F.Cu at (121.1, -39.0)
- added C1012: 100n, Capacitor_SMD:C_0603_1608Metric_Pad1.08x0.95mm_HandSolder, F.Cu at (121.1, -35.6)
- added C1013: 100n, Capacitor_SMD:C_0603_1608Metric_Pad1.08x0.95mm_HandSolder, F.Cu at (41.2, -13.3)
- added C1109: 22u, Capacitor_Tantalum_SMD:CP_EIA-7343-31_Kemet-D_Pad2.25x2.55mm_HandSolder, F.Cu at (106.1, -48.0)
- added C1167: 22u, Capacitor_Tantalum_SMD:CP_EIA-7343-31_Kemet-D_Pad2.25x2.55mm_HandSolder, F.Cu at (106.1, -42.1)
- added C1168: 22u, Capacitor_Tantalum_SMD:CP_EIA-7343-31_Kemet-D_Pad2.25x2.55mm_HandSolder, F.Cu at (106.1, -36.3)
- added C1202: 22u, Capacitor_Tantalum_SMD:CP_EIA-7343-31_Kemet-D_Pad2.25x2.55mm_HandSolder, F.Cu at (111.0, -67.8)
- added C1206: 22u, Capacitor_Tantalum_SMD:CP_EIA-7343-31_Kemet-D_Pad2.25x2.55mm_HandSolder, F.Cu at (111.0, -61.9)
- added C1301: 100p, Capacitor_SMD:C_0603_1608Metric_Pad1.08x0.95mm_HandSolder, F.Cu at (9.04, -55.4)
- added C1302: 10u, Capacitor_SMD:C_1206_3216Metric_Pad1.33x1.80mm_HandSolder, F.Cu at (40.3, -48.6)
- added C1305: 100n, Capacitor_SMD:C_0603_1608Metric_Pad1.08x0.95mm_HandSolder, F.Cu at (9.04, -52.9)
- added C1306: 100n, Capacitor_SMD:C_0603_1608Metric_Pad1.08x0.95mm_HandSolder, F.Cu at (9.04, -50.4)
- added C1307: 100p, Capacitor_SMD:C_0603_1608Metric_Pad1.08x0.95mm_HandSolder, F.Cu at (9.04, -47.9)
- added C1308: 100p, Capacitor_SMD:C_0603_1608Metric_Pad1.08x0.95mm_HandSolder, F.Cu at (9.04, -45.4)
- added C1309: 1n, Capacitor_SMD:C_0603_1608Metric_Pad1.08x0.95mm_HandSolder, F.Cu at (9.04, -42.9)
- added C1310: 1n, Capacitor_SMD:C_0603_1608Metric_Pad1.08x0.95mm_HandSolder, F.Cu at (9.04, -40.4)
- added C1311: 1n, Capacitor_SMD:C_0603_1608Metric_Pad1.08x0.95mm_HandSolder, F.Cu at (9.04, -37.9)
- added C1312: 1u, Capacitor_SMD:C_0603_1608Metric_Pad1.08x0.95mm_HandSolder, F.Cu at (122.1, 24.3)
- added C1313: 1u, Capacitor_SMD:C_0603_1608Metric_Pad1.08x0.95mm_HandSolder, F.Cu at (122.1, 26.8)
- added C1314: 100p, Capacitor_SMD:C_0603_1608Metric_Pad1.08x0.95mm_HandSolder, F.Cu at (9.04, -35.4)
- added C1315: 100p, Capacitor_SMD:C_0603_1608Metric_Pad1.08x0.95mm_HandSolder, F.Cu at (9.04, -32.8)
- added C1316: 1u, Capacitor_SMD:C_0603_1608Metric_Pad1.08x0.95mm_HandSolder, F.Cu at (122.1, 29.3)
- added C1317: 10n, Capacitor_SMD:C_0603_1608Metric_Pad1.08x0.95mm_HandSolder, F.Cu at (9.04, -30.3)
- added C1318: 27p, Capacitor_SMD:C_0603_1608Metric_Pad1.08x0.95mm_HandSolder, F.Cu at (9.04, -27.8)
- added C1319: 3p3, Capacitor_SMD:C_0603_1608Metric_Pad1.08x0.95mm_HandSolder, F.Cu at (9.04, -25.3)
- added C1320: 18p, Capacitor_SMD:C_0603_1608Metric_Pad1.08x0.95mm_HandSolder, F.Cu at (9.04, -22.8)
- added C1321: 18p, Capacitor_SMD:C_0603_1608Metric_Pad1.08x0.95mm_HandSolder, F.Cu at (9.04, -20.3)
- added C1322: 100p, Capacitor_SMD:C_0603_1608Metric_Pad1.08x0.95mm_HandSolder, F.Cu at (13.4, -55.4)
- added C1323: 100p, Capacitor_SMD:C_0603_1608Metric_Pad1.08x0.95mm_HandSolder, F.Cu at (13.4, -52.9)
- added C1324: 100n, Capacitor_SMD:C_0603_1608Metric_Pad1.08x0.95mm_HandSolder, F.Cu at (13.4, -50.4)
- added C1325: 100n, Capacitor_SMD:C_0603_1608Metric_Pad1.08x0.95mm_HandSolder, F.Cu at (13.4, -47.9)
- added C1326: 100n, Capacitor_SMD:C_0603_1608Metric_Pad1.08x0.95mm_HandSolder, F.Cu at (13.4, -45.4)
- added C1327: 100n, Capacitor_SMD:C_0603_1608Metric_Pad1.08x0.95mm_HandSolder, F.Cu at (13.4, -42.9)
- added C1328: 1n, Capacitor_SMD:C_0603_1608Metric_Pad1.08x0.95mm_HandSolder, F.Cu at (13.4, -40.4)
- added C906: 22u, Capacitor_Tantalum_SMD:CP_EIA-7343-31_Kemet-D_Pad2.25x2.55mm_HandSolder, F.Cu at (135.5, -46.9)
- added C907: 150n, Capacitor_SMD:C_0603_1608Metric_Pad1.08x0.95mm_HandSolder, F.Cu at (9.04, -15.8)
- added C908: 220n, Capacitor_SMD:C_0603_1608Metric_Pad1.08x0.95mm_HandSolder, F.Cu at (9.04, -13.3)
- added C909: 220n, Capacitor_SMD:C_0603_1608Metric_Pad1.08x0.95mm_HandSolder, F.Cu at (9.04, -10.8)
- added C910: 220n, Capacitor_SMD:C_0603_1608Metric_Pad1.08x0.95mm_HandSolder, F.Cu at (9.04, -8.25)
- added C911: 100n, Capacitor_SMD:C_0603_1608Metric_Pad1.08x0.95mm_HandSolder, F.Cu at (9.04, -5.74)
- added C912: 220n, Capacitor_SMD:C_0603_1608Metric_Pad1.08x0.95mm_HandSolder, F.Cu at (9.04, -3.23)
- added C913: 100n, Capacitor_SMD:C_0603_1608Metric_Pad1.08x0.95mm_HandSolder, F.Cu at (9.04, -0.72)
- added C914: 100n, Capacitor_SMD:C_0603_1608Metric_Pad1.08x0.95mm_HandSolder, F.Cu at (9.04, 1.79)
- added C915: 1000p, Capacitor_SMD:C_0603_1608Metric_Pad1.08x0.95mm_HandSolder, F.Cu at (13.4, -15.8)
- added C916: 1000p, Capacitor_SMD:C_0603_1608Metric_Pad1.08x0.95mm_HandSolder, F.Cu at (13.4, -13.3)
- added C917: 10n, Capacitor_SMD:C_0603_1608Metric_Pad1.08x0.95mm_HandSolder, F.Cu at (13.4, -10.8)
- added D1001: BAV99, Package_TO_SOT_SMD:SOT-23, F.Cu at (54.6, -1.91)
- added D1002: BAV99, Package_TO_SOT_SMD:SOT-23, F.Cu at (54.6, 2.54)
- added D1302: SZ1SMB5918BT3G, Diode_SMD:D_SMB, F.Cu at (122.3, -60.2)
- added D1303: SZ1SMB5918BT3G, Diode_SMD:D_SMB, F.Cu at (122.3, -54.6)
- added D1304: SMCJ43CA, Diode_SMD:D_SMC, F.Cu at (138.9, -56.6)
- added D1306: 1N4148, Diode_SMD:D_SOD-123, F.Cu at (129.4, -61.3)
- added FB1001: KMZ1608SHR102ATD25, Inductor_SMD:L_0603_1608Metric_Pad1.05x0.95mm_HandSolder, F.Cu at (41.2, -10.8)
- added FB1002: KMZ1608SHR102ATD25, Inductor_SMD:L_0603_1608Metric_Pad1.05x0.95mm_HandSolder, F.Cu at (41.2, -8.25)
- added FB1003: KMZ1608SHR102ATD25, Inductor_SMD:L_0603_1608Metric_Pad1.05x0.95mm_HandSolder, F.Cu at (41.2, -5.74)
- added K1101: G6SU-2F-DC3, Relay_SMD:Relay_DPDT_Omron_G6SK-2F, F.Cu at (118.0, 91.8)
- added K1102: G6SU-2F-DC3, Relay_SMD:Relay_DPDT_Omron_G6SK-2F, F.Cu at (105.2, 91.7)
- added K1301: G6SU-2F-DC3, Relay_SMD:Relay_DPDT_Omron_G6SK-2F, F.Cu at (183.9, 48.8)
- added K1302: G6SU-2F-DC3, Relay_SMD:Relay_DPDT_Omron_G6SK-2F, F.Cu at (-82.8, 79.1)
- added K1303: G6SU-2F-DC3, Relay_SMD:Relay_DPDT_Omron_G6SK-2F, F.Cu at (-71.1, 79.1)
- added K1304: G6SU-2F-DC3, Relay_SMD:Relay_DPDT_Omron_G6SK-2F, F.Cu at (-59.3, 79.1)
- added L1101: 470n, Inductor_SMD:L_0603_1608Metric_Pad1.05x0.95mm_HandSolder, F.Cu at (61.8, -43.2)
- added L1102: 470n, Inductor_SMD:L_0603_1608Metric_Pad1.05x0.95mm_HandSolder, F.Cu at (49.9, -52.9)
- added L1103: 470n, Inductor_SMD:L_0603_1608Metric_Pad1.05x0.95mm_HandSolder, F.Cu at (49.9, -50.4)
- added L1104: 470n, Inductor_SMD:L_0603_1608Metric_Pad1.05x0.95mm_HandSolder, F.Cu at (49.9, -47.9)
- added L1105: 470n, Inductor_SMD:L_0603_1608Metric_Pad1.05x0.95mm_HandSolder, F.Cu at (49.9, -45.4)
- added L1106: 470n, Inductor_SMD:L_0603_1608Metric_Pad1.05x0.95mm_HandSolder, F.Cu at (49.9, -42.9)
- added L1107: 680n, Inductor_SMD:L_0603_1608Metric_Pad1.05x0.95mm_HandSolder, F.Cu at (49.9, -40.4)
- added L1108: 680n, Inductor_SMD:L_0603_1608Metric_Pad1.05x0.95mm_HandSolder, F.Cu at (54.3, -55.4)
- added L1109: 560n, Inductor_SMD:L_0603_1608Metric_Pad1.05x0.95mm_HandSolder, F.Cu at (54.3, -52.9)
- added L1110: 560n, Inductor_SMD:L_0603_1608Metric_Pad1.05x0.95mm_HandSolder, F.Cu at (54.3, -50.4)
- added L1111: 910n, Inductor_SMD:L_0603_1608Metric_Pad1.05x0.95mm_HandSolder, F.Cu at (54.3, -47.9)
- added L1112: 910n, Inductor_SMD:L_0603_1608Metric_Pad1.05x0.95mm_HandSolder, F.Cu at (54.3, -45.4)
- added L1113: 750n, Inductor_SMD:L_0603_1608Metric_Pad1.05x0.95mm_HandSolder, F.Cu at (54.3, -42.9)
- added L1114: 750n, Inductor_SMD:L_0603_1608Metric_Pad1.05x0.95mm_HandSolder, F.Cu at (54.3, -40.4)
- added L1115: 1u, Inductor_SMD:L_0603_1608Metric_Pad1.05x0.95mm_HandSolder, F.Cu at (58.6, -55.4)
- added L1116: 1u, Inductor_SMD:L_0603_1608Metric_Pad1.05x0.95mm_HandSolder, F.Cu at (58.6, -52.9)
- added L1117: 1u2, Inductor_SMD:L_0603_1608Metric_Pad1.05x0.95mm_HandSolder, F.Cu at (58.6, -50.4)
- added L1118: 100n, Inductor_SMD:L_0603_1608Metric_Pad1.05x0.95mm_HandSolder, F.Cu at (58.6, -47.9)
- added L1201: 1m, Inductor_SMD:L_0603_1608Metric_Pad1.05x0.95mm_HandSolder, F.Cu at (49.9, -35.9)
- added L1202: 82n, Inductor_SMD:L_0603_1608Metric_Pad1.05x0.95mm_HandSolder, F.Cu at (49.9, -33.4)
- added L1203: 82n, Inductor_SMD:L_0603_1608Metric_Pad1.05x0.95mm_HandSolder, F.Cu at (49.9, -30.8)
- added L1301: 1m, Inductor_SMD:L_0603_1608Metric_Pad1.05x0.95mm_HandSolder, F.Cu at (13.4, -37.9)
- added L1302: 180n, Inductor_SMD:L_0603_1608Metric_Pad1.05x0.95mm_HandSolder, F.Cu at (13.4, -35.4)
- added L1303: 47n, Inductor_SMD:L_0603_1608Metric_Pad1.05x0.95mm_HandSolder, F.Cu at (13.4, -32.8)
- added L1304: 47n, Inductor_SMD:L_0603_1608Metric_Pad1.05x0.95mm_HandSolder, F.Cu at (13.4, -30.3)
- added Q1101: MMBT5087LT1G, Package_TO_SOT_SMD:SOT-23, F.Cu at (113.7, -48.7)
- added Q1201: MMBF4416A, Package_TO_SOT_SMD:SOT-23, F.Cu at (103.4, -68.5)
- added Q1202: MMBFJ175LT1, Package_TO_SOT_SMD:SOT-23, F.Cu at (103.4, -64.0)
- added Q1203: MMBT5087LT1G, Package_TO_SOT_SMD:SOT-23, F.Cu at (103.4, -59.6)
- added Q1204: MMBT6429LT1, Package_TO_SOT_SMD:SOT-23, F.Cu at (103.4, -55.1)
- added R1001: 10k, Resistor_SMD:R_0603_1608Metric_Pad0.98x0.95mm_HandSolder, F.Cu at (41.2, -3.23)
- added R1002: 10k, Resistor_SMD:R_0603_1608Metric_Pad0.98x0.95mm_HandSolder, F.Cu at (41.2, -0.72)
- added R1003: 10k, Resistor_SMD:R_0603_1608Metric_Pad0.98x0.95mm_HandSolder, F.Cu at (45.6, -15.8)
- added R1004: 10k, Resistor_SMD:R_0603_1608Metric_Pad0.98x0.95mm_HandSolder, F.Cu at (45.6, -13.3)
- added R1005: 10k, Resistor_SMD:R_0603_1608Metric_Pad0.98x0.95mm_HandSolder, F.Cu at (45.6, -10.8)
- added R1006: 10k, Resistor_SMD:R_0603_1608Metric_Pad0.98x0.95mm_HandSolder, F.Cu at (45.6, -8.25)
- added R1007: 10k, Resistor_SMD:R_0603_1608Metric_Pad0.98x0.95mm_HandSolder, F.Cu at (45.6, -5.74)
- added R1008: 6k81, Resistor_SMD:R_0603_1608Metric_Pad0.98x0.95mm_HandSolder, F.Cu at (45.6, -3.23)
- added R1009: 237k, Resistor_SMD:R_0603_1608Metric_Pad0.98x0.95mm_HandSolder, F.Cu at (45.6, -0.72)
- added R1010: 6k81, Resistor_SMD:R_0603_1608Metric_Pad0.98x0.95mm_HandSolder, F.Cu at (49.9, -15.8)
- added R1011: 6k81, Resistor_SMD:R_0603_1608Metric_Pad0.98x0.95mm_HandSolder, F.Cu at (49.9, -13.3)
- added R1012: 619, Resistor_SMD:R_0603_1608Metric_Pad0.98x0.95mm_HandSolder, F.Cu at (49.9, -10.8)
- added R1013: 10k, Resistor_SMD:R_0603_1608Metric_Pad0.98x0.95mm_HandSolder, F.Cu at (49.9, -8.25)
- added R1014: 1k, Resistor_SMD:R_0603_1608Metric_Pad0.98x0.95mm_HandSolder, F.Cu at (49.9, -5.74)
- added R1301: 21k5, Resistor_SMD:R_0603_1608Metric_Pad0.98x0.95mm_HandSolder, F.Cu at (13.4, -27.8)
- added R1302: 21k5, Resistor_SMD:R_0603_1608Metric_Pad0.98x0.95mm_HandSolder, F.Cu at (13.4, -25.3)
- added R1303: 10k, Resistor_SMD:R_0603_1608Metric_Pad0.98x0.95mm_HandSolder, F.Cu at (13.4, -22.8)
- added R1304: 100k, Resistor_SMD:R_0603_1608Metric_Pad0.98x0.95mm_HandSolder, F.Cu at (13.4, -20.3)
- added R1305: 12k4, Resistor_SMD:R_0603_1608Metric_Pad0.98x0.95mm_HandSolder, F.Cu at (17.7, -55.4)
- added R1306: 34R8, Resistor_SMD:R_0603_1608Metric_Pad0.98x0.95mm_HandSolder, F.Cu at (17.7, -52.9)
- added R1307: 100k, Resistor_SMD:R_0603_1608Metric_Pad0.98x0.95mm_HandSolder, F.Cu at (17.7, -50.4)
- added R1308: 1k, Resistor_SMD:R_0603_1608Metric_Pad0.98x0.95mm_HandSolder, F.Cu at (17.7, -47.9)
- added R1309: 34R8, Resistor_SMD:R_0603_1608Metric_Pad0.98x0.95mm_HandSolder, F.Cu at (17.7, -45.4)
- added R1310: 383, Resistor_SMD:R_0603_1608Metric_Pad0.98x0.95mm_HandSolder, F.Cu at (17.7, -42.9)
- added R1311: 383, Resistor_SMD:R_0603_1608Metric_Pad0.98x0.95mm_HandSolder, F.Cu at (17.7, -40.4)
- added R1312: 287, Resistor_SMD:R_0603_1608Metric_Pad0.98x0.95mm_HandSolder, F.Cu at (17.7, -37.9)
- added R1313: 287, Resistor_SMD:R_0603_1608Metric_Pad0.98x0.95mm_HandSolder, F.Cu at (17.7, -35.4)
- added R1314: 383, Resistor_SMD:R_0603_1608Metric_Pad0.98x0.95mm_HandSolder, F.Cu at (17.7, -32.8)
- added R1315: 383, Resistor_SMD:R_0603_1608Metric_Pad0.98x0.95mm_HandSolder, F.Cu at (17.7, -30.3)
- added R1316: 45k3, Resistor_SMD:R_0603_1608Metric_Pad0.98x0.95mm_HandSolder, F.Cu at (17.7, -27.8)
- added R1317: 10, Resistor_SMD:R_0603_1608Metric_Pad0.98x0.95mm_HandSolder, F.Cu at (17.7, -25.3)
- added R1318: 10, Resistor_SMD:R_0603_1608Metric_Pad0.98x0.95mm_HandSolder, F.Cu at (17.7, -22.8)
- added R1319: 10k, Resistor_SMD:R_0603_1608Metric_Pad0.98x0.95mm_HandSolder, F.Cu at (17.7, -20.3)
- added R1320: 10, Resistor_SMD:R_0603_1608Metric_Pad0.98x0.95mm_HandSolder, F.Cu at (22.1, -55.4)
- added R1321: 10, Resistor_SMD:R_0603_1608Metric_Pad0.98x0.95mm_HandSolder, F.Cu at (22.1, -52.9)
- added R1322: 31R6, Resistor_SMD:R_0603_1608Metric_Pad0.98x0.95mm_HandSolder, F.Cu at (22.1, -50.4)
- added R1323: 383, Resistor_SMD:R_0603_1608Metric_Pad0.98x0.95mm_HandSolder, F.Cu at (22.1, -47.9)
- added R1324: 383, Resistor_SMD:R_0603_1608Metric_Pad0.98x0.95mm_HandSolder, F.Cu at (22.1, -45.4)
- added R1325: 162, Resistor_SMD:R_0603_1608Metric_Pad0.98x0.95mm_HandSolder, F.Cu at (22.1, -42.9)
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Connections:
- net /Connector/SIGNAL renamed /Connector/MAIN_OUTPUT
- C1303 pad 1: -15V_WFD3 -> +15V_WFD3
- C1304 pad 1: +15V_WFD3 -> GNDA
- C1304 pad 2: GNDA -> /Output/SET_SIN_ARB
- C203 pad 1: Net-(U202-PH0,EVENTOUT,OSC_IN) -> +3.3V
- C205 pad 1: Net-(U202-PH1,EVENTOUT,OSC_OUT) -> +3.3V
- C206 pad 1: Net-(U202-VCAP_1) -> +3.3V
- C208 pad 1: Net-(U202-VCAP_2) -> +3.3V
- C209 pad 1: +3.3V -> Net-(U201-PH0)
- C211 pad 1: +3.3V -> Net-(U201-PH1)
- C213 pad 1: +3.3V -> /MCU/NRST
- C215 pad 1: +3.3V -> Net-(C215-Pad1)
- C217 pad 1: +3.3V -> Net-(C217-Pad1)
- C219 pad 1: +3.3V -> VDDA
- C220 pad 1: +3.3V -> VDDA
- C221 pad 1: /MCU/MCU_VDDA -> GNDA
- C221 pad 2: GNDA -> +3.3V
- C222 pad 1: /MCU/NRST -> GNDA
- C222 pad 2: GNDA -> +3.3V
- C903 pad 1: Net-(U902-AVDD) -> Net-(U901C-V+)
- C904 pad 1: Net-(U901C-V+) -> Net-(U901C-V-)
- C905 pad 1: Net-(U901C-V-) -> Net-(U903-AVDD)
- FB201 pad 1: /MCU/MCU_VDDA -> VDDA
- FB903 pad 2: Net-(U902-AVDD) -> Net-(U903-AVDD)
- R201 pad 1: /MCU/LED_BLUE -> /MCU/MCU_DEFAULT
- R201 pad 2: Net-(D201-K) -> +3.3V
- R202 pad 1: /MCU/MCU_DEFAULT -> /MCU/LED_BLUE
- R202 pad 2: +3.3V -> Net-(D201-K)
- R204 pad 1: +3.3V -> /MCU/LED_GREEN
- R204 pad 2: /MCU/SENS_SCL -> Net-(D203-K)
- R205 pad 1: /MCU/LED_GREEN -> +3.3V
- R205 pad 2: Net-(D203-K) -> /MCU/NRST
- R206 pad 1: +3.3V -> GNDA
- R206 pad 2: /MCU/SENS_SDA -> Net-(U201-BOOT0)
- R207 pad 2: /MCU/EEPROM_SDA -> /MCU/I2C1_SCL
- R208 pad 2: /MCU/EEPROM_SCL -> /MCU/I2C1_SDA
- R209 pad 1: Net-(U202-BOOT0) -> +3.3V
- R209 pad 2: GNDA -> /MCU/I2C1_SDA
- R210 pad 2: /MCU/NRST -> /MCU/I2C1_SCL
- R817 pad 2: /MCU/EEPROM_SCL -> /MCU/I2C2_SCL
- R818 pad 2: /MCU/EEPROM_SDA -> /MCU/I2C2_SDA
- U201 pad 1: /MCU/SENS_SDA -> unconnected-(U201-PE2-Pad1)
- U201 pad 2: GNDA -> unconnected-(U201-PE3-Pad2)
- U201 pad 5: +3.3V -> unconnected-(U201-PE6-Pad5)
- U201 pad 6: /MCU/SENS_SCL -> +3.3V
- U202 pad 1: unconnected-(U202-PE2,TRACECLK,SPI4_SCK,SAI1_MCLK_A,QUADSPI_BK1_IO2,ETH_MII_TXD3,FMC_A23,EVENTOUT-Pad1) -> GNDA
- U202 pad 2: unconnected-(U202-PE3,TRACED0,SAI1_SD_B,FMC_A19,EVENTOUT-Pad2) -> GNDA
- U202 pad 3: unconnected-(U202-PE4,TRACED1,SPI4_NSS,SAI1_FS_A,DFSDM1_DATIN3,FMC_A20,DCMI_D4,LCD_B0,EVENTOUT-Pad3) -> GNDA
- U202 pad 4: unconnected-(U202-PE5,TRACED2,TIM9_CH1,SPI4_MISO,SAI1_SCK_A,DFSDM1_CKIN3,FMC_A21,DCMI_D6,LCD_G0,EVENTOUT-Pad4) -> GNDA
- U202 pad 5: unconnected-(U202-PE6,TRACED3,TIM1_BKIN2,TIM9_CH2,SPI4_MOSI,SAI1_SD_A,SAI2_MCLK_B,FMC_A22,DCMI_D7,LCD_G1,EVENTOUT-Pad5) -> /MCU/I2C1_SDA
- U202 pad 6: +3.3V -> /MCU/I2C1_SCL
- U202 pad 7: unconnected-(U202-PC13,EVENTOUT,RTC_TAMP2,RTC_TS,WKUP5-Pad7) -> /MCU/EEPROM_WP
- U202 pad 8: unconnected-(U202-PC14,EVENTOUT,OSC32_IN-Pad8) -> +3.3V
- U203 pad 1: GNDA -> /MCU/I2C1_SDA
- U203 pad 3: GNDA -> unconnected-(U203-NC-Pad3)
- U203 pad 4: GNDA -> unconnected-(U203-NC-Pad4)
- U203 pad 5: /MCU/EEPROM_SDA -> +3.3V
- U203 pad 6: /MCU/EEPROM_SCL -> /MCU/I2C1_SCL
- U203 pad 7: /MCU/EEPROM_WP -> unconnected-(U203-DAP-Pad7)
- U803 pad 13: /MCU/EEPROM_SCL -> /MCU/I2C2_SCL
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
Commit message: PCB design
Parts:
- removed C1165, C1166, C1178: 47p, Capacitor_SMD:C_0603_1608Metric_Pad1.08x0.95mm_HandSolder
- removed C1167, C1168: 22u, Capacitor_Tantalum_SMD:CP_EIA-7343-31_Kemet-D_Pad2.25x2.55mm_HandSolder
- removed C1169, C912: 220n, Capacitor_SMD:C_0603_1608Metric_Pad1.08x0.95mm_HandSolder
- removed C1170, C1171: 22p, Capacitor_SMD:C_0603_1608Metric_Pad1.08x0.95mm_HandSolder
- removed C1172, C1176, C1177: 10p, Capacitor_SMD:C_0603_1608Metric_Pad1.08x0.95mm_HandSolder
- removed C1173, C1175: 100p, Capacitor_SMD:C_0603_1608Metric_Pad1.08x0.95mm_HandSolder
- removed C1174: 1p, Capacitor_SMD:C_0603_1608Metric_Pad1.08x0.95mm_HandSolder
- removed C1179: 15p, Capacitor_SMD:C_0603_1608Metric_Pad1.08x0.95mm_HandSolder
- removed C1180: 33p, Capacitor_SMD:C_0603_1608Metric_Pad1.08x0.95mm_HandSolder
- removed C1181: 150p, Capacitor_SMD:C_0603_1608Metric_Pad1.08x0.95mm_HandSolder
- removed C808, C913, C914: 100n, Capacitor_SMD:C_0603_1608Metric_Pad1.08x0.95mm_HandSolder
- removed C809: 1u, Capacitor_SMD:C_0603_1608Metric_Pad1.08x0.95mm_HandSolder
- removed C915, C916: 1000p, Capacitor_SMD:C_0603_1608Metric_Pad1.08x0.95mm_HandSolder
- removed C917: 10n, Capacitor_SMD:C_0603_1608Metric_Pad1.08x0.95mm_HandSolder
- removed FB1101, FB1102, FB1103, FB1104, FB1105, FB1106, FB1107, FB1108, FB901, FB902, FB903: KMZ1608SHR102ATD25, Inductor_SMD:L_0603_1608Metric_Pad1.05x0.95mm_HandSolder
- added FL1301: ACP3225-102-2P-T000, ETH1CFGEN1:ACP3225, F.Cu at (188.5, 51.4)
- added J701: Conn_02x05_Odd_Even, Connector_PinHeader_2.54mm:PinHeader_2x05_P2.54mm_Vertical, F.Cu at (147.7, 80.1)
- added K1305: TX2SA-4.5V, Relay_SMD:Relay_DPDT_Omron_G6S-2F, F.Cu at (178.3, 47.5)
- added X701: ASFL1-100.000MHZ-L-T, Crystal:Crystal_SMD_5032-4Pin_5.0x3.2mm, B.Cu at (144.5, 101.6)
- C1001, C1006, C1008, C1009, C1013, C1143, C1301, C1304, C1305, C1306, C1307, C1308, C1309, C1310, C1311, C1312, C1313, C1314, C1315, C1316, C1317, C1318, C1319, C1322, C1323, C1324, C1325, C1326, C1327, C1328, C301, C302, C304, C305, C306, C308, C309, C310, C312, C313, C314, C401, C402, C403, C404, C405, C406, C407, C408, C501, C601, C604, C607, C608, C609, C610, C611, C612, C613, C614, C615, C616, C617, C618, C619, C620, C621, C622, C629, C630, C631, C632, C633, C634, C635, C636, C637, C638, C639, C640, C641, C642, C703, C706, C708, C710, C713, C715, C801, C802, C803, C804, C806, C807, C905, D1001, D1002, D1101, D1301, D1305, D1306, D601, D602, D606, D607, FB301, Q1101, Q1301, R1001, R1002, R1003, R1004, R1005, R1006, R1007, R1008, R1009, R1010, R1011, R1013, R1014, R1102, R1105, R1106, R1107, R1108, R1111, R1112, R1114, R1117, R1118, R1123, R1126, R1127, R1134, R1301, R1302, R1305, R1306, R1307, R1308, R1309, R1310, R1311, R1312, R1313, R1314, R1315, R1316, R1317, R1318, R1319, R1321, R1322, R1323, R1324, R1326, R1327, R1330, R1331, R1332, R1333, R1334, R1335, R1336, R1337, R1338, R1339, R1340, R1341, R1342, R1343, R1344, R1345, R1346, R1347, R1361, R1362, R1366, R1367, R1370, R1372, R1373, R1375, R1376, R1378, R304, R305, R306, R307, R308, R311, R312, R313, R314, R315, R316, R317, R318, R319, R320, R321, R401, R402, R403, R405, R602, R609, R613, R616, R617, R621, R803, R804, R808, R814, R901, R904, R905, R910, R912, R916, R917, U202, U704, X1101, Y201: moved to B.Cu
- C1105, C1106: value 100n -> 100p; moved to B.Cu
- C1107, C1108: value 10u -> 33p; footprint Capacitor_SMD:C_1206_3216Metric_Pad1.33x1.80mm_HandSolder -> Capacitor_SMD:C_0603_1608Metric_Pad1.08x0.95mm_HandSolder
- C1109: value 22u -> 30p; footprint Capacitor_Tantalum_SMD:CP_EIA-7343-31_Kemet-D_Pad2.25x2.55mm_HandSolder -> Capacitor_SMD:C_0603_1608Metric_Pad1.08x0.95mm_HandSolder
- C1110: value 100p -> 30p
- C1111: value 100p -> 33p; moved to B.Cu
- C1112, C1144: value 100n -> 33p; moved to B.Cu
- C1113, C1114, C1118, C1142: value 33p -> 56p
- C1115, C1116: value 30p -> 3p3
- C1117, C1141: value 100n -> 56p
- C1119: value 33p -> 120p
- C1120: value 56p -> 120p
- C1121, C1132, C1133: value 56p -> 33p; moved to B.Cu
- C1122: value 3p3 -> 33p; moved to B.Cu
- C1123: value 3p3 -> 56p
- C1124: value 10u -> 56p; footprint Capacitor_SMD:C_1206_3216Metric_Pad1.33x1.80mm_HandSolder -> Capacitor_SMD:C_0603_1608Metric_Pad1.08x0.95mm_HandSolder
- C1125: value 10u -> 150p; footprint Capacitor_SMD:C_1206_3216Metric_Pad1.33x1.80mm_HandSolder -> Capacitor_SMD:C_0603_1608Metric_Pad1.08x0.95mm_HandSolder
- C1126: value 56p -> 150p
- C1127: value 56p -> 62p
- C1128: value 120p -> 62p
- C1129: value 120p -> 8p2
- C1130: value 33p -> 8p2
- C1131: value 33p -> 100n; moved to B.Cu
- C1134, C1135: value 150p -> 130p
- C1136, C1137: value 62p -> 330p
- C1138: value 8p2 -> 100n; moved to B.Cu
- C1139: value 8p2 -> 15p
- C1140: value 100n -> 15p
- C1145: value 130p -> 220n; moved to B.Cu
- C1146: value 130p -> 100p
- C1147: value 330p -> 100p
- C1148: value 330p -> 5p6
- C1149: value 100n -> 5p6
- C1150, C1151: value 15p -> 47p
- C1152: value 56p -> 220n; moved to B.Cu
- C1153: value 56p -> 22p
- C1154: value 10u -> 22p; footprint Capacitor_SMD:C_1206_3216Metric_Pad1.33x1.80mm_HandSolder -> Capacitor_SMD:C_0603_1608Metric_Pad1.08x0.95mm_HandSolder
- C1155: value 10u -> 10p; footprint Capacitor_SMD:C_1206_3216Metric_Pad1.33x1.80mm_HandSolder -> Capacitor_SMD:C_0603_1608Metric_Pad1.08x0.95mm_HandSolder
- C1156: value 33p -> 100p; moved to B.Cu
- C1157: value 33p -> 1p
- C1158: value 220n -> 100p; moved to B.Cu
- C1159, C1160: value 100p -> 10p
- C1161: value 5p6 -> 47p
- C1162: value 5p6 -> 15p
- C1163: value 100n -> 33p
- C1164: value 100n -> 150p
- C805: value 100n -> 1u; moved to B.Cu
- C901: value 100n -> 150n; moved to B.Cu
- C902: value 100n -> 220n; moved to B.Cu
- C903, C904: value 10u -> 220n; footprint Capacitor_SMD:C_1206_3216Metric_Pad1.33x1.80mm_HandSolder -> Capacitor_SMD:C_0603_1608Metric_Pad1.08x0.95mm_HandSolder; moved to B.Cu
- C906: value 22u -> 220n; footprint Capacitor_Tantalum_SMD:CP_EIA-7343-31_Kemet-D_Pad2.25x2.55mm_HandSolder -> Capacitor_SMD:C_0603_1608Metric_Pad1.08x0.95mm_HandSolder; moved to B.Cu
- C907: value 150n -> 100n; moved to B.Cu
- C908: value 220n -> 100n
- C909, C910: value 220n -> 1000p; moved to B.Cu
- C911: value 100n -> 10n; moved to B.Cu
- L1101, L1102, L1103, L1104, L1105, L1106, L1107, L1108, L1109, L1110, L1111, L1112, L1113, L1114, L1115, L1116, L1117, L1118, L1201, L1202, L1203, L1301, L1303, L1304: footprint Inductor_SMD:L_0603_1608Metric_Pad1.05x0.95mm_HandSolder -> Inductor_SMD:L_0805_2012Metric_Pad1.15x1.40mm_HandSolder
- L1302: footprint Inductor_SMD:L_0603_1608Metric_Pad1.05x0.95mm_HandSolder -> Inductor_SMD:L_0805_2012Metric_Pad1.15x1.40mm_HandSolder; moved to B.Cu
- U201: footprint Package_QFP:LQFP-144_20x20mm_P0.5mm -> ETH1CFGEN1:TQFP-144_20x20mm_P0.5mm
- moved D605 300.0 mm to (213.7, 113.7), turned to 90 degrees
- moved D604 298.1 mm to (216.4, 109.5), turned to -90 degrees
- moved R605 293.7 mm to (213.1, 127.8), turned to 90 degrees
- moved R610 292.9 mm to (216.4, 114.4), turned to 90 degrees
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Connections:
- C1103 pad 1: +3V3_WFD2 -> Net-(C1103-Pad1)
- C1104 pad 1: +3V3_WFD2 -> Net-(C1104-Pad1)
- C1105 pad 1: +3V3_WFD1 -> /WaveformDAC/SET_ARB_FLTR1
- C1106 pad 1: Net-(C1106-Pad1) -> GNDA
- C1106 pad 2: GNDA -> /WaveformDAC/SET_SIN_FLTR1
- C1108 pad 1: +3V3_WFD2 -> GNDA
- C1108 pad 2: GNDA -> Net-(C1108-Pad2)
- C1109 pad 1: +3V3_WFD1 -> Net-(C1109-Pad1)
- C1110 pad 1: /WaveformDAC/SET_ARB_FLTR1 -> GNDA
- C1110 pad 2: GNDA -> Net-(C1110-Pad2)
- C1111 pad 1: GNDA -> Net-(C1107-Pad1)
- C1111 pad 2: /WaveformDAC/SET_SIN_FLTR1 -> Net-(C1111-Pad2)
- C1112 pad 1: +15V_WFD2 -> Net-(C1108-Pad2)
- C1112 pad 2: GNDA -> Net-(C1112-Pad2)
- C1113 pad 1: Net-(C1113-Pad1) -> Net-(C1111-Pad2)
- C1114 pad 2: Net-(C1114-Pad2) -> Net-(C1112-Pad2)
- C1115 pad 1: Net-(C1115-Pad1) -> Net-(C1109-Pad1)
- C1116 pad 2: Net-(C1116-Pad2) -> Net-(C1110-Pad2)
- C1117 pad 1: +15V_WFD1 -> Net-(C1111-Pad2)
- C1118 pad 1: Net-(C1113-Pad1) -> GNDA
- C1118 pad 2: Net-(C1118-Pad2) -> Net-(C1112-Pad2)
- C1119 pad 1: Net-(C1114-Pad2) -> Net-(C1119-Pad1)
- C1119 pad 2: Net-(C1119-Pad2) -> GNDA
- C1120 pad 1: Net-(C1118-Pad2) -> GNDA
- C1120 pad 2: GNDA -> Net-(C1120-Pad2)
- C1121 pad 1: GNDA -> Net-(C1111-Pad2)
- C1121 pad 2: Net-(C1119-Pad2) -> Net-(C1121-Pad2)
- C1122 pad 1: Net-(C1115-Pad1) -> Net-(C1112-Pad2)
- C1122 pad 2: GNDA -> Net-(C1122-Pad2)
- C1123 pad 1: GNDA -> Net-(C1121-Pad2)
- C1123 pad 2: Net-(C1116-Pad2) -> GNDA
- C1124 pad 1: +15V_WFD2 -> GNDA
- C1124 pad 2: GNDA -> Net-(C1122-Pad2)
- C1125 pad 1: +15V_WFD1 -> Net-(C1125-Pad1)
- C1126 pad 1: Net-(C1118-Pad2) -> GNDA
- C1126 pad 2: GNDA -> Net-(C1126-Pad2)
- C1127 pad 1: GNDA -> Net-(C1121-Pad2)
- C1127 pad 2: Net-(C1119-Pad2) -> GNDA
- C1128 pad 1: Net-(C1128-Pad1) -> GNDA
- C1128 pad 2: GNDA -> Net-(C1122-Pad2)
- C1129 pad 1: GNDA -> Net-(C1125-Pad1)
- C1129 pad 2: Net-(C1129-Pad2) -> GNDA
- C1130 pad 1: Net-(C1118-Pad2) -> GNDA
- C1130 pad 2: Net-(C1130-Pad2) -> Net-(C1126-Pad2)
- C1131 pad 1: Net-(C1119-Pad2) -> /WaveformDAC/V_DTY_CYCL
- C1131 pad 2: Net-(C1131-Pad2) -> GNDA
- C1132 pad 1: Net-(C1130-Pad2) -> Net-(C1121-Pad2)
- C1132 pad 2: GNDA -> Net-(C1132-Pad2)
- C1133 pad 1: GNDA -> Net-(C1122-Pad2)
- C1133 pad 2: Net-(C1131-Pad2) -> Net-(C1133-Pad2)
- C1134 pad 1: Net-(C1134-Pad1) -> Net-(C1132-Pad2)
- C1135 pad 2: Net-(C1135-Pad2) -> Net-(C1133-Pad2)
- C1136 pad 1: Net-(C1130-Pad2) -> Net-(C1136-Pad1)
- C1137 pad 2: Net-(C1131-Pad2) -> Net-(C1137-Pad2)
- C1138 pad 1: Net-(C1134-Pad1) -> /WaveformDAC/V_DTY_CYCL
- C1138 pad 2: GNDA -> Net-(C1138-Pad2)
- C1139 pad 1: GNDA -> Net-(C1132-Pad2)
- C1139 pad 2: Net-(C1135-Pad2) -> GNDA
- C1140 pad 1: /WaveformDAC/V_DTY_CYCL -> GNDA
- C1140 pad 2: GNDA -> Net-(C1133-Pad2)
- C1141 pad 1: -15V_WFD2 -> Net-(C1136-Pad1)
- C1142 pad 1: Net-(C1130-Pad2) -> GNDA
- C1142 pad 2: Net-(C1142-Pad2) -> Net-(C1137-Pad2)
- C1143 pad 1: Net-(C1131-Pad2) -> Net-(C1132-Pad2)
- C1144 pad 1: -15V_WFD1 -> Net-(C1133-Pad2)
- C1144 pad 2: GNDA -> Net-(C1144-Pad2)
- C1145 pad 1: Net-(C1142-Pad2) -> Net-(U1101A-+)
- C1146 pad 1: GNDA -> Net-(C1143-Pad2)
- C1146 pad 2: Net-(C1143-Pad2) -> GNDA
- C1147 pad 1: Net-(C1147-Pad1) -> GNDA
- C1147 pad 2: GNDA -> Net-(C1144-Pad2)
- C1148 pad 1: GNDA -> Net-(C1143-Pad2)
- C1148 pad 2: Net-(C1148-Pad2) -> GNDA
- C1149 pad 1: /WaveformDAC/V_DTY_CYCL -> GNDA
- C1149 pad 2: Net-(C1149-Pad2) -> Net-(C1144-Pad2)
- C1150 pad 1: Net-(C1142-Pad2) -> Net-(C1150-Pad1)
- C1151 pad 2: Net-(C1143-Pad2) -> Net-(C1151-Pad2)
- C1152 pad 1: Net-(C1147-Pad1) -> Net-(C1152-Pad1)
- C1153 pad 1: GNDA -> Net-(C1150-Pad1)
- C1153 pad 2: Net-(C1148-Pad2) -> GNDA
- C1154 pad 1: -15V_WFD2 -> GNDA
- C1154 pad 2: GNDA -> Net-(C1151-Pad2)
- C1155 pad 1: -15V_WFD1 -> Net-(U1103-+)
- C1155 pad 2: GNDA -> Net-(U1103--)
- C1156 pad 1: Net-(C1142-Pad2) -> /WaveformDAC/SET_ARB_FLTR2
- C1156 pad 2: Net-(C1156-Pad2) -> GNDA
- C1157 pad 1: Net-(C1143-Pad2) -> Net-(U1103--)
- C1158 pad 1: Net-(U1101A-+) -> GNDA
- C1158 pad 2: GNDA -> /WaveformDAC/SET_SIN_FLTR2
- C1159 pad 1: Net-(C1156-Pad2) -> GNDA
- C1159 pad 2: GNDA -> Net-(C1159-Pad2)
- C1160 pad 1: GNDA -> Net-(C1160-Pad1)
- C1160 pad 2: Net-(C1157-Pad2) -> GNDA
- C1161 pad 1: Net-(C1156-Pad2) -> Net-(U1103-+)
- C1162 pad 1: GNDA -> Net-(C1162-Pad1)
- C1162 pad 2: Net-(C1157-Pad2) -> GNDA
- C1163 pad 1: +5V_WFD -> Net-(C1163-Pad1)
- C1164 pad 1: -5V_WFD -> /WaveformDAC/SINE_ARB
- C1321 pad 1: /Output/MAIN_OUTPUT -> /Connector/MAIN_OUTPUT
- C805 pad 2: +15V -> +5V
- C806 pad 2: -15V -> +3.3V
- C807 pad 2: +5V -> Net-(U803-DECAP)
- C901 pad 1: Net-(U901C-V+) -> GNDA
- C901 pad 2: GNDA -> Net-(U903-VREF)
- C902 pad 1: Net-(U901C-V-) -> /DAC/V_PEDGE
- C903 pad 1: Net-(U901C-V+) -> /DAC/V_NEDGE
- C904 pad 1: Net-(U901C-V-) -> Net-(U902A-+)
- C905 pad 1: Net-(U903-AVDD) -> Net-(C905-Pad1)
- C905 pad 2: GNDA -> /DAC/V_AMPL
- C906 pad 1: Net-(U903-AVDD) -> Net-(U901A-+)
- C907 pad 1: GNDA -> Net-(U901B-+)
- C907 pad 2: Net-(U903-VREF) -> GNDA
- C908 pad 1: /DAC/V_PEDGE -> Net-(C908-Pad1)
- C909 pad 1: /DAC/V_NEDGE -> Net-(U901A--)
- C909 pad 2: GNDA -> /DAC/V_NULL_SINE
- C910 pad 1: Net-(U902A-+) -> Net-(U902A--)
- C910 pad 2: GNDA -> /DAC/V_NULL_SQ
- C911 pad 1: Net-(C911-Pad1) -> /DAC/V_OFFSET
- C911 pad 2: /DAC/V_AMPL -> GNDA
- D1101 pad 2: +3V3_WFD1 -> +3.3V
- D1304 pad 2: /Output/MAIN_OUTPUT -> /Connector/MAIN_OUTPUT
- D902 pad 2: Net-(C914-Pad1) -> Net-(C908-Pad1)
- D902 pad 4: Net-(C914-Pad1) -> Net-(C908-Pad1)
- K1101 pad 10: Net-(C1116-Pad2) -> Net-(C1110-Pad2)
- K1101 pad 3: Net-(C1115-Pad1) -> Net-(C1109-Pad1)
- K1101 pad 5: Net-(C1113-Pad1) -> Net-(C1107-Pad1)
- K1101 pad 8: Net-(C1114-Pad2) -> Net-(C1108-Pad2)
- K1102 pad 10: Net-(C1157-Pad2) -> Net-(C1144-Pad2)
- K1102 pad 3: Net-(C1156-Pad2) -> Net-(C1143-Pad2)
- K1102 pad 4: Net-(C1176-Pad2) -> Net-(C1159-Pad2)
- K1102 pad 5: Net-(C1147-Pad1) -> Net-(C1136-Pad1)
- K1102 pad 8: Net-(C1148-Pad2) -> Net-(C1137-Pad2)
- K1102 pad 9: Net-(C1177-Pad1) -> Net-(C1160-Pad1)
- K501 pad 3: Net-(U501-O6) -> Net-(U501-O1)
- K502 pad 3: Net-(U501-O5) -> Net-(U501-O2)
- K505 pad 3: Net-(U501-O2) -> Net-(U501-O5)
- K506 pad 3: Net-(U501-O1) -> Net-(U501-O6)
- L1101 pad 1: Net-(C1113-Pad1) -> Net-(C1107-Pad1)
- L1101 pad 2: Net-(C1118-Pad2) -> Net-(C1111-Pad2)
- L1102 pad 1: Net-(C1114-Pad2) -> Net-(C1108-Pad2)
- L1102 pad 2: Net-(C1119-Pad2) -> Net-(C1112-Pad2)
- L1103 pad 1: Net-(C1115-Pad1) -> Net-(C1109-Pad1)
- L1103 pad 2: Net-(C1128-Pad1) -> Net-(C1119-Pad1)
- L1104 pad 1: Net-(C1116-Pad2) -> Net-(C1110-Pad2)
- L1104 pad 2: Net-(C1129-Pad2) -> Net-(C1120-Pad2)
- L1105 pad 1: Net-(C1118-Pad2) -> Net-(C1111-Pad2)
- L1105 pad 2: Net-(C1130-Pad2) -> Net-(C1121-Pad2)
- L1106 pad 1: Net-(C1119-Pad2) -> Net-(C1112-Pad2)
- L1106 pad 2: Net-(C1131-Pad2) -> Net-(C1122-Pad2)
- L1107 pad 1: Net-(C1128-Pad1) -> Net-(C1119-Pad1)
- L1107 pad 2: Net-(C1134-Pad1) -> Net-(C1125-Pad1)
- L1108 pad 1: Net-(C1129-Pad2) -> Net-(C1120-Pad2)
- L1108 pad 2: Net-(C1135-Pad2) -> Net-(C1126-Pad2)
- L1109 pad 1: Net-(C1130-Pad2) -> Net-(C1121-Pad2)
- L1109 pad 2: Net-(C1142-Pad2) -> Net-(C1132-Pad2)
- L1110 pad 1: Net-(C1131-Pad2) -> Net-(C1122-Pad2)
- L1110 pad 2: Net-(C1143-Pad2) -> Net-(C1133-Pad2)
- L1111 pad 1: Net-(C1134-Pad1) -> Net-(C1125-Pad1)
- L1111 pad 2: Net-(C1147-Pad1) -> Net-(C1136-Pad1)
- L1112 pad 1: Net-(C1135-Pad2) -> Net-(C1126-Pad2)
- L1112 pad 2: Net-(C1148-Pad2) -> Net-(C1137-Pad2)
- L1113 pad 1: Net-(C1142-Pad2) -> Net-(C1132-Pad2)
- L1113 pad 2: Net-(C1156-Pad2) -> Net-(C1143-Pad2)
- L1114 pad 1: Net-(C1143-Pad2) -> Net-(C1133-Pad2)
- L1114 pad 2: Net-(C1157-Pad2) -> Net-(C1144-Pad2)
- L1115 pad 1: Net-(C1165-Pad1) -> Net-(C1150-Pad1)
- L1116 pad 2: Net-(C1166-Pad2) -> Net-(C1151-Pad2)
- L1117 pad 2: Net-(C1179-Pad1) -> Net-(C1162-Pad1)
- L1118 pad 1: Net-(C1180-Pad1) -> Net-(C1163-Pad1)
- L1304 pad 2: /Output/MAIN_OUTPUT -> /Connector/MAIN_OUTPUT
- Q1101 pad 3: -15V_WFD1 -> -15V
- R1107 pad 2: +3V3_WFD2 -> +3.3V
- R1109 pad 2: Net-(C1106-Pad1) -> Net-(C1103-Pad1)
- R1110 pad 1: Net-(C1106-Pad1) -> Net-(C1103-Pad1)
- R1110 pad 2: Net-(C1107-Pad1) -> Net-(C1104-Pad1)
- R1111 pad 1: Net-(C1107-Pad1) -> Net-(C1104-Pad1)
- R1112 pad 2: +15V_WFD1 -> +15V
- R1113 pad 2: Net-(C1106-Pad1) -> Net-(C1103-Pad1)
- R1115 pad 1: Net-(C1147-Pad1) -> Net-(C1136-Pad1)
- R1116 pad 2: Net-(C1148-Pad2) -> Net-(C1137-Pad2)
- R1118 pad 1: Net-(C1147-Pad1) -> Net-(C1136-Pad1)
- R1118 pad 2: Net-(C1148-Pad2) -> Net-(C1137-Pad2)
- R1119 pad 1: Net-(C1156-Pad2) -> Net-(C1143-Pad2)
- R1119 pad 2: Net-(C1165-Pad1) -> Net-(C1150-Pad1)
- R1120 pad 1: Net-(C1165-Pad1) -> Net-(C1150-Pad1)
- R1121 pad 2: Net-(C1166-Pad2) -> Net-(C1151-Pad2)
- R1122 pad 1: Net-(C1166-Pad2) -> Net-(C1151-Pad2)
- R1122 pad 2: Net-(C1157-Pad2) -> Net-(C1144-Pad2)
- R1123 pad 2: Net-(C1149-Pad2) -> Net-(C1138-Pad2)
- R1124 pad 1: Net-(C1149-Pad2) -> Net-(C1138-Pad2)
- R1124 pad 2: Net-(C1169-Pad1) -> Net-(C1152-Pad1)
- R1125 pad 1: Net-(C1169-Pad1) -> Net-(C1152-Pad1)
- R1126 pad 1: Net-(C1156-Pad2) -> Net-(C1143-Pad2)
- R1126 pad 2: Net-(C1157-Pad2) -> Net-(C1144-Pad2)
- R1128 pad 1: Net-(U1103-~{Q}) -> Net-(C1157-Pad2)
- R1129 pad 1: Net-(C1176-Pad2) -> Net-(C1159-Pad2)
- R1130 pad 1: Net-(C1177-Pad1) -> Net-(C1160-Pad1)
- R1136 pad 2: Net-(C1180-Pad1) -> Net-(C1163-Pad1)
- R1137 pad 2: Net-(C1179-Pad1) -> Net-(C1162-Pad1)
- R906 pad 2: Net-(C911-Pad1) -> Net-(C905-Pad1)
- R907 pad 2: Net-(C914-Pad1) -> Net-(C908-Pad1)
- R908 pad 1: Net-(C911-Pad1) -> Net-(C905-Pad1)
- R913 pad 1: Net-(C914-Pad1) -> Net-(C908-Pad1)
- U1101 pad 1: Net-(C1149-Pad2) -> Net-(C1138-Pad2)
- U1101 pad 4: -15V_WFD1 -> -15V
- U1101 pad 8: +15V_WFD1 -> +15V
- U1102 pad 24: +3V3_WFD1 -> +3.3V
- U1102 pad 27: +3V3_WFD2 -> +3.3V
- U1103 pad 1: +5V_WFD -> +5V
- U1103 pad 4: -5V_WFD -> -5V
- U1104 pad 4: -15V_WFD2 -> -15V
- U1104 pad 7: +15V_WFD2 -> +15V
- U1104 pad 9: -15V_WFD2 -> -15V
- U901 pad 4: Net-(U901C-V-) -> -15V
- U901 pad 8: Net-(U901C-V+) -> +15V
- U902 pad 4: Net-(U901C-V-) -> -15V
- U902 pad 8: Net-(U901C-V+) -> +15V
- U903 pad 3: Net-(U903-AVDD) -> +3.3V
Other:
- copper layers 4 -> 6

Commit message: PCB design
Parts:
- C1214, C1216, C1219, C1220, C1223, C1224, C1225, C409, R1203, R1206, R1208, R1209, R1216, R1220, R1222, R1223, R1229, R406: moved to B.Cu
- C706, C713: moved to F.Cu
- moved C409 196.7 mm to (211.2, 87.0), turned to 180 degrees
- moved R406 188.7 mm to (207.9, 87.0), turned to 180 degrees
- moved U1207 158.9 mm to (125.1, 53.5)
- moved C1227 156.6 mm to (133.5, 55.2), turned to 90 degrees
- moved C1225 148.7 mm to (123.1, 58.0), turned to 180 degrees
- moved C1226 148.0 mm to (123.1, 58.0), turned to 180 degrees
- moved U1203 146.9 mm to (108.2, 65.8)
- moved U1201 145.2 mm to (108.1, 46.4)
- moved U1205 143.1 mm to (108.2, 53.1)
- moved U1206 143.1 mm to (108.2, 59.4)
- moved R1232 142.0 mm to (133.5, 51.8), turned to -90 degrees
- moved C1219 139.3 mm to (113.9, 51.6), turned to 90 degrees
- moved C1220 138.7 mm to (110.5, 65.8), turned to -90 degrees
- moved R1235 138.7 mm to (130.9, 55.2), turned to -90 degrees
- moved C1218 138.6 mm to (113.9, 45.0), turned to 90 degrees
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
Commit message: PCB design
Parts:
- removed C1202, C1206: 22u, Capacitor_Tantalum_SMD:CP_EIA-7343-31_Kemet-D_Pad2.25x2.55mm_HandSolder
- removed FB1001, FB1002, FB1003, FB1201, FB1202, FB1203, FB1301, FB1302: KMZ1608SHR102ATD25, Inductor_SMD:L_0603_1608Metric_Pad1.05x0.95mm_HandSolder
- added C1014: 100n, Capacitor_SMD:C_0603_1608Metric_Pad1.08x0.95mm_HandSolder, B.Cu at (132.3, 75.6)
- added C643: 22u/35V, Capacitor_Tantalum_SMD:CP_EIA-7343-31_Kemet-D_Pad2.25x2.55mm_HandSolder, F.Cu at (85.3, 106.0)
- added C644: 22u/35V, Capacitor_Tantalum_SMD:CP_EIA-7343-31_Kemet-D_Pad2.25x2.55mm_HandSolder, F.Cu at (85.3, 122.4)
- added C645: 22u/35V, Capacitor_Tantalum_SMD:CP_EIA-7343-31_Kemet-D_Pad2.25x2.55mm_HandSolder, F.Cu at (119.1, 106.0)
- added C646: 22u/35V, Capacitor_Tantalum_SMD:CP_EIA-7343-31_Kemet-D_Pad2.25x2.55mm_HandSolder, F.Cu at (119.1, 122.3)
- added C912: 150n, Capacitor_SMD:C_0603_1608Metric_Pad1.08x0.95mm_HandSolder, B.Cu at (129.5, 83.2)
- added C913: 100n, Capacitor_SMD:C_0603_1608Metric_Pad1.08x0.95mm_HandSolder, B.Cu at (116.3, 77.3)
- added C914: 100n, Capacitor_SMD:C_0603_1608Metric_Pad1.08x0.95mm_HandSolder, B.Cu at (111.8, 83.3)
- added C915: 100n, Capacitor_SMD:C_0603_1608Metric_Pad1.08x0.95mm_HandSolder, B.Cu at (116.7, 73.2)
- added C916: 100n, Capacitor_SMD:C_0603_1608Metric_Pad1.08x0.95mm_HandSolder, B.Cu at (111.8, 76.5)
- C1002: value 22u -> 100n; footprint Capacitor_Tantalum_SMD:CP_EIA-7343-31_Kemet-D_Pad2.25x2.55mm_HandSolder -> Capacitor_SMD:C_0603_1608Metric_Pad1.08x0.95mm_HandSolder; moved to B.Cu
- C1003, C1007: value 10u -> 100n; footprint Capacitor_SMD:C_1206_3216Metric_Pad1.33x1.80mm_HandSolder -> Capacitor_SMD:C_0603_1608Metric_Pad1.08x0.95mm_HandSolder; moved to B.Cu
- C1159, C1161, C1201, C1203, C1204, C1205, C1207, C1210, C1211, C1212, C1213, C201, C202, C203, C204, C205, C206, C207, C208, C209, C210, C211, C212, C213, C214, C215, C216, C217, C218, C219, C220, C221, C222, C701, C702, C704, C705, C707, C709, C711, C712, C714, C716, C717, C718, C719, C720, C721, C722, C723, C724, C725, C726, C727, C728, C729, FB201, R1101, R1103, R1104, R1131, R205, R206, R209, R210, R701, R702, R703, R704, R705, R706, R707, R708, R709: moved to B.Cu
- R1305: moved to F.Cu
- moved FB201 179.8 mm to (177.2, 101.6), turned to 90 degrees
- moved C206 176.6 mm to (180.8, 86.6), turned to -90 degrees
- moved C207 176.5 mm to (180.8, 91.4), turned to -90 degrees
- moved C208 176.4 mm to (180.8, 96.4), turned to -90 degrees
- moved C210 173.0 mm to (180.8, 101.2), turned to 90 degrees
- moved R201 170.9 mm to (184.0, 88.0), turned to 90 degrees
- moved C203 170.1 mm to (174.5, 83.7)
- moved C215 169.6 mm to (178.2, 86.6), turned to -90 degrees
- moved C219 167.6 mm to (178.9, 107.4)
- moved C209 166.7 mm to (171.1, 98.8)
- moved C211 166.1 mm to (174.4, 98.8), turned to 180 degrees
- moved C221 165.9 mm to (178.7, 76.3)
- moved C205 165.2 mm to (169.4, 83.7)
- moved C202 165.1 mm to (168.4, 105.0), turned to 180 degrees
- moved R207 164.6 mm to (181.9, 76.1), turned to 90 degrees
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Connections:
- C1002 pad 1: +5V_ADC -> +15V
- C1003 pad 1: +15V_ADC -> -15V
- C1007 pad 1: -15V_ADC -> +15V
- C1012 pad 1: +5V_ADC -> +5V
- C1201 pad 1: Net-(U1204-+Vl) -> +5V
- C1203 pad 1: Net-(U1204--Vs) -> -5V
- C1204 pad 1: Net-(U1204-+VS) -> +5V
- C1205 pad 1: +5V_WFD -> +5V
- C1207 pad 1: +5V_WFD -> +5V
- C1210 pad 1: +5V_WFD -> +5V
- C1211 pad 1: -5V_WFD -> -5V
- C1212 pad 1: -5V_WFD -> -5V
- C1213 pad 1: -5V_WFD -> -5V
- C1302 pad 1: -15V_WFD3 -> -15V
- C1303 pad 1: +15V_WFD3 -> +15V
- D1001 pad 1: +15V_ADC -> +15V
- D1001 pad 3: +15V_ADC -> +15V
- D1002 pad 2: -15V_ADC -> -15V
- D1002 pad 3: -15V_ADC -> -15V
- R1002 pad 1: +5V_ADC -> +5V
- R1013 pad 1: +5V_ADC -> +5V
- R1365 pad 1: -15V_WFD3 -> -15V
- R1366 pad 1: +15V_WFD3 -> +15V
- U1001 pad 4: -15V_ADC -> -15V
- U1001 pad 8: +15V_ADC -> +15V
- U1002 pad 4: -15V_ADC -> -15V
- U1002 pad 8: +15V_ADC -> +15V
- U1004 pad 8: +5V_ADC -> +5V
- U1201 pad 4: -15V_WFD1 -> -15V
- U1201 pad 8: +15V_WFD1 -> +15V
- U1202 pad 4: -15V_WFD1 -> -15V
- U1202 pad 8: +15V_WFD1 -> +15V
- U1203 pad 4: -15V_WFD1 -> -15V
- U1203 pad 8: +15V_WFD1 -> +15V
- U1204 pad 1: Net-(U1204--Vs) -> -5V
- U1204 pad 16: Net-(U1204-+VS) -> +5V
- U1204 pad 3: Net-(U1204-+Vl) -> +5V
- U1205 pad 4: +5V_WFD -> +5V
- U1205 pad 5: -5V_WFD -> -5V
- U1206 pad 4: -5V_WFD -> -5V
- U1206 pad 7: +5V_WFD -> +5V
- U1207 pad 4: -5V_WFD -> -5V
- U1207 pad 7: +5V_WFD -> +5V
- U1301 pad 4: -15V_WFD3 -> -15V
- U1301 pad 8: +15V_WFD3 -> +15V
- U1302 pad 12: -15V_WFD3 -> -15V
- U1302 pad 3: +15V_WFD3 -> +15V
- U1303 pad 4: -15V_WFD3 -> -15V
- U1303 pad 8: +15V_WFD3 -> +15V
