File: hardware/ETH1CFGEN1/Ethernet.kicad_sch (KiCad schematic)
At the start: 43 parts, among them U201 LAN8742, U202 LC03-3.3BTG, U203 LC03-3.3BTG, Y201 NX5032GA-25.000000MHZ-LN-CD-1

Commit message: PCB design
Changed lines of the file:
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@@
       (effects (font (size 1.27 1.27)) hide)
     )
-    (property "Value" "GNDD" (at 31.115 83.82 0)
+    (property "Value" "GNDD" (at 29.21 83.82 90)
       (effects (font (size 1.27 1.27)))
     )

Commit message: PCB design
Parts:
- U201: footprint Package_DFN_QFN:QFN-24-1EP_4x4mm_P0.5mm_EP2.6x2.6mm -> Package_DFN_QFN:QFN-24-1EP_4x4mm_P0.5mm_EP2.6x2.6mm_ThermalVias
Changed lines of the file:
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@@
       (effects (font (size 1.27 1.27)) (justify right))
     )
-    (property "Footprint" "Package_DFN_QFN:QFN-24-1EP_4x4mm_P0.5mm_EP2.6x2.6mm" (at 87.63 113.03 0)
+    (property "Footprint" "Package_DFN_QFN:QFN-24-1EP_4x4mm_P0.5mm_EP2.6x2.6mm_ThermalVias" (at 87.63 113.03 0)
       (effects (font (size 1.27 1.27)) (justify left) hide)
     )
