File: hardware/ETH1CFGEN1/ADC.kicad_sch (KiCad schematic)
At the start: 27 parts, among them U701 TL072CD, U702 TL072CD, U703 DG408DY, U704 ADS7818EB

Commit message: Development
Parts:
- added C1003, C1007: 10u, Capacitor_SMD:C_1206_3216Metric_Pad1.33x1.80mm_HandSolder, symbol Device:C
- added C309: 22u, Capacitor_Tantalum_SMD:CP_EIA-7343-31_Kemet-D_Pad2.25x2.55mm_HandSolder, symbol Device:C_Polarized
- added C707: 100n, Capacitor_SMD:C_0603_1608Metric_Pad1.08x0.95mm_HandSolder, symbol Device:C
- added D1001, D1002: BAV99, Package_TO_SOT_SMD:SOT-23, symbol Diode:BAV99
- added FB303 (x3): KMZ1608SHR102ATD25, Inductor_SMD:L_0603_1608Metric_Pad1.05x0.95mm_HandSolder, symbol Device:FerriteBead_Small
- C701, C702, C703, C704, C705, C706, C707, C709: footprint (none) -> Capacitor_SMD:C_0603_1608Metric_Pad1.08x0.95mm_HandSolder
- C708: footprint (none) -> Capacitor_SMD:C_1206_3216Metric_Pad1.33x1.80mm_HandSolder
- R1013, R1014, R701, R702, R703, R704, R705, R706, R707, R708, R709, R710, R711, R?: footprint (none) -> Resistor_SMD:R_0603_1608Metric_Pad0.98x0.95mm_HandSolder
- U701, U702: footprint (none) -> Package_SO:SOIC-8_3.9x4.9mm_P1.27mm
- U703: value DG408DY -> DG408DY-T1-E3; footprint (none) -> Package_SO:SOIC-16_3.9x9.9mm_P1.27mm
- U704: footprint (none) -> Package_SO:TSSOP-8_3x3mm_P0.65mm
Connections:
- net GNDA: now also C1003.2, C1007.2, C309.2, C707.2
- net +5V_ADC: now reaches R1013.1, U704.8 (VDD)
- net +5V_ADC: now also R?.1, C309.1, C707.1, FB303.2
- net MSEL0: now reaches U703.1 (A0)
- net MEAS_BUF: now reaches U703.12 (S4)
- net at U703.13 (V+): now also D1001.2 (A)
- net MSEL2: now reaches U703.15 (A2)
- net MSEL1: now reaches U703.16 (A1)
- net at U703.3 (V-): now also D1002.1 (K)
- net MEAS_OUT: now reaches U703.5 (S1)
- net MEAS_MOD_DAC: now reaches U703.6 (S2)
- net MEAS_AMPL: now reaches U703.7 (S3)
- net -15V_ADC: now reaches U701.4 (V-)
- net -15V_ADC: now also U702.4 (V-), C1007.1, D1002.2 (A), D1002.3 (K), FB303.2
- net +15V_ADC: now reaches U701.8 (V+)
- net +15V_ADC: now also U702.8 (V+), C1003.1, D1001.1 (K), D1001.3 (K), FB303.2
- new net +15V: FB303.1
- new net +5V: FB303.1
- new net -15V: FB303.1
Other:
- moved on the sheet: C701, C702, C703, C704, C705, C706, C707, C708, C709, R1013, R1014, R701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

Commit message: PCB design
Changed lines of the file:
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@@
     (stroke (width 0) (type default))
   )
-  (wire (pts (xy 215.9 78.105) (xy 220.345 78.105))
+  (wire (pts (xy 215.9 73.025) (xy 220.345 73.025))
     (stroke (width 0) (type default))
   )
@@
     (stroke (width 0) (type default))
   )
-  (wire (pts (xy 215.9 113.665) (xy 215.9 78.105))
+  (wire (pts (xy 215.9 73.025) (xy 215.9 113.665))
     (stroke (width 0) (type default))
   )
@@
     (stroke (width 0) (type default))
   )
-  (wire (pts (xy 220.345 78.105) (xy 220.345 73.025))
-    (stroke (width 0) (type default))
-  )

Commit message: PCB design
Parts:
- removed C1003, C1007: 10u, Capacitor_SMD:C_1206_3216Metric_Pad1.33x1.80mm_HandSolder, symbol Device:C
- removed C309: 22u, Capacitor_Tantalum_SMD:CP_EIA-7343-31_Kemet-D_Pad2.25x2.55mm_HandSolder, symbol Device:C_Polarized
- removed FB303 (x3): KMZ1608SHR102ATD25, Inductor_SMD:L_0603_1608Metric_Pad1.05x0.95mm_HandSolder, symbol Device:FerriteBead_Small
- added C707 (x4): 100n, Capacitor_SMD:C_0603_1608Metric_Pad1.08x0.95mm_HandSolder, symbol Device:C
Connections:
- net +15V_ADC is gone; now on net +15V: D1001.1 (K), D1001.3 (K), U701.8 (V+), U702.8 (V+)
- net +5V_ADC is gone; now on net +5V: C707.1, R1013.1, R?.1, U704.8 (VDD)
- net -15V_ADC is gone; now on net -15V: D1002.2 (A), D1002.3 (K), U701.4 (V-), U702.4 (V-)
- net +15V: now also C707.1, C707.1
- net -15V: now also C707.1, C707.1
- net GNDA: now also C707.2, C707.2, C707.2, C707.2
Other:
- moved on the sheet: U702C

Commit message: PCB design
Parts:
- C705: value 1000p -> 1n
- C707: value 4700p -> 4n7
Changed lines of the file:
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@@
   (symbol (lib_id "Device:C") (at 203.2 67.945 0) (unit 1)
     (in_bom yes) (on_board yes) (dnp no) (fields_autoplaced)
-    (property "Reference" "C707" (at 206.375 66.675 0)
-      (effects (font (size 1.27 1.27)) (justify left))
-    )
-    (property "Value" "4700p" (at 206.375 69.215 0)
+    (property "Reference" "C707" (at 207.01 66.675 0)
+      (effects (font (size 1.27 1.27)) (justify left))
+    )
+    (property "Value" "4n7" (at 207.01 69.215 0)
       (effects (font (size 1.27 1.27)) (justify left))
     )
@@
     )
   )
+  (symbol (lib_id "power:PWR_FLAG") (at 102.235 185.42 180) (unit 1)
+    (in_bom yes) (on_board yes) (dnp no)
+    (property "Reference" "#FLG01001" (at 102.235 187.325 0)
+      (effects (font (size 1.27 1.27)) hide)
+    )
+    (property "Value" "PWR_FLAG" (at 102.235 189.23 0)
+      (effects (font (size 1.27 1.27)))
+    )
+    (property "Footprint" "" (at 102.235 185.42 0)
+      (effects (font (size 1.27 1.27)) hide)
+    )
+    (property "Datasheet" "~" (at 102.235 185.42 0)
+      (effects (font (size 1.27 1.27)) hide)
+    )
+    (pin "1")
+    (instances
+      (project "ETH1CFGEN1"
+        (path "/44bc1157-6d68-4ab3-afc0-b8d9f089cc50/d6e8baa1-1cb1-436f-aba5-7e42524c9d57"
+          (reference "#FLG01001") (unit 1)
+        )
+      )
+    )
+  )
   (symbol (lib_id "Device:C") (at 215.9 118.745 0) (unit 1)
     (in_bom yes) (on_board yes) (dnp no) (fields_autoplaced)
@@
         (path "/44bc1157-6d68-4ab3-afc0-b8d9f089cc50/d6e8baa1-1cb1-436f-aba5-7e42524c9d57"
           (reference "D1002") (unit 1)
+        )
+      )
+    )
+  )
+  (symbol (lib_id "power:+2V5") (at 102.235 185.42 0) (unit 1)
+    (in_bom yes) (on_board yes) (dnp no)
+    (property "Reference" "#PWR0711" (at 102.235 189.23 0)
+      (effects (font (size 1.27 1.27)) hide)
+    )
+    (property "Value" "+2V5" (at 102.235 180.975 0)
+      (effects (font (size 1.27 1.27)))
+    )
+    (property "Footprint" "" (at 102.235 185.42 0)
+      (effects (font (size 1.27 1.27)) hide)
+    )
+    (property "Datasheet" "" (at 102.235 185.42 0)
+      (effects (font (size 1.27 1.27)) hide)
+    )
+    (pin "1")
+    (instances
+      (project "ETH1CFGEN1B"
+        (path "/3dceb0a1-97ad-435d-a235-e3839b959163/f742b0a0-f239-4818-b7fd-6c1a7dccca2f"
+          (reference "#PWR0711") (unit 1)
+        )
+      )
+      (project "ETH1CFGEN1"
+        (path "/44bc1157-6d68-4ab3-afc0-b8d9f089cc50/d6e8baa1-1cb1-436f-aba5-7e42524c9d57"
+          (reference "#PWR01017") (unit 1)
         )
       )
@@
     )
   )
+  (symbol (lib_id "power:-2V5") (at 116.84 185.42 0) (unit 1)
+    (in_bom yes) (on_board yes) (dnp no) (fields_autoplaced)
+    (property "Reference" "#PWR0712" (at 116.84 182.88 0)
+      (effects (font (size 1.27 1.27)) hide)
+    )
+    (property "Value" "-2V5" (at 116.84 180.975 0)
+      (effects (font (size 1.27 1.27)))
+    )
+    (property "Footprint" "" (at 116.84 185.42 0)
+      (effects (font (size 1.27 1.27)) hide)
+    )
+    (property "Datasheet" "" (at 116.84 185.42 0)
+      (effects (font (size 1.27 1.27)) hide)
+    )
+    (pin "1")
+    (instances
+      (project "ETH1CFGEN1B"
+        (path "/3dceb0a1-97ad-435d-a235-e3839b959163/f742b0a0-f239-4818-b7fd-6c1a7dccca2f"
+          (reference "#PWR0712") (unit 1)
+        )
+      )
+      (project "ETH1CFGEN1"
+        (path "/44bc1157-6d68-4ab3-afc0-b8d9f089cc50/d6e8baa1-1cb1-436f-aba5-7e42524c9d57"
+          (reference "#PWR01020") (unit 1)
+        )
+      )
+    )
+  )
   (symbol (lib_id "Device:C") (at 118.745 69.85 0) (unit 1)
     (in_bom yes) (on_board yes) (dnp no)
@@
       (effects (font (size 1.27 1.27)) (justify left))
     )
-    (property "Value" "1000p" (at 159.385 60.96 0)
+    (property "Value" "1n" (at 159.385 60.96 0)
       (effects (font (size 1.27 1.27)) (justify left))
     )
@@
         )
       )
+    )
+  )
+  (symbol (lib_id "power:PWR_FLAG") (at 116.84 185.42 180) (unit 1)
+    (in_bom yes) (on_board yes) (dnp no)
+    (property "Reference" "#FLG01002" (at 116.84 187.325 0)
+      (effects (font (size 1.27 1.27)) hide)
+    )
+    (property "Value" "PWR_FLAG" (at 116.84 189.23 0)
+      (effects (font (size 1.27 1.27)))
+    )
+    (property "Footprint" "" (at 116.84 185.42 0)
+      (effects (font (size 1.27 1.27)) hide)
+    )
+    (property "Datasheet" "~" (at 116.84 185.42 0)
+      (effects (font (size 1.27 1.27)) hide)
+    )
+    (pin "1")
+    (instances
+      (project "ETH1CFGEN1"
+        (path "/44bc1157-6d68-4ab3-afc0-b8d9f089cc50/d6e8baa1-1cb1-436f-aba5-7e42524c9d57"
+          (reference "#FLG01002") (unit 1)
+        )
+      )
