File: hardware/ETH1CFGEN1/Connector.kicad_sch (KiCad schematic)
At the start: 9 parts, among them J301 C64AC, K301 HE3621A0510, K302 HE3621A0510, K303 HE3621A0510, K304 HE3621A0510, K305 HE3621A0510, K306 HE3621A0510, U301 ULN2003AIPWR

Commit message: Development
Connections:
- net SIGNAL renamed MAIN_OUTPUT
Changed lines of the file:
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@@
 (kicad_sch (version 20230121) (generator eeschema)
   (paper "A4")
+  (title_block
+    (date "2023-07-12")
+    (rev "1.1")
+  )
   (junction (at 132.715 39.37) (diameter 0) (color 0 0 0 0)
   )
@@
     (effects (font (size 1.27 1.27)) (justify left))
   )
+  (hierarchical_label "MAIN_OUTPUT" (shape input) (at 40.005 30.48 180) (fields_autoplaced)
+    (effects (font (size 1.27 1.27)) (justify right))
+  )
   (hierarchical_label "RX-" (shape bidirectional) (at 81.915 125.73 180) (fields_autoplaced)
     (effects (font (size 1.27 1.27)) (justify right))
   )
-  (hierarchical_label "SIGNAL" (shape bidirectional) (at 40.005 30.48 180) (fields_autoplaced)
-    (effects (font (size 1.27 1.27)) (justify right))
-  )

Commit message: PCB design
Connections:
- net at K306.3: now also U301.16 (O1); no longer U301.11 (O6)
- net at K301.3: now also U301.11 (O6); no longer U301.16 (O1)
- net at K305.3: now also U301.15 (O2); no longer U301.12 (O5)
- net at K302.3: now also U301.12 (O5); no longer U301.15 (O2)
Other:
- moved on the sheet: K301B, K302B, K305B, K306B
Changed lines of the file:
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@@
     (effects (font (size 1.27 1.27)) (justify left))
   )
-  (symbol (lib_id "ETH1CFGEN1:HE3621A0510") (at 113.665 44.45 0) (unit 2)
-    (in_bom yes) (on_board yes) (dnp no)
-    (property "Reference" "K306" (at 115.6462 43.2816 0)
-      (effects (font (size 1.27 1.27)) (justify left))
-    )
-    (property "Value" "HE3621A0510" (at 115.6462 45.593 0)
-      (effects (font (size 1.27 1.27)) (justify left))
-    )
-    (property "Footprint" "ETH1CFGEN1:HE360_x-5050462-8" (at 120.015 45.72 0)
-      (effects (font (size 1.27 1.27)) hide)
-    )
-    (property "Datasheet" "" (at 120.015 45.72 0)
+  (symbol (lib_id "ETH1CFGEN1:HE3621A0510") (at 203.835 44.45 0) (unit 2)
+    (in_bom yes) (on_board yes) (dnp no)
+    (property "Reference" "K306" (at 205.8162 43.2816 0)
+      (effects (font (size 1.27 1.27)) (justify left))
+    )
+    (property "Value" "HE3621A0510" (at 205.8162 45.593 0)
+      (effects (font (size 1.27 1.27)) (justify left))
+    )
+    (property "Footprint" "ETH1CFGEN1:HE360_x-5050462-8" (at 210.185 45.72 0)
+      (effects (font (size 1.27 1.27)) hide)
+    )
+    (property "Datasheet" "" (at 210.185 45.72 0)
       (effects (font (size 1.27 1.27)) hide)
     )
@@
     )
   )
-  (symbol (lib_id "ETH1CFGEN1:HE3621A0510") (at 203.835 44.45 0) (unit 2)
-    (in_bom yes) (on_board yes) (dnp no)
-    (property "Reference" "K301" (at 205.8162 43.2816 0)
-      (effects (font (size 1.27 1.27)) (justify left))
-    )
-    (property "Value" "HE3621A0510" (at 205.8162 45.593 0)
-      (effects (font (size 1.27 1.27)) (justify left))
-    )
-    (property "Footprint" "ETH1CFGEN1:HE360_x-5050462-8" (at 210.185 45.72 0)
-      (effects (font (size 1.27 1.27)) hide)
-    )
-    (property "Datasheet" "" (at 210.185 45.72 0)
+  (symbol (lib_id "ETH1CFGEN1:HE3621A0510") (at 113.665 44.45 0) (unit 2)
+    (in_bom yes) (on_board yes) (dnp no)
+    (property "Reference" "K301" (at 115.6462 43.2816 0)
+      (effects (font (size 1.27 1.27)) (justify left))
+    )
+    (property "Value" "HE3621A0510" (at 115.6462 45.593 0)
+      (effects (font (size 1.27 1.27)) (justify left))
+    )
+    (property "Footprint" "ETH1CFGEN1:HE360_x-5050462-8" (at 120.015 45.72 0)
+      (effects (font (size 1.27 1.27)) hide)
+    )
+    (property "Datasheet" "" (at 120.015 45.72 0)
       (effects (font (size 1.27 1.27)) hide)
     )
@@
     )
   )
-  (symbol (lib_id "ETH1CFGEN1:HE3621A0510") (at 132.715 44.45 0) (unit 2)
-    (in_bom yes) (on_board yes) (dnp no)
-    (property "Reference" "K305" (at 134.6962 43.2816 0)
-      (effects (font (size 1.27 1.27)) (justify left))
-    )
-    (property "Value" "HE3621A0510" (at 134.6962 45.593 0)
-      (effects (font (size 1.27 1.27)) (justify left))
-    )
-    (property "Footprint" "ETH1CFGEN1:HE360_x-5050462-8" (at 139.065 45.72 0)
-      (effects (font (size 1.27 1.27)) hide)
-    )
-    (property "Datasheet" "" (at 139.065 45.72 0)
+  (symbol (lib_id "ETH1CFGEN1:HE3621A0510") (at 186.055 44.45 0) (unit 2)
+    (in_bom yes) (on_board yes) (dnp no)
+    (property "Reference" "K305" (at 188.0362 43.2816 0)
+      (effects (font (size 1.27 1.27)) (justify left))
+    )
+    (property "Value" "HE3621A0510" (at 188.0362 45.593 0)
+      (effects (font (size 1.27 1.27)) (justify left))
+    )
+    (property "Footprint" "ETH1CFGEN1:HE360_x-5050462-8" (at 192.405 45.72 0)
+      (effects (font (size 1.27 1.27)) hide)
+    )
+    (property "Datasheet" "" (at 192.405 45.72 0)
       (effects (font (size 1.27 1.27)) hide)
     )
@@
     )
   )
-  (symbol (lib_id "ETH1CFGEN1:HE3621A0510") (at 186.055 44.45 0) (unit 2)
-    (in_bom yes) (on_board yes) (dnp no)
-    (property "Reference" "K302" (at 188.0362 43.2816 0)
-      (effects (font (size 1.27 1.27)) (justify left))
-    )
-    (property "Value" "HE3621A0510" (at 188.0362 45.593 0)
-      (effects (font (size 1.27 1.27)) (justify left))
-    )
-    (property "Footprint" "ETH1CFGEN1:HE360_x-5050462-8" (at 192.405 45.72 0)
-      (effects (font (size 1.27 1.27)) hide)
-    )
-    (property "Datasheet" "" (at 192.405 45.72 0)
-      (effects (font (size 1.27 1.27)) hide)
-    )
+  (symbol (lib_id "ETH1CFGEN1:HE3621A0510") (at 132.715 44.45 0) (unit 2)
+    (in_bom yes) (on_board yes) (dnp no)
+    (property "Reference" "K302" (at 134.6962 43.2816 0)
+      (effects (font (size 1.27 1.27)) (justify left))
+    )
+    (property "Value" "HE3621A0510" (at 134.6962 45.593 0)
+      (effects (font (size 1.27 1.27)) (justify left))
+    )
+    (property "Footprint" "ETH1CFGEN1:HE360_x-5050462-8" (at 139.065 45.72 0)
+      (effects (font (size 1.27 1.27)) hide)
+    )
+    (property "Datasheet" "" (at 139.065 45.72 0)
+      (effects (font (size 1.27 1.27)) hide)
+    )

Commit message: PCB design
Connections:
- net at K304.3: now also U301.14 (O3); no longer U301.13 (O4)
- net at K303.3: now also U301.13 (O4); no longer U301.14 (O3)
Other:
- moved on the sheet: K303B, K304B
Changed lines of the file:
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@@
     )
   )
-  (symbol (lib_id "ETH1CFGEN1:HE3621A0510") (at 150.495 44.45 0) (unit 2)
-    (in_bom yes) (on_board yes) (dnp no)
-    (property "Reference" "K304" (at 152.4762 43.2816 0)
-      (effects (font (size 1.27 1.27)) (justify left))
-    )
-    (property "Value" "HE3621A0510" (at 152.4762 45.593 0)
-      (effects (font (size 1.27 1.27)) (justify left))
-    )
-    (property "Footprint" "ETH1CFGEN1:HE360_x-5050462-8" (at 156.845 45.72 0)
-      (effects (font (size 1.27 1.27)) hide)
-    )
-    (property "Datasheet" "" (at 156.845 45.72 0)
+  (symbol (lib_id "ETH1CFGEN1:HE3621A0510") (at 168.275 44.45 0) (unit 2)
+    (in_bom yes) (on_board yes) (dnp no)
+    (property "Reference" "K304" (at 170.2562 43.2816 0)
+      (effects (font (size 1.27 1.27)) (justify left))
+    )
+    (property "Value" "HE3621A0510" (at 170.2562 45.593 0)
+      (effects (font (size 1.27 1.27)) (justify left))
+    )
+    (property "Footprint" "ETH1CFGEN1:HE360_x-5050462-8" (at 174.625 45.72 0)
+      (effects (font (size 1.27 1.27)) hide)
+    )
+    (property "Datasheet" "" (at 174.625 45.72 0)
       (effects (font (size 1.27 1.27)) hide)
     )
@@
     )
   )
-  (symbol (lib_id "ETH1CFGEN1:HE3621A0510") (at 168.275 44.45 0) (unit 2)
-    (in_bom yes) (on_board yes) (dnp no)
-    (property "Reference" "K303" (at 170.2562 43.2816 0)
-      (effects (font (size 1.27 1.27)) (justify left))
-    )
-    (property "Value" "HE3621A0510" (at 170.2562 45.593 0)
-      (effects (font (size 1.27 1.27)) (justify left))
-    )
-    (property "Footprint" "ETH1CFGEN1:HE360_x-5050462-8" (at 174.625 45.72 0)
-      (effects (font (size 1.27 1.27)) hide)
-    )
-    (property "Datasheet" "" (at 174.625 45.72 0)
-      (effects (font (size 1.27 1.27)) hide)
-    )
+  (symbol (lib_id "ETH1CFGEN1:HE3621A0510") (at 150.495 44.45 0) (unit 2)
+    (in_bom yes) (on_board yes) (dnp no)
+    (property "Reference" "K303" (at 152.4762 43.2816 0)
+      (effects (font (size 1.27 1.27)) (justify left))
+    )
+    (property "Value" "HE3621A0510" (at 152.4762 45.593 0)
+      (effects (font (size 1.27 1.27)) (justify left))
+    )
+    (property "Footprint" "ETH1CFGEN1:HE360_x-5050462-8" (at 156.845 45.72 0)
+      (effects (font (size 1.27 1.27)) hide)
+    )
+    (property "Datasheet" "" (at 156.845 45.72 0)
+      (effects (font (size 1.27 1.27)) hide)
+    )
