File: hardware/ETH1CFGEN1/DAC.kicad_sch (KiCad schematic)
At the start: 42 parts, among them U601 TL072CD, U602 DAC8568IxPWR, U603 TL072CD

Commit message: Development
Parts:
- C309: footprint (none) -> Capacitor_Tantalum_SMD:CP_EIA-7343-31_Kemet-D_Pad2.25x2.55mm_HandSolder
- C607, C608, C609, C610, C611, C612, C613, C614, C615, C616, C617: footprint (none) -> Capacitor_SMD:C_0603_1608Metric_Pad1.08x0.95mm_HandSolder
- R601, R602, R603, R604, R605, R606, R607, R608, R609, R610, R611, R612, R613, R614, R615, R616, R617: footprint (none) -> Resistor_SMD:R_0603_1608Metric_Pad0.98x0.95mm_HandSolder
- U601, U603: footprint (none) -> Package_SO:SOIC-8_3.9x4.9mm_P1.27mm
- U602: value DAC8568IxPWR -> DAC8568IBPW; footprint (none) -> Package_SO:TSSOP-16_4.4x5mm_P0.65mm
Connections:
- net DAC_nLDAC: now reaches U602.1 (~{LDAC})
- net DAC_DIN: now reaches U602.15 (DIN)
- net DAC_SCLK: now reaches U602.16 (SCLK)
- net DAC_nSYNC: now reaches U602.2 (~{SYNC})
- net DAC_nCLR: now reaches U602.9 (~{CLR})
Other:
- moved on the sheet: C305, C309, C312, C320, C607, C608, C609, C610, C611, C612, C613, C614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

Commit message: PCB design
Parts:
- removed C305, C312 (x2): 100n, Capacitor_SMD:C_0603_1608Metric_Pad1.08x0.95mm_HandSolder, symbol Device:C
- removed C309: 22u, Capacitor_Tantalum_SMD:CP_EIA-7343-31_Kemet-D_Pad2.25x2.55mm_HandSolder, symbol Device:C_Polarized
- removed C320 (x2): 10u, Capacitor_SMD:C_1206_3216Metric_Pad1.33x1.80mm_HandSolder, symbol Device:C
- removed FB302, FB303 (x2): KMZ1608SHR102ATD25, Inductor_SMD:L_0603_1608Metric_Pad1.05x0.95mm_HandSolder, symbol Device:FerriteBead_Small
Connections:
- net +15V: now also U601.8 (V+), U603.8 (V+)
- net +3.3V: now also U602.3 (AVDD)
- net -15V: now also U601.4 (V-), U603.4 (V-)
Other:
- moved on the sheet: U601C, U603C

Commit message: PCB design
Parts:
- added C607: 150n, Capacitor_SMD:C_0603_1608Metric_Pad1.08x0.95mm_HandSolder, symbol Device:C
- added C707 (x4): 100n, Capacitor_SMD:C_0603_1608Metric_Pad1.08x0.95mm_HandSolder, symbol Device:C
Connections:
- net +15V: now also C707.1, C707.1
- net +3.3V: now also C607.2
- net -15V: now also C707.1, C707.1
- net GNDA: now also C607.1, C707.2, C707.2, C707.2, C707.2
Other:
- moved on the sheet: U603B, U603C

Commit message: PCB design
Parts:
- added C609: 220n, Capacitor_SMD:C_0603_1608Metric_Pad1.08x0.95mm_HandSolder, symbol Device:C
- added R603: 1k, Resistor_SMD:R_0603_1608Metric_Pad0.98x0.95mm_HandSolder, symbol Device:R
- added TP901: TestPoint, TestPoint:TestPoint_Pad_1.0x1.0mm, symbol Connector:TestPoint
- C615, C616: value 1000p -> 1n
Connections:
- net GNDA: now also C609.2
- net at U602.10 (VOUTH): now also R603.1
- new net: C609.1, R603.2, TP901.1
- no-connect marks 1 -> 0
Changed lines of the file:
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@@
   (junction (at 236.22 43.815) (diameter 0) (color 0 0 0 0)
   )
+  (junction (at 153.67 126.365) (diameter 0) (color 0 0 0 0)
+  )
   (junction (at 198.12 65.405) (diameter 0) (color 0 0 0 0)
   )
@@
   (junction (at 228.6 102.235) (diameter 0) (color 0 0 0 0)
   )
-  (no_connect (at 123.825 80.645))
   (wire (pts (xy 185.42 41.275) (xy 185.42 62.865))
     (stroke (width 0) (type default))
@@
     (stroke (width 0) (type default))
   )
-  (wire (pts (xy 142.875 102.87) (xy 127 102.87))
+  (wire (pts (xy 142.875 102.87) (xy 132.715 102.87))
     (stroke (width 0) (type default))
   )
@@
     (stroke (width 0) (type default))
   )
-  (wire (pts (xy 130.81 75.565) (xy 123.825 75.565))
+  (wire (pts (xy 137.16 75.565) (xy 123.825 75.565))
     (stroke (width 0) (type default))
   )
@@
     (stroke (width 0) (type default))
   )
+  (wire (pts (xy 128.27 80.645) (xy 123.825 80.645))
+    (stroke (width 0) (type default))
+  )
   (wire (pts (xy 136.525 167.005) (xy 136.525 172.72))
     (stroke (width 0) (type default))
@@
     (stroke (width 0) (type default))
   )
+  (wire (pts (xy 128.27 126.365) (xy 128.27 80.645))
+    (stroke (width 0) (type default))
+  )
   (wire (pts (xy 185.42 102.235) (xy 194.31 102.235))
     (stroke (width 0) (type default))
@@
     (stroke (width 0) (type default))
   )
+  (wire (pts (xy 142.875 126.365) (xy 128.27 126.365))
+    (stroke (width 0) (type default))
+  )
   (wire (pts (xy 236.22 149.225) (xy 236.22 136.525))
     (stroke (width 0) (type default))
@@
     (stroke (width 0) (type default))
   )
+  (wire (pts (xy 153.67 126.365) (xy 156.845 126.365))
+    (stroke (width 0) (type default))
+  )
   (wire (pts (xy 138.43 167.005) (xy 136.525 167.005))
     (stroke (width 0) (type default))
@@
     (stroke (width 0) (type default))
   )
-  (wire (pts (xy 142.875 80.645) (xy 130.81 80.645))
+  (wire (pts (xy 142.875 80.645) (xy 137.16 80.645))
     (stroke (width 0) (type default))
   )
@@
     (stroke (width 0) (type default))
   )
+  (wire (pts (xy 153.67 126.365) (xy 153.67 127))
+    (stroke (width 0) (type default))
+  )
   (wire (pts (xy 92.075 67.945) (xy 93.345 67.945))
     (stroke (width 0) (type default))
@@
     (stroke (width 0) (type default))
   )
-  (wire (pts (xy 130.81 80.645) (xy 130.81 75.565))
+  (wire (pts (xy 137.16 80.645) (xy 137.16 75.565))
     (stroke (width 0) (type default))
   )
@@
     (stroke (width 0) (type default))
   )
-  (wire (pts (xy 127 102.87) (xy 127 78.105))
+  (wire (pts (xy 132.715 102.87) (xy 132.715 78.105))
     (stroke (width 0) (type default))
   )
@@
     (stroke (width 0) (type default))
   )
-  (wire (pts (xy 127 78.105) (xy 123.825 78.105))
+  (wire (pts (xy 132.715 78.105) (xy 123.825 78.105))
     (stroke (width 0) (type default))
   )
@@
   )
   (wire (pts (xy 187.96 41.275) (xy 185.42 41.275))
+    (stroke (width 0) (type default))
+  )
+  (wire (pts (xy 150.495 126.365) (xy 153.67 126.365))
     (stroke (width 0) (type default))
   )
@@
       (effects (font (size 1.27 1.27)))
     )
-    (property "Value" "1000p" (at 227.965 154.94 90)
+    (property "Value" "1n" (at 227.965 154.94 90)
       (effects (font (size 1.27 1.27)))
     )
@@
         (path "/44bc1157-6d68-4ab3-afc0-b8d9f089cc50/8b56ddc3-2841-4bbc-aa12-e659a81ab8f9"
           (reference "U901") (unit 2)
+        )
+      )
+    )
+  )
+  (symbol (lib_id "Connector:TestPoint") (at 156.845 126.365 270) (unit 1)
+    (in_bom yes) (on_board yes) (dnp no) (fields_autoplaced)
+    (property "Reference" "TP901" (at 162.56 125.095 90)
+      (effects (font (size 1.27 1.27)) (justify left))
+    )
+    (property "Value" "TestPoint" (at 162.56 127.635 90)
+      (effects (font (size 1.27 1.27)) (justify left))
+    )
+    (property "Footprint" "TestPoint:TestPoint_Pad_1.0x1.0mm" (at 156.845 131.445 0)
+      (effects (font (size 1.27 1.27)) hide)
+    )
+    (property "Datasheet" "~" (at 156.845 131.445 0)
+      (effects (font (size 1.27 1.27)) hide)
+    )
+    (pin "1")
+    (instances
+      (project "ETH1CFGEN1"
+        (path "/44bc1157-6d68-4ab3-afc0-b8d9f089cc50/8b56ddc3-2841-4bbc-aa12-e659a81ab8f9"
+          (reference "TP901") (unit 1)
         )
       )
@@
     )
   )
+  (symbol (lib_id "Device:R") (at 146.685 126.365 90) (unit 1)
+    (in_bom yes) (on_board yes) (dnp no) (fields_autoplaced)
+    (property "Reference" "R603" (at 146.685 120.65 90)
+      (effects (font (size 1.27 1.27)))
+    )
+    (property "Value" "1k" (at 146.685 123.19 90)
+      (effects (font (size 1.27 1.27)))
+    )
+    (property "Footprint" "Resistor_SMD:R_0603_1608Metric_Pad0.98x0.95mm_HandSolder" (at 146.685 128.143 90)
+      (effects (font (size 1.27 1.27)) hide)
+    )
+    (property "Datasheet" "~" (at 146.685 126.365 0)
+      (effects (font (size 1.27 1.27)) hide)
+    )
+    (pin "1")
+    (pin "2")
+    (instances
+      (project "ETH1CFGEN1B"
+        (path "/3dceb0a1-97ad-435d-a235-e3839b959163/4ac0516f-db36-4471-9493-49791ab70a77"
+          (reference "R603") (unit 1)
+        )
+      )
+      (project "ETH1CFGEN1"
+        (path "/44bc1157-6d68-4ab3-afc0-b8d9f089cc50/8b56ddc3-2841-4bbc-aa12-e659a81ab8f9"
+          (reference "R918") (unit 1)
+        )
+      )
+    )
+  )
   (symbol (lib_id "power:+15V") (at 80.645 158.115 0) (unit 1)
     (in_bom yes) (on_board yes) (dnp no) (fields_autoplaced)
@@
         (path "/44bc1157-6d68-4ab3-afc0-b8d9f089cc50/8b56ddc3-2841-4bbc-aa12-e659a81ab8f9"
           (reference "#PWR0905") (unit 1)
+        )
+      )
+    )
+  )
+  (symbol (lib_id "power:GNDA") (at 153.67 134.62 0) (unit 1)
+    (in_bom yes) (on_board yes) (dnp no)
+    (property "Reference" "#PWR0615" (at 153.67 140.97 0)
+      (effects (font (size 1.27 1.27)) hide)
+    )
+    (property "Value" "GNDA" (at 153.67 139.065 0)
+      (effects (font (size 1.27 1.27)))
+    )
+    (property "Footprint" "" (at 153.67 134.62 0)
+      (effects (font (size 1.27 1.27)) hide)
+    )
+    (property "Datasheet" "" (at 153.67 134.62 0)
+      (effects (font (size 1.27 1.27)) hide)
+    )
+    (pin "1")
+    (instances
+      (project "ETH1CFGEN1B"
+        (path "/3dceb0a1-97ad-435d-a235-e3839b959163/4ac0516f-db36-4471-9493-49791ab70a77"
+          (reference "#PWR0615") (unit 1)
+        )
+      )
+      (project "ETH1CFGEN1"
+        (path "/44bc1157-6d68-4ab3-afc0-b8d9f089cc50/8b56ddc3-2841-4bbc-aa12-e659a81ab8f9"
+          (reference "#PWR0926") (unit 1)
         )
       )
@@
       (effects (font (size 1.27 1.27)))
     )
-    (property "Value" "1000p" (at 227.965 86.36 90)
+    (property "Value" "1n" (at 227.965 86.36 90)
       (effects (font (size 1.27 1.27)))
     )
@@
         )
       )
+    )
+  )
+  (symbol (lib_id "Device:C") (at 153.67 130.81 0) (unit 1)
+    (in_bom yes) (on_board yes) (dnp no) (fields_autoplaced)
+    (property "Reference" "C609" (at 156.845 129.54 0)
+      (effects (font (size 1.27 1.27)) (justify left))
+    )
+    (property "Value" "220n" (at 156.845 132.08 0)
+      (effects (font (size 1.27 1.27)) (justify left))
+    )
+    (property "Footprint" "Capacitor_SMD:C_0603_1608Metric_Pad1.08x0.95mm_HandSolder" (at 154.6352 134.62 0)
+      (effects (font (size 1.27 1.27)) hide)
+    )
+    (property "Datasheet" "~" (at 153.67 130.81 0)
+      (effects (font (size 1.27 1.27)) hide)
+    )
+    (pin "1")
+    (pin "2")
+    (instances
+      (project "ETH1CFGEN1B"
+        (path "/3dceb0a1-97ad-435d-a235-e3839b959163/4ac0516f-db36-4471-9493-49791ab70a77"
+          (reference "C609") (unit 1)
+        )
+      )
+      (project "ETH1CFGEN1"
+        (path "/44bc1157-6d68-4ab3-afc0-b8d9f089cc50/8b56ddc3-2841-4bbc-aa12-e659a81ab8f9"
+          (reference "C917") (unit 1)
+        )
+      )
