File: hardware/ETH1CFGEN1/Output.kicad_sch (KiCad schematic)
At the start: 133 parts, among them K1305 TX2SA-4.5V, K301 G6SU-2F-DC3, Q1301 2N7002, U1301 TL072CD, U1302 LMV339, U1303 TL072CD, U1304 THS3001IDG, U1305 THS3001IDG, U1306 THS3001IDG, U1307 THS3001IDG

Commit message: Development
Parts:
- C1301, C1305, C1306, C1307, C1308, C1309, C1310, C1311, C1312, C1313, C1314, C1315, C1316, C1317, C1318, C1319, C1320, C1321, C1322, C1323, C1324, C1325, C1326, C1327, C1328: footprint (none) -> Capacitor_SMD:C_0603_1608Metric_Pad1.08x0.95mm_HandSolder
- C1304: renamed from C1302; footprint (none) -> Capacitor_SMD:C_0603_1608Metric_Pad1.08x0.95mm_HandSolder
- D1302, D1303: value 5V1 -> SZ1SMB5918BT3G; footprint (none) -> Diode_SMD:D_SMB
- D1304: value D_TVS -> SMCJ43CA; footprint (none) -> Diode_SMD:D_SMC
- D1306: value 1N4184 -> 1N4148; footprint (none) -> Diode_SMD:D_SOD-123
- K1305: footprint (none) -> Relay_SMD:Relay_DPDT_Omron_G6S-2F
- K301: footprint (none) -> Relay_SMD:Relay_DPDT_Omron_G6SK-2F
- L1301, L1302, L1303, L1304: footprint (none) -> Inductor_SMD:L_0603_1608Metric_Pad1.05x0.95mm_HandSolder
- R1301, R1302, R1303, R1304, R1305, R1306, R1307, R1308, R1309, R1310, R1311, R1312, R1313, R1314, R1315, R1316, R1317, R1318, R1319, R1320, R1321, R1322, R1323, R1324, R1325, R1326, R1327, R1328, R1329, R1330, R1331, R1332, R1333, R1334, R1335, R1336, R1337, R1338, R1339, R1340, R1341, R1342, R1343, R1344, R1345, R1346, R1347, R1348, R1349, R1350, R1351, R1352, R1353, R1354, R1355, R1356, R1357, R1358, R1359, R1360, R1361, R1362, R1363, R1364, R1365, R1366, R1367, R1368, R1369, R1370, R1371, R1374, R1375, R1376, R1377, R1378, R1379: footprint (none) -> Resistor_SMD:R_0603_1608Metric_Pad0.98x0.95mm_HandSolder
- R1372: renamed from R1373; footprint (none) -> Resistor_SMD:R_0603_1608Metric_Pad0.98x0.95mm_HandSolder
- R1373: renamed from R1372; footprint (none) -> Resistor_SMD:R_0603_1608Metric_Pad0.98x0.95mm_HandSolder
- U1301, U1303: footprint (none) -> Package_SO:SOIC-8_3.9x4.9mm_P1.27mm
- U1302: value LMV339 -> LMV339IPWR; footprint (none) -> Package_SO:TSSOP-14_4.4x5mm_P0.65mm
Connections:
- net GNDA: now also D1303.1 (K); no longer D1303.2 (A)
- net at C1306.1, D1301.1 (K), R1302.1: now also D1303.2 (A); no longer D1303.1 (K)
Other:
- moved on the sheet: C1306, D1303, R1302

Commit message: PCB design
Parts:
- FL1301: footprint (none) -> ETH1CFGEN1:ACP3225
- L1301, L1302, L1303, L1304: footprint Inductor_SMD:L_0603_1608Metric_Pad1.05x0.95mm_HandSolder -> Inductor_SMD:L_0805_2012Metric_Pad1.15x1.40mm_HandSolder
Changed lines of the file:
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@@
       (effects (font (size 1.27 1.27)))
     )
-    (property "Footprint" "Inductor_SMD:L_0603_1608Metric_Pad1.05x0.95mm_HandSolder" (at 184.15 179.705 0)
+    (property "Footprint" "Inductor_SMD:L_0805_2012Metric_Pad1.15x1.40mm_HandSolder" (at 184.15 179.705 0)
       (effects (font (size 1.27 1.27)) hide)
     )
@@
       (effects (font (size 1.27 1.27)))
     )
-    (property "Footprint" "Inductor_SMD:L_0603_1608Metric_Pad1.05x0.95mm_HandSolder" (at 235.585 64.135 0)
+    (property "Footprint" "Inductor_SMD:L_0805_2012Metric_Pad1.15x1.40mm_HandSolder" (at 235.585 64.135 0)
       (effects (font (size 1.27 1.27)) hide)
     )
@@
       (effects (font (size 1.27 1.27)))
     )
-    (property "Footprint" "" (at 216.535 257.175 0)
+    (property "Footprint" "ETH1CFGEN1:ACP3225" (at 216.535 257.175 0)
       (effects (font (size 1.27 1.27)) hide)
     )
@@
       (effects (font (size 1.27 1.27)))
     )
-    (property "Footprint" "Inductor_SMD:L_0603_1608Metric_Pad1.05x0.95mm_HandSolder" (at 248.285 260.985 0)
+    (property "Footprint" "Inductor_SMD:L_0805_2012Metric_Pad1.15x1.40mm_HandSolder" (at 248.285 260.985 0)
       (effects (font (size 1.27 1.27)) hide)
     )
@@
       (effects (font (size 1.27 1.27)))
     )
-    (property "Footprint" "Inductor_SMD:L_0603_1608Metric_Pad1.05x0.95mm_HandSolder" (at 235.585 260.985 0)
-      (effects (font (size 1.27 1.27)) hide)
-    )
+    (property "Footprint" "Inductor_SMD:L_0805_2012Metric_Pad1.15x1.40mm_HandSolder" (at 235.585 260.985 0)
+      (effects (font (size 1.27 1.27)) hide)
+    )

Commit message: PCB design
Parts:
- removed FB303 (x2): KMZ1608SHR102ATD25, Inductor_SMD:L_0603_1608Metric_Pad1.05x0.95mm_HandSolder, symbol Device:FerriteBead_Small
Connections:
- net +15V_WFD3 is gone; now on net +15V: C320.1, R1366.1, U1301.8 (V+), U1302.3 (V+), U1303.8 (V+)
- net -15V_WFD3 is gone; now on net -15V: C320.1, R1365.1, U1301.4 (V-), U1302.12 (V-), U1303.4 (V-)
Changed lines of the file:
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@@
     (stroke (width 0) (type default))
   )
-  (wire (pts (xy 31.496 267.97) (xy 41.656 267.97))
+  (wire (pts (xy 29.845 267.97) (xy 41.656 267.97))
     (stroke (width 0) (type default))
   )
@@
     (stroke (width 0) (type default))
   )
-  (wire (pts (xy 25.4 247.65) (xy 27.305 247.65))
+  (wire (pts (xy 30.734 247.65) (xy 41.91 247.65))
     (stroke (width 0) (type default))
   )
@@
     (stroke (width 0) (type default))
   )
-  (wire (pts (xy 24.511 267.97) (xy 26.416 267.97))
-    (stroke (width 0) (type default))
-  )
   (wire (pts (xy 280.67 186.055) (xy 297.815 186.055))
     (stroke (width 0) (type default))
@@
     (stroke (width 0) (type default))
   )
-  (wire (pts (xy 32.385 247.65) (xy 41.91 247.65))
-    (stroke (width 0) (type default))
-  )
   (wire (pts (xy 355.6 38.735) (xy 373.38 38.735))
     (stroke (width 0) (type default))
@@
     )
   )
-  (symbol (lib_id "Device:FerriteBead_Small") (at 29.845 247.65 90) (unit 1)
-    (in_bom yes) (on_board yes) (dnp no)
-    (property "Reference" "FB303" (at 29.845 241.935 90)
-      (effects (font (size 1.27 1.27)))
-    )
-    (property "Value" "KMZ1608SHR102ATD25" (at 29.845 244.475 90)
-      (effects (font (size 1.27 1.27)))
-    )
-    (property "Footprint" "Inductor_SMD:L_0603_1608Metric_Pad1.05x0.95mm_HandSolder" (at 29.845 249.428 90)
-      (effects (font (size 1.27 1.27)) hide)
-    )
-    (property "Datasheet" "~" (at 29.845 247.65 0)
-      (effects (font (size 1.27 1.27)) hide)
-    )
-    (pin "1")
-    (pin "2")
-    (instances
-      (project "ETH1CFGEN1B"
-        (path "/3dceb0a1-97ad-435d-a235-e3839b959163/4a966eb3-1da9-4a67-ba6c-e557098bb995"
-          (reference "FB303") (unit 1)
-        )
-        (path "/3dceb0a1-97ad-435d-a235-e3839b959163/4ac0516f-db36-4471-9493-49791ab70a77"
-          (reference "FB601") (unit 1)
-        )
-      )
-      (project "ETH1CFGEN1"
-        (path "/44bc1157-6d68-4ab3-afc0-b8d9f089cc50/8b56ddc3-2841-4bbc-aa12-e659a81ab8f9"
-          (reference "FB901") (unit 1)
-        )
-        (path "/44bc1157-6d68-4ab3-afc0-b8d9f089cc50/89f867e2-a5cd-41fe-8de0-7333d1a4ffe5"
-          (reference "FB1302") (unit 1)
-        )
-      )
-    )
-  )
   (symbol (lib_id "power:GNDA") (at 273.685 42.545 0) (unit 1)
     (in_bom yes) (on_board yes) (dnp no) (fields_autoplaced)
@@
     )
   )
-  (symbol (lib_id "power:+15V") (at 25.4 247.65 90) (unit 1)
+  (symbol (lib_id "power:+15V") (at 30.734 247.65 90) (unit 1)
     (in_bom yes) (on_board yes) (dnp no)
-    (property "Reference" "#PWR0332" (at 29.21 247.65 0)
+    (property "Reference" "#PWR0332" (at 34.544 247.65 0)
       (effects (font (size 1.27 1.27)) hide)
     )
-    (property "Value" "+15V" (at 19.685 247.65 90)
+    (property "Value" "+15V" (at 25.019 247.65 90)
       (effects (font (size 1.27 1.27)))
     )
-    (property "Footprint" "" (at 25.4 247.65 0)
+    (property "Footprint" "" (at 30.734 247.65 0)
       (effects (font (size 1.27 1.27)) hide)
     )
-    (property "Datasheet" "" (at 25.4 247.65 0)
+    (property "Datasheet" "" (at 30.734 247.65 0)
       (effects (font (size 1.27 1.27)) hide)
     )
@@
     )
   )
-  (symbol (lib_id "power:-15V") (at 24.511 267.97 90) (unit 1)
+  (symbol (lib_id "power:-15V") (at 29.845 267.97 90) (unit 1)
     (in_bom yes) (on_board yes) (dnp no) (fields_autoplaced)
-    (property "Reference" "#PWR0602" (at 21.971 267.97 0)
+    (property "Reference" "#PWR0602" (at 27.305 267.97 0)
       (effects (font (size 1.27 1.27)) hide)
     )
-    (property "Value" "-15V" (at 20.701 267.97 90)
+    (property "Value" "-15V" (at 26.035 267.97 90)
       (effects (font (size 1.27 1.27)) (justify left))
     )
-    (property "Footprint" "" (at 24.511 267.97 0)
+    (property "Footprint" "" (at 29.845 267.97 0)
       (effects (font (size 1.27 1.27)) hide)
     )
-    (property "Datasheet" "" (at 24.511 267.97 0)
+    (property "Datasheet" "" (at 29.845 267.97 0)
       (effects (font (size 1.27 1.27)) hide)
     )
@@
         )
       )
-    )
-  )
-  (symbol (lib_id "Device:FerriteBead_Small") (at 28.956 267.97 90) (unit 1)
-    (in_bom yes) (on_board yes) (dnp no)
-    (property "Reference" "FB303" (at 28.956 262.255 90)
-      (effects (font (size 1.27 1.27)))
-    )
-    (property "Value" "KMZ1608SHR102ATD25" (at 28.956 264.795 90)
-      (effects (font (size 1.27 1.27)))
-    )
-    (property "Footprint" "Inductor_SMD:L_0603_1608Metric_Pad1.05x0.95mm_HandSolder" (at 28.956 269.748 90)
-      (effects (font (size 1.27 1.27)) hide)
-    )
-    (property "Datasheet" "~" (at 28.956 267.97 0)
-      (effects (font (size 1.27 1.27)) hide)
-    )
-    (pin "1")
-    (pin "2")
-    (instances
-      (project "ETH1CFGEN1B"
-        (path "/3dceb0a1-97ad-435d-a235-e3839b959163/4a966eb3-1da9-4a67-ba6c-e557098bb995"
-          (reference "FB303") (unit 1)
-        )
-        (path "/3dceb0a1-97ad-435d-a235-e3839b959163/4ac0516f-db36-4471-9493-49791ab70a77"
-          (reference "FB602") (unit 1)
-        )
-      )
-      (project "ETH1CFGEN1"
-        (path "/44bc1157-6d68-4ab3-afc0-b8d9f089cc50/8b56ddc3-2841-4bbc-aa12-e659a81ab8f9"
-          (reference "FB902") (unit 1)
-        )
-        (path "/44bc1157-6d68-4ab3-afc0-b8d9f089cc50/89f867e2-a5cd-41fe-8de0-7333d1a4ffe5"
-          (reference "FB1301") (unit 1)
-        )
-      )

Commit message: PCB design
Parts:
- added C1329, C1331, C1332, C1333: 100n, Capacitor_SMD:C_0603_1608Metric_Pad1.08x0.95mm_HandSolder, symbol Device:C
- added C1330: 1n, Capacitor_SMD:C_0603_1608Metric_Pad1.08x0.95mm_HandSolder, symbol Device:C
- added R1380: 100, Resistor_SMD:R_0603_1608Metric_Pad0.98x0.95mm_HandSolder, symbol Device:R
- R1323: value 383 -> 237
- R1324: value 383 -> 249
- R1326: value 287 -> 16k2
- R1327: value 287 -> 511
- R1333: value 383 -> 3k6
Connections:
- net +15V: now also C1332.2
- net -15V: now also C1333.2
- net GNDA: now also C1329.2, C1330.1, C1331.1, C1332.1, C1333.1, R1380.2
- net OUTPUT_ENABLE: now also C1330.2
- net at D1306.2 (A), K1305.12, Q1301.3 (D): now also C1331.2
- net at K301.3: now also C1329.1, R1380.1
Other:
- moved on the sheet: D1306, Q1301

Commit message: PCB design
Parts:
- removed C320 (x2): 10u, Capacitor_SMD:C_1206_3216Metric_Pad1.33x1.80mm_HandSolder, symbol Device:C
Connections:
- net +5V renamed +5VD
Changed lines of the file:
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@@
   (junction (at 309.245 186.055) (diameter 0) (color 0 0 0 0)
   )
-  (junction (at 41.656 267.97) (diameter 0) (color 0 0 0 0)
-  )
   (junction (at 109.855 104.775) (diameter 0) (color 0 0 0 0)
   )
@@
   (junction (at 319.405 87.63) (diameter 0) (color 0 0 0 0)
   )
-  (junction (at 41.91 247.65) (diameter 0) (color 0 0 0 0)
-  )
   (junction (at 218.44 149.225) (diameter 0) (color 0 0 0 0)
   )
@@
     (stroke (width 0) (type default))
   )
-  (wire (pts (xy 29.845 267.97) (xy 41.656 267.97))
-    (stroke (width 0) (type default))
-  )
   (wire (pts (xy 41.275 114.3) (xy 41.275 112.395))
     (stroke (width 0) (type default))
@@
     (stroke (width 0) (type default))
   )
-  (wire (pts (xy 41.91 247.65) (xy 55.88 247.65))
+  (wire (pts (xy 30.734 247.65) (xy 55.88 247.65))
     (stroke (width 0) (type default))
   )
@@
     (stroke (width 0) (type default))
   )
-  (wire (pts (xy 41.656 276.225) (xy 41.656 276.86))
-    (stroke (width 0) (type default))
-  )
   (wire (pts (xy 109.855 104.775) (xy 109.855 106.045))
     (stroke (width 0) (type default))
@@
     (stroke (width 0) (type default))
   )
-  (wire (pts (xy 41.91 247.65) (xy 41.91 248.285))
-    (stroke (width 0) (type default))
-  )
   (wire (pts (xy 309.245 186.055) (xy 313.055 186.055))
     (stroke (width 0) (type default))
@@
     (stroke (width 0) (type default))
   )
-  (wire (pts (xy 30.734 247.65) (xy 41.91 247.65))
-    (stroke (width 0) (type default))
-  )
   (wire (pts (xy 243.84 219.71) (xy 245.11 219.71))
     (stroke (width 0) (type default))
@@
     (stroke (width 0) (type default))
   )
-  (wire (pts (xy 41.91 255.905) (xy 41.91 256.54))
-    (stroke (width 0) (type default))
-  )
   (wire (pts (xy 153.67 124.46) (xy 153.67 132.715))
     (stroke (width 0) (type default))
@@
     (stroke (width 0) (type default))
   )
-  (wire (pts (xy 41.656 267.97) (xy 41.656 268.605))
-    (stroke (width 0) (type default))
-  )
   (wire (pts (xy 223.52 64.135) (xy 227.965 64.135))
     (stroke (width 0) (type default))
@@
     (stroke (width 0) (type default))
   )
-  (wire (pts (xy 41.656 267.97) (xy 55.88 267.97))
+  (wire (pts (xy 29.845 267.97) (xy 55.88 267.97))
     (stroke (width 0) (type default))
   )
@@
     )
   )
-  (symbol (lib_id "power:GNDA") (at 41.656 276.86 0) (unit 1)
-    (in_bom yes) (on_board yes) (dnp no) (fields_autoplaced)
-    (property "Reference" "#PWR0338" (at 41.656 283.21 0)
-      (effects (font (size 1.27 1.27)) hide)
-    )
-    (property "Value" "GNDA" (at 41.656 281.305 0)
-      (effects (font (size 1.27 1.27)))
-    )
-    (property "Footprint" "" (at 41.656 276.86 0)
-      (effects (font (size 1.27 1.27)) hide)
-    )
-    (property "Datasheet" "" (at 41.656 276.86 0)
-      (effects (font (size 1.27 1.27)) hide)
-    )
-    (pin "1")
-    (instances
-      (project "ETH1CFGEN1B"
-        (path "/3dceb0a1-97ad-435d-a235-e3839b959163/4a966eb3-1da9-4a67-ba6c-e557098bb995"
-          (reference "#PWR0338") (unit 1)
-        )
-        (path "/3dceb0a1-97ad-435d-a235-e3839b959163/4ac0516f-db36-4471-9493-49791ab70a77"
-          (reference "#PWR0608") (unit 1)
-        )
-      )
-      (project "ETH1CFGEN1"
-        (path "/44bc1157-6d68-4ab3-afc0-b8d9f089cc50/8b56ddc3-2841-4bbc-aa12-e659a81ab8f9"
-          (reference "#PWR0908") (unit 1)
-        )
-        (path "/44bc1157-6d68-4ab3-afc0-b8d9f089cc50/89f867e2-a5cd-41fe-8de0-7333d1a4ffe5"
-          (reference "#PWR01305") (unit 1)
-        )
-      )
-    )
-  )
   (symbol (lib_id "power:+15V") (at 30.734 247.65 90) (unit 1)
     (in_bom yes) (on_board yes) (dnp no)
@@
     )
   )
+  (symbol (lib_id "power:+5VD") (at 379.095 61.595 270) (unit 1)
+    (in_bom yes) (on_board yes) (dnp no) (fields_autoplaced)
+    (property "Reference" "#PWR01314" (at 375.285 61.595 0)
+      (effects (font (size 1.27 1.27)) hide)
+    )
+    (property "Value" "+5VD" (at 382.27 61.595 90)
+      (effects (font (size 1.27 1.27)) (justify left))
+    )
+    (property "Footprint" "" (at 379.095 61.595 0)
+      (effects (font (size 1.27 1.27)) hide)
+    )
+    (property "Datasheet" "" (at 379.095 61.595 0)
+      (effects (font (size 1.27 1.27)) hide)
+    )
+    (pin "1")
+    (instances
+      (project "ETH1CFGEN1"
+        (path "/44bc1157-6d68-4ab3-afc0-b8d9f089cc50/89f867e2-a5cd-41fe-8de0-7333d1a4ffe5"
+          (reference "#PWR01314") (unit 1)
+        )
+      )
+    )
+  )
   (symbol (lib_id "Device:R") (at 139.065 132.715 90) (unit 1)
     (in_bom yes) (on_board yes) (dnp no)
@@
     )
   )
-  (symbol (lib_id "power:+5V") (at 379.095 61.595 270) (unit 1)
-    (in_bom yes) (on_board yes) (dnp no) (fields_autoplaced)
-    (property "Reference" "#PWR01361" (at 375.285 61.595 0)
-      (effects (font (size 1.27 1.27)) hide)
-    )
-    (property "Value" "+5V" (at 382.27 61.595 90)
-      (effects (font (size 1.27 1.27)) (justify left))
-    )
-    (property "Footprint" "" (at 379.095 61.595 0)
-      (effects (font (size 1.27 1.27)) hide)
-    )
-    (property "Datasheet" "" (at 379.095 61.595 0)
-      (effects (font (size 1.27 1.27)) hide)
-    )
-    (pin "1")
-    (instances
-      (project "ETH1CFGEN1"
-        (path "/44bc1157-6d68-4ab3-afc0-b8d9f089cc50/89f867e2-a5cd-41fe-8de0-7333d1a4ffe5"
-          (reference "#PWR01361") (unit 1)
-        )
-      )
-    )
-  )
   (symbol (lib_id "Device:R") (at 271.145 102.87 90) (unit 1)
     (in_bom yes) (on_board yes) (dnp no)
@@
     )
   )
-  (symbol (lib_id "Device:C") (at 41.91 252.095 0) (unit 1)
-    (in_bom yes) (on_board yes) (dnp no) (fields_autoplaced)
-    (property "Reference" "C320" (at 45.085 250.825 0)
-      (effects (font (size 1.27 1.27)) (justify left))
-    )
-    (property "Value" "10u" (at 45.085 253.365 0)
-      (effects (font (size 1.27 1.27)) (justify left))
-    )
-    (property "Footprint" "Capacitor_SMD:C_1206_3216Metric_Pad1.33x1.80mm_HandSolder" (at 42.8752 255.905 0)
-      (effects (font (size 1.27 1.27)) hide)
-    )
-    (property "Datasheet" "~" (at 41.91 252.095 0)
-      (effects (font (size 1.27 1.27)) hide)
-    )
-    (pin "1")
-    (pin "2")
-    (instances
-      (project "ETH1CFGEN1B"
-        (path "/3dceb0a1-97ad-435d-a235-e3839b959163/4a966eb3-1da9-4a67-ba6c-e557098bb995"
-          (reference "C320") (unit 1)
-        )
-        (path "/3dceb0a1-97ad-435d-a235-e3839b959163/4ac0516f-db36-4471-9493-49791ab70a77"
-          (reference "C604") (unit 1)
-        )
-      )
-      (project "ETH1CFGEN1"
-        (path "/44bc1157-6d68-4ab3-afc0-b8d9f089cc50/8b56ddc3-2841-4bbc-aa12-e659a81ab8f9"
-          (reference "C904") (unit 1)
-        )
-        (path "/44bc1157-6d68-4ab3-afc0-b8d9f089cc50/89f867e2-a5cd-41fe-8de0-7333d1a4ffe5"
-          (reference "C1303") (unit 1)
-        )
-      )
-    )
-  )
   (symbol (lib_id "power:GNDA") (at 109.22 104.775 270) (unit 1)
     (in_bom yes) (on_board yes) (dnp no) (fields_autoplaced)
@@
     )
   )
-  (symbol (lib_id "Device:C") (at 41.656 272.415 0) (unit 1)
-    (in_bom yes) (on_board yes) (dnp no) (fields_autoplaced)
-    (property "Reference" "C320" (at 44.831 271.145 0)
-      (effects (font (size 1.27 1.27)) (justify left))
-    )
-    (property "Value" "10u" (at 44.831 273.685 0)
-      (effects (font (size 1.27 1.27)) (justify left))
-    )
-    (property "Footprint" "Capacitor_SMD:C_1206_3216Metric_Pad1.33x1.80mm_HandSolder" (at 42.6212 276.225 0)
-      (effects (font (size 1.27 1.27)) hide)
-    )
-    (property "Datasheet" "~" (at 41.656 272.415 0)
-      (effects (font (size 1.27 1.27)) hide)
-    )
-    (pin "1")
-    (pin "2")
-    (instances
-      (project "ETH1CFGEN1B"
-        (path "/3dceb0a1-97ad-435d-a235-e3839b959163/4a966eb3-1da9-4a67-ba6c-e557098bb995"
-          (reference "C320") (unit 1)
-        )
-        (path "/3dceb0a1-97ad-435d-a235-e3839b959163/4ac0516f-db36-4471-9493-49791ab70a77"
-          (reference "C605") (unit 1)
-        )
-      )
-      (project "ETH1CFGEN1"
-        (path "/44bc1157-6d68-4ab3-afc0-b8d9f089cc50/8b56ddc3-2841-4bbc-aa12-e659a81ab8f9"
-          (reference "C905") (unit 1)
-        )
-        (path "/44bc1157-6d68-4ab3-afc0-b8d9f089cc50/89f867e2-a5cd-41fe-8de0-7333d1a4ffe5"
-          (reference "C1302") (unit 1)
-        )
-      )
-    )
-  )
   (symbol (lib_id "Amplifier_Operational:TL072") (at 130.175 192.405 0) (mirror x) (unit 2)
     (in_bom yes) (on_board yes) (dnp no)
@@
         )
       )
-    )
-  )
-  (symbol (lib_id "power:GNDA") (at 41.91 256.54 0) (unit 1)
-    (in_bom yes) (on_board yes) (dnp no) (fields_autoplaced)
-    (property "Reference" "#PWR0338" (at 41.91 262.89 0)
-      (effects (font (size 1.27 1.27)) hide)
-    )
-    (property "Value" "GNDA" (at 41.91 260.985 0)
-      (effects (font (size 1.27 1.27)))
-    )
-    (property "Footprint" "" (at 41.91 256.54 0)
-      (effects (font (size 1.27 1.27)) hide)
-    )
-    (property "Datasheet" "" (at 41.91 256.54 0)
-      (effects (font (size 1.27 1.27)) hide)
-    )
-    (pin "1")
-    (instances
-      (project "ETH1CFGEN1B"
-        (path "/3dceb0a1-97ad-435d-a235-e3839b959163/4a966eb3-1da9-4a67-ba6c-e557098bb995"
-          (reference "#PWR0338") (unit 1)
-        )
-        (path "/3dceb0a1-97ad-435d-a235-e3839b959163/4ac0516f-db36-4471-9493-49791ab70a77"
-          (reference "#PWR0607") (unit 1)
-        )
-      )
-      (project "ETH1CFGEN1"
-        (path "/44bc1157-6d68-4ab3-afc0-b8d9f089cc50/8b56ddc3-2841-4bbc-aa12-e659a81ab8f9"
-          (reference "#PWR0907") (unit 1)
-        )
-        (path "/44bc1157-6d68-4ab3-afc0-b8d9f089cc50/89f867e2-a5cd-41fe-8de0-7333d1a4ffe5"
-          (reference "#PWR01306") (unit 1)
-        )
-      )

Commit message: PCB design
Parts:
- removed C1301, C1304, C1307, C1308, C1314, C1315, C1322, C1323: 100p, Capacitor_SMD:C_0603_1608Metric_Pad1.08x0.95mm_HandSolder, symbol Device:C
- removed C1330: 1n, Capacitor_SMD:C_0603_1608Metric_Pad1.08x0.95mm_HandSolder, symbol Device:C
- removed K1305: TX2SA-4.5V, Relay_SMD:Relay_DPDT_Omron_G6S-2F, symbol Relay:G6S-2
- removed Q1301: 2N7002, Package_TO_SOT_SMD:SOT-23, symbol Transistor_FET:2N7002
- added D? (x4): 1N4148W, Diode_SMD:D_SOD-123, symbol Diode:1N4148W
- added K301: G6S-2F-DC5, Relay_SMD:Relay_DPDT_Omron_G6SK-2F, symbol Relay:G6S-2
- added Q? (x5): BC847, Package_TO_SOT_SMD:SOT-23, symbol Transistor_BJT:BC847
- added R307 (x5): 1k, Resistor_SMD:R_0603_1608Metric_Pad0.98x0.95mm_HandSolder, symbol Device:R
- K301: value G6SU-2F-DC3 -> G6S-2F-DC5; symbol Relay:G6SU-2 -> Relay:G6S-2
Connections:
- net RST_-10DB is gone; now on net +5VD: K301.1
- net RST_-20DB is gone; now on net +5VD: K301.1
- net SET_+20DB is gone; now on net +5VD: K301.1
- net SET_SQ_PLS is gone; now on net +5VD: K301.1
- net +5VD: now also D?.1 (K), D?.1 (K), D?.1 (K), D?.1 (K), K301.1
- net GNDA: now also K301.3, K301.4, K301.5, Q?.2 (E)
- net OUTPUT: now also K301.8
- net OUTPUT_ENABLE: now also R307.2
- net at C1331.2, D1306.2 (A): now also K301.12, Q?.3 (C)
- net at D1305.3 (K), K301.9, R1361.2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: now also K301.9
- net at R1378.1: now also K301.10
- net RST_+20DB: no longer names the net of K301.12
- net RST_+20DB: now also D?.2 (A), Q?.3 (C)
- net SET_-10DB: no longer names the net of K301.12
- net SET_-10DB: now also D?.2 (A), Q?.3 (C)
- net SET_-20DB: no longer names the net of K301.12
- net SET_-20DB: now also D?.2 (A), Q?.3 (C)
- net SET_SIN_ARB: no longer names the net of K301.12
- net SET_SIN_ARB: now also D?.2 (A), Q?.3 (C)
- new net: Q?.1 (B), R307.1 (x5)
- new net GNDD: Q?.2 (E), Q?.2 (E), Q?.2 (E), Q?.2 (E)
- new net REL_+20DB: R307.2
- new net REL_-10DB: R307.2
- new net REL_-20DB: R307.2
- new net REL_SQ-SIN: R307.2

Commit message: Schematic and PCB design
Parts:
- gave numbers to parts that had none: 9
- renumbered C1305 to C1301, C1306 to C1302, C1309 to C1303, C1310 to C1304, C1311 to C1305, C1312 to C1306, C1313 to C1307, C1316 to C1308, C1317 to C1309, C1318 to C1310, C1319 to C1311, C1320 to C1312, C1321 to C1313, C1329 to C1314, C1324 to C1315, C1325 to C1316, C1326 to C1317, C1332 to C1318, C1333 to C1319, C1327 to C1320, C1328 to C1321, C1331 to C1322, D1301 to D1302, D1302 to D1303, D1303 to D1304, D1304 to D1307, D1305 to D1309, D1306 to D1310, R1301 to R1302, R1302 to R1303, R1303 to R1304, R1304 to R1306, R1305 to R1307, R1306 to R1308, R1307 to R1309, R1308 to R1310, R1309 to R1311, R1310 to R1312, R1311 to R1313, R1312 to R1314, R1313 to R1315, R1314 to R1316, R1315 to R1317, R1316 to R1318, R1317 to R1319, R1318 to R1320, R1319 to R1322, R1320 to R1323, R1321 to R1324, R1322 to R1325, R1323 to R1326, R1324 to R1327, R1325 to R1328, R1326 to R1329, R1327 to R1330, R1328 to R1331, R1329 to R1332, R1330 to R1333, R1331 to R1334, R1332 to R1335, R1333 to R1336, R1334 to R1337, R1335 to R1338, R1336 to R1339, R1337 to R1340, R1338 to R1341, R1339 to R1342, R1340 to R1343, R1341 to R1344, R1342 to R1345, R1343 to R1347, R1344 to R1348, R1345 to R1349, R1346 to R1350, R1347 to R1351, R1348 to R1352, R1349 to R1353, R1350 to R1354, R1351 to R1355, R1352 to R1356, R1353 to R1357, R1354 to R1358, R1355 to R1359, R1356 to R1360, R1357 to R1361, R1358 to R1362, R1380 to R1363, R1359 to R1364, R1360 to R1365, R1361 to R1366, R1362 to R1367, R1363 to R1368, R1364 to R1369, R1365 to R1370, R1366 to R1371, R1367 to R1372, R1368 to R1373, R1369 to R1374, R1370 to R1375, R1371 to R1376, R1372 to R1377, R1373 to R1378, R1374 to R1379, R1375 to R1380, R1376 to R1381, R1377 to R1382, R1378 to R1383, R1379 to R1385
