File: hardware/ETH1CFGEN1/SelftTest.kicad_sch (KiCad schematic)
At the start: 30 parts, among them U801 TL074HIPWR, U802 TL074HIPWR, U803 TLA2528IRTER

Commit message: Development
Connections:
- net I2C_SCL renamed ADC_I2C_SCL
- net I2C_SDA renamed ADC_I2C_SDA
Changed lines of the file:
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@@
 (kicad_sch (version 20230121) (generator eeschema)
   (paper "A4")
+  (title_block
+    (date "2023-07-12")
+    (rev "1.1")
+  )
   (junction (at 193.675 27.305) (diameter 0) (color 0 0 0 0)
   )
@@
     (effects (font (size 1.27 1.27)) (justify right bottom))
   )
-  (hierarchical_label "I2C_SDA" (shape bidirectional) (at 252.73 111.125 0) (fields_autoplaced)
+  (hierarchical_label "ADC_I2C_SDA" (shape bidirectional) (at 252.73 111.125 0) (fields_autoplaced)
     (effects (font (size 1.27 1.27)) (justify left))
   )
-  (hierarchical_label "I2C_SCL" (shape bidirectional) (at 252.73 108.585 0) (fields_autoplaced)
+  (hierarchical_label "ADC_I2C_SCL" (shape bidirectional) (at 252.73 108.585 0) (fields_autoplaced)
     (effects (font (size 1.27 1.27)) (justify left))
   )

Commit message: PCB design
Parts:
- removed C803, C804: 100n, Capacitor_SMD:C_0603_1608Metric_Pad1.08x0.95mm_HandSolder, symbol Device:C
- renumbered C805 to C803, C806 to C804, C807 to C805, C808 to C806, C809 to C807
Other:
- moved on the sheet: C803, C804, C805, C806

Commit message: PCB design
Other:
- moved on the sheet: C801, C802, C803, C804
