File: hardware/ETH1CFGEN1/Square.kicad_sch (KiCad schematic)
At the start: 85 parts, among them Q401 MMBF4416A, Q402 MMBFJ175LT1, Q403 MMBT5087LT1G, Q404 MMBT6429LT1, U401 AD706ARZ, U402 AD706ARZ, U403 AD706ARZ, U404 AD1851RZ, U405 AD8180ARZ, U406 AD8009AR, U407 AD8009AR

Commit message: Development
Parts:
- removed C369 (x2): 22u, symbol Device:C_Polarized
- added C309 (x2): 22u, Capacitor_Tantalum_SMD:CP_EIA-7343-31_Kemet-D_Pad2.25x2.55mm_HandSolder, symbol Device:C_Polarized
- L401, L402, L403: footprint (none) -> Inductor_SMD:L_0603_1608Metric_Pad1.05x0.95mm_HandSolder
- Q401, Q402, Q403, Q404: footprint (none) -> Package_TO_SOT_SMD:SOT-23
Connections:
- net GNDA: now also C309.1, C309.2
- net at C404.1, FB307.2, U404.16 (+VS): now also C309.1
- net at C403.1, FB307.2, U404.1 (-Vs): now also C309.2
Changed lines of the file:
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@@
 (kicad_sch (version 20230121) (generator eeschema)
   (paper "A3")
+  (title_block
+    (date "2023-07-12")
+    (rev "1.1")
+  )
   (junction (at 255.905 43.18) (diameter 0) (color 0 0 0 0)
   )
@@
       (effects (font (size 1.27 1.27)) (justify left))
     )
-    (property "Footprint" "" (at 354.33 162.56 0)
+    (property "Footprint" "Inductor_SMD:L_0603_1608Metric_Pad1.05x0.95mm_HandSolder" (at 354.33 162.56 0)
       (effects (font (size 1.27 1.27)) hide)
     )
@@
       (effects (font (size 1.27 1.27)))
     )
-    (property "Footprint" "" (at 115.57 112.395 0)
+    (property "Footprint" "Inductor_SMD:L_0603_1608Metric_Pad1.05x0.95mm_HandSolder" (at 115.57 112.395 0)
       (effects (font (size 1.27 1.27)) hide)
     )
@@
     )
   )
-  (symbol (lib_id "Device:C_Polarized") (at 90.805 74.295 0) (unit 1)
-    (in_bom yes) (on_board yes) (dnp no) (fields_autoplaced)
-    (property "Reference" "C369" (at 93.98 72.136 0)
-      (effects (font (size 1.27 1.27)) (justify left))
-    )
-    (property "Value" "22u" (at 93.98 74.676 0)
-      (effects (font (size 1.27 1.27)) (justify left))
-    )
-    (property "Footprint" "" (at 91.7702 78.105 0)
-      (effects (font (size 1.27 1.27)) hide)
-    )
-    (property "Datasheet" "~" (at 90.805 74.295 0)
-      (effects (font (size 1.27 1.27)) hide)
-    )
-    (pin "1")
-    (pin "2")
-    (instances
-      (project "ETH1CFGEN1B"
-        (path "/3dceb0a1-97ad-435d-a235-e3839b959163/4a966eb3-1da9-4a67-ba6c-e557098bb995"
-          (reference "C369") (unit 1)
-        )
-        (path "/3dceb0a1-97ad-435d-a235-e3839b959163/a29df865-98bf-4fa6-a65a-56d8d0a1d3db"
-          (reference "C406") (unit 1)
-        )
-      )
-      (project "ETH1CFGEN1"
-        (path "/44bc1157-6d68-4ab3-afc0-b8d9f089cc50/9b89076f-b382-432c-8652-bfba09d4fc07"
-          (reference "C1206") (unit 1)
-        )
-      )
-    )
-  )
   (symbol (lib_id "Device:C") (at 96.52 117.475 0) (unit 1)
     (in_bom yes) (on_board yes) (dnp no) (fields_autoplaced)
@@
     )
   )
+  (symbol (lib_id "Device:C_Polarized") (at 61.595 138.43 180) (unit 1)
+    (in_bom yes) (on_board yes) (dnp no) (fields_autoplaced)
+    (property "Reference" "C309" (at 64.77 138.049 0)
+      (effects (font (size 1.27 1.27)) (justify right))
+    )
+    (property "Value" "22u" (at 64.77 140.589 0)
+      (effects (font (size 1.27 1.27)) (justify right))
+    )
+    (property "Footprint" "Capacitor_Tantalum_SMD:CP_EIA-7343-31_Kemet-D_Pad2.25x2.55mm_HandSolder" (at 60.6298 134.62 0)
+      (effects (font (size 1.27 1.27)) hide)
+    )
+    (property "Datasheet" "~" (at 61.595 138.43 0)
+      (effects (font (size 1.27 1.27)) hide)
+    )
+    (pin "1")
+    (pin "2")
+    (instances
+      (project "ETH1CFGEN1B"
+        (path "/3dceb0a1-97ad-435d-a235-e3839b959163/4a966eb3-1da9-4a67-ba6c-e557098bb995"
+          (reference "C309") (unit 1)
+        )
+        (path "/3dceb0a1-97ad-435d-a235-e3839b959163/4ac0516f-db36-4471-9493-49791ab70a77"
+          (reference "C606") (unit 1)
+        )
+      )
+      (project "ETH1CFGEN1"
+        (path "/44bc1157-6d68-4ab3-afc0-b8d9f089cc50/8b56ddc3-2841-4bbc-aa12-e659a81ab8f9"
+          (reference "C906") (unit 1)
+        )
+        (path "/44bc1157-6d68-4ab3-afc0-b8d9f089cc50/9b89076f-b382-432c-8652-bfba09d4fc07"
+          (reference "C1202") (unit 1)
+        )
+      )
+    )
+  )
   (symbol (lib_id "ETH1CFGEN1:AD706") (at 179.705 180.34 0) (unit 1)
     (in_bom yes) (on_board yes) (dnp no)
@@
     )
   )
-  (symbol (lib_id "Device:C_Polarized") (at 61.595 138.43 0) (unit 1)
-    (in_bom yes) (on_board yes) (dnp no) (fields_autoplaced)
-    (property "Reference" "C369" (at 64.77 136.271 0)
-      (effects (font (size 1.27 1.27)) (justify left))
-    )
-    (property "Value" "22u" (at 64.77 138.811 0)
-      (effects (font (size 1.27 1.27)) (justify left))
-    )
-    (property "Footprint" "" (at 62.5602 142.24 0)
-      (effects (font (size 1.27 1.27)) hide)
-    )
-    (property "Datasheet" "~" (at 61.595 138.43 0)
-      (effects (font (size 1.27 1.27)) hide)
-    )
-    (pin "1")
-    (pin "2")
-    (instances
-      (project "ETH1CFGEN1B"
-        (path "/3dceb0a1-97ad-435d-a235-e3839b959163/4a966eb3-1da9-4a67-ba6c-e557098bb995"
-          (reference "C369") (unit 1)
-        )
-        (path "/3dceb0a1-97ad-435d-a235-e3839b959163/a29df865-98bf-4fa6-a65a-56d8d0a1d3db"
-          (reference "C402") (unit 1)
-        )
-      )
-      (project "ETH1CFGEN1"
-        (path "/44bc1157-6d68-4ab3-afc0-b8d9f089cc50/9b89076f-b382-432c-8652-bfba09d4fc07"
-          (reference "C1202") (unit 1)
-        )
-      )
-    )
-  )
   (symbol (lib_id "power:GNDA") (at 304.165 52.07 0) (unit 1)
     (in_bom yes) (on_board yes) (dnp no) (fields_autoplaced)
@@
       (effects (font (size 1.27 1.27)) (justify left))
     )
-    (property "Footprint" "" (at 210.185 177.8 0)
+    (property "Footprint" "Package_TO_SOT_SMD:SOT-23" (at 210.185 177.8 0)
       (effects (font (size 1.27 1.27)) hide)
     )
@@
       (effects (font (size 1.27 1.27)) (justify left))
     )
-    (property "Footprint" "" (at 294.005 69.85 0)
+    (property "Footprint" "Package_TO_SOT_SMD:SOT-23" (at 294.005 69.85 0)
       (effects (font (size 1.27 1.27)) hide)
     )
@@
       (effects (font (size 1.27 1.27)) (justify left))
     )
-    (property "Footprint" "" (at 204.47 58.42 0)
+    (property "Footprint" "Package_TO_SOT_SMD:SOT-23" (at 204.47 58.42 0)
       (effects (font (size 1.27 1.27)) hide)
     )
@@
     )
   )
+  (symbol (lib_id "Device:C_Polarized") (at 90.805 74.295 0) (unit 1)
+    (in_bom yes) (on_board yes) (dnp no) (fields_autoplaced)
+    (property "Reference" "C309" (at 93.98 72.136 0)
+      (effects (font (size 1.27 1.27)) (justify left))
+    )
+    (property "Value" "22u" (at 93.98 74.676 0)
+      (effects (font (size 1.27 1.27)) (justify left))
+    )
+    (property "Footprint" "Capacitor_Tantalum_SMD:CP_EIA-7343-31_Kemet-D_Pad2.25x2.55mm_HandSolder" (at 91.7702 78.105 0)
+      (effects (font (size 1.27 1.27)) hide)
+    )
+    (property "Datasheet" "~" (at 90.805 74.295 0)
+      (effects (font (size 1.27 1.27)) hide)
+    )
+    (pin "1")
+    (pin "2")
+    (instances
+      (project "ETH1CFGEN1B"
+        (path "/3dceb0a1-97ad-435d-a235-e3839b959163/4a966eb3-1da9-4a67-ba6c-e557098bb995"
+          (reference "C309") (unit 1)
+        )
+        (path "/3dceb0a1-97ad-435d-a235-e3839b959163/4ac0516f-db36-4471-9493-49791ab70a77"
+          (reference "C606") (unit 1)
+        )
+      )
+      (project "ETH1CFGEN1"
+        (path "/44bc1157-6d68-4ab3-afc0-b8d9f089cc50/8b56ddc3-2841-4bbc-aa12-e659a81ab8f9"
+          (reference "C906") (unit 1)
+        )
+        (path "/44bc1157-6d68-4ab3-afc0-b8d9f089cc50/9b89076f-b382-432c-8652-bfba09d4fc07"
+          (reference "C1206") (unit 1)
+        )
+      )
+    )
+  )
   (symbol (lib_id "power:GNDA") (at 159.385 122.555 0) (unit 1)
     (in_bom yes) (on_board yes) (dnp no) (fields_autoplaced)
@@
       (effects (font (size 1.27 1.27)) (justify left))
     )
-    (property "Footprint" "" (at 245.745 149.225 0)
+    (property "Footprint" "Inductor_SMD:L_0603_1608Metric_Pad1.05x0.95mm_HandSolder" (at 245.745 149.225 0)
       (effects (font (size 1.27 1.27)) hide)
     )
@@
       (effects (font (size 1.27 1.27)) (justify left))
     )
-    (property "Footprint" "" (at 294.005 177.8 0)
+    (property "Footprint" "Package_TO_SOT_SMD:SOT-23" (at 294.005 177.8 0)
       (effects (font (size 1.27 1.27)) hide)
     )

Commit message: PCB design
Parts:
- L401, L402, L403: footprint Inductor_SMD:L_0603_1608Metric_Pad1.05x0.95mm_HandSolder -> Inductor_SMD:L_0805_2012Metric_Pad1.15x1.40mm_HandSolder
Changed lines of the file:
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@@
       (effects (font (size 1.27 1.27)) (justify left))
     )
-    (property "Footprint" "Inductor_SMD:L_0603_1608Metric_Pad1.05x0.95mm_HandSolder" (at 354.33 162.56 0)
+    (property "Footprint" "Inductor_SMD:L_0805_2012Metric_Pad1.15x1.40mm_HandSolder" (at 354.33 162.56 0)
       (effects (font (size 1.27 1.27)) hide)
     )
@@
       (effects (font (size 1.27 1.27)))
     )
-    (property "Footprint" "Inductor_SMD:L_0603_1608Metric_Pad1.05x0.95mm_HandSolder" (at 115.57 112.395 0)
+    (property "Footprint" "Inductor_SMD:L_0805_2012Metric_Pad1.15x1.40mm_HandSolder" (at 115.57 112.395 0)
       (effects (font (size 1.27 1.27)) hide)
     )
@@
       (effects (font (size 1.27 1.27)) (justify left))
     )
-    (property "Footprint" "Inductor_SMD:L_0603_1608Metric_Pad1.05x0.95mm_HandSolder" (at 245.745 149.225 0)
+    (property "Footprint" "Inductor_SMD:L_0805_2012Metric_Pad1.15x1.40mm_HandSolder" (at 245.745 149.225 0)
       (effects (font (size 1.27 1.27)) hide)
     )

Commit message: PCB design
Parts:
- removed C309 (x2): 22u, Capacitor_Tantalum_SMD:CP_EIA-7343-31_Kemet-D_Pad2.25x2.55mm_HandSolder, symbol Device:C_Polarized
- removed FB307 (x3): KMZ1608SHR102ATD25, Inductor_SMD:L_0603_1608Metric_Pad1.05x0.95mm_HandSolder, symbol Device:FerriteBead_Small
Connections:
- net +5V_WFD is gone; now on net +5V: C405.1, C407.1, C410.1, U405.4 (+VS), U406.7 (V+), U407.7 (V+)
- net -5V_WFD is gone; now on net -5V: C411.1, C412.1, C413.1, U405.5 (-VS), U406.4 (V-), U407.4 (V-)
- net +15V_WFD1: no longer U401.8 (V+), U402.8 (V+), U403.8 (V+)
- net +5V: now also C401.1, C404.1, U404.16 (+VS), U404.3 (+Vl)
- net -15V_WFD1: no longer U401.4 (V-), U402.4 (V-), U403.4 (V-)
- net -5V: now also C403.1, U404.1 (-Vs)
- new net +15V: U401.8 (V+), U402.8 (V+), U403.8 (V+)
- new net -15V: U401.4 (V-), U402.4 (V-), U403.4 (V-)
Other:
- moved on the sheet: C405, C407, C410, C411, C412, C413, U401C, U402C

Commit message: PCB design
Connections:
- net +15V_WFD1 is gone; now on net +15V: D401.3 (K)
- net -15V_WFD1 is gone; now on net -15V: D402.1 (A)
- net at Q404.2 (E), R430.1: now also D404.1 (K), R425.2
Other:
- moved on the sheet: C426, R431
