File: hardware/ETH1CFGEN1/Trigger.kicad_sch (KiCad schematic)
At the start: 22 parts, among them U701 TXB0104PW, U702 ADuM5402, U703 74AC125

Commit message: PCB design
Connections:
- net +5V renamed +5VD
Changed lines of the file:
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@@
-    )
-  )
-  (symbol (lib_id "power:+5V") (at 82.55 21.59 0) (unit 1)
-    (in_bom yes) (on_board yes) (dnp no)
-    (property "Reference" "#PWR0709" (at 82.55 25.4 0)
-      (effects (font (size 1.27 1.27)) hide)
-    )
-    (property "Value" "+5V" (at 82.55 18.034 0)
-      (effects (font (size 1.27 1.27)))
-    )
-    (property "Footprint" "" (at 82.55 21.59 0)
-      (effects (font (size 1.27 1.27)) hide)
-    )
-    (property "Datasheet" "" (at 82.55 21.59 0)
-      (effects (font (size 1.27 1.27)) hide)
-    )
-    (pin "1")
-    (instances
-      (project "ETH1CSMU2"
-        (path "/1fc6a863-b4aa-4691-87d2-d385f614c99b/e18d2576-cacb-49ee-98d9-d91c481fdd25"
-          (reference "#PWR0709") (unit 1)
-        )
-      )
-      (project "ETH1CFGEN1"
-        (path "/44bc1157-6d68-4ab3-afc0-b8d9f089cc50/064703a1-ee1f-4a0b-949a-89ec1ae8066a"
-          (reference "#PWR0409") (unit 1)
-        )
-      )
     )
   )
@@
     )
   )
-  (symbol (lib_id "power:+5V") (at 110.49 66.04 0) (unit 1)
-    (in_bom yes) (on_board yes) (dnp no)
-    (property "Reference" "#PWR0714" (at 110.49 69.85 0)
-      (effects (font (size 1.27 1.27)) hide)
-    )
-    (property "Value" "+5V" (at 110.49 62.484 0)
-      (effects (font (size 1.27 1.27)))
-    )
-    (property "Footprint" "" (at 110.49 66.04 0)
-      (effects (font (size 1.27 1.27)) hide)
-    )
-    (property "Datasheet" "" (at 110.49 66.04 0)
-      (effects (font (size 1.27 1.27)) hide)
-    )
-    (pin "1")
-    (instances
-      (project "ETH1CSMU2"
-        (path "/1fc6a863-b4aa-4691-87d2-d385f614c99b/e18d2576-cacb-49ee-98d9-d91c481fdd25"
-          (reference "#PWR0714") (unit 1)
-        )
-      )
-      (project "ETH1CFGEN1"
-        (path "/44bc1157-6d68-4ab3-afc0-b8d9f089cc50/064703a1-ee1f-4a0b-949a-89ec1ae8066a"
-          (reference "#PWR0414") (unit 1)
-        )
-      )
-    )
-  )
   (symbol (lib_id "power:GNDD") (at 57.15 34.29 0) (unit 1)
     (in_bom yes) (on_board yes) (dnp no)
@@
         (path "/44bc1157-6d68-4ab3-afc0-b8d9f089cc50/064703a1-ee1f-4a0b-949a-89ec1ae8066a"
           (reference "C403") (unit 1)
-        )
-      )
-    )
-  )
-  (symbol (lib_id "power:+5V") (at 81.28 63.5 0) (unit 1)
-    (in_bom yes) (on_board yes) (dnp no)
-    (property "Reference" "#PWR0708" (at 81.28 67.31 0)
-      (effects (font (size 1.27 1.27)) hide)
-    )
-    (property "Value" "+5V" (at 81.28 59.944 0)
-      (effects (font (size 1.27 1.27)))
-    )
-    (property "Footprint" "" (at 81.28 63.5 0)
-      (effects (font (size 1.27 1.27)) hide)
-    )
-    (property "Datasheet" "" (at 81.28 63.5 0)
-      (effects (font (size 1.27 1.27)) hide)
-    )
-    (pin "1")
-    (instances
-      (project "ETH1CSMU2"
-        (path "/1fc6a863-b4aa-4691-87d2-d385f614c99b/e18d2576-cacb-49ee-98d9-d91c481fdd25"
-          (reference "#PWR0708") (unit 1)
-        )
-      )
-      (project "ETH1CFGEN1"
-        (path "/44bc1157-6d68-4ab3-afc0-b8d9f089cc50/064703a1-ee1f-4a0b-949a-89ec1ae8066a"
-          (reference "#PWR0408") (unit 1)
         )
       )
@@
     )
   )
+  (symbol (lib_id "power:+5VD") (at 100.33 21.59 0) (unit 1)
+    (in_bom yes) (on_board yes) (dnp no)
+    (property "Reference" "#PWR0607" (at 100.33 25.4 0)
+      (effects (font (size 1.27 1.27)) hide)
+    )
+    (property "Value" "+5VD" (at 100.33 17.145 0)
+      (effects (font (size 1.27 1.27)))
+    )
+    (property "Footprint" "" (at 100.33 21.59 0)
+      (effects (font (size 1.27 1.27)) hide)
+    )
+    (property "Datasheet" "" (at 100.33 21.59 0)
+      (effects (font (size 1.27 1.27)) hide)
+    )
+    (pin "1")
+    (instances
+      (project "ETH1CFGEN1"
+        (path "/44bc1157-6d68-4ab3-afc0-b8d9f089cc50/61e965c1-e946-4500-a63b-fb711a3a2ae7"
+          (reference "#PWR0607") (unit 1)
+        )
+        (path "/44bc1157-6d68-4ab3-afc0-b8d9f089cc50/064703a1-ee1f-4a0b-949a-89ec1ae8066a"
+          (reference "#PWR0414") (unit 1)
+        )
+      )
+    )
+  )
   (symbol (lib_id "Device:C") (at 123.19 27.94 0) (unit 1)
     (in_bom yes) (on_board yes) (dnp no)
@@
         (path "/44bc1157-6d68-4ab3-afc0-b8d9f089cc50/064703a1-ee1f-4a0b-949a-89ec1ae8066a"
           (reference "#PWR0413") (unit 1)
-        )
-      )
-    )
-  )
-  (symbol (lib_id "power:+5V") (at 100.33 21.59 0) (unit 1)
-    (in_bom yes) (on_board yes) (dnp no)
-    (property "Reference" "#PWR0711" (at 100.33 25.4 0)
-      (effects (font (size 1.27 1.27)) hide)
-    )
-    (property "Value" "+5V" (at 100.33 18.034 0)
-      (effects (font (size 1.27 1.27)))
-    )
-    (property "Footprint" "" (at 100.33 21.59 0)
-      (effects (font (size 1.27 1.27)) hide)
-    )
-    (property "Datasheet" "" (at 100.33 21.59 0)
-      (effects (font (size 1.27 1.27)) hide)
-    )
-    (pin "1")
-    (instances
-      (project "ETH1CSMU2"
-        (path "/1fc6a863-b4aa-4691-87d2-d385f614c99b/e18d2576-cacb-49ee-98d9-d91c481fdd25"
-          (reference "#PWR0711") (unit 1)
-        )
-      )
-      (project "ETH1CFGEN1"
-        (path "/44bc1157-6d68-4ab3-afc0-b8d9f089cc50/064703a1-ee1f-4a0b-949a-89ec1ae8066a"
-          (reference "#PWR0411") (unit 1)
         )
       )
@@
     )
   )
+  (symbol (lib_id "power:+5VD") (at 110.49 66.04 0) (unit 1)
+    (in_bom yes) (on_board yes) (dnp no)
+    (property "Reference" "#PWR0607" (at 110.49 69.85 0)
+      (effects (font (size 1.27 1.27)) hide)
+    )
+    (property "Value" "+5VD" (at 110.49 61.595 0)
+      (effects (font (size 1.27 1.27)))
+    )
+    (property "Footprint" "" (at 110.49 66.04 0)
+      (effects (font (size 1.27 1.27)) hide)
+    )
+    (property "Datasheet" "" (at 110.49 66.04 0)
+      (effects (font (size 1.27 1.27)) hide)
+    )
+    (pin "1")
+    (instances
+      (project "ETH1CFGEN1"
+        (path "/44bc1157-6d68-4ab3-afc0-b8d9f089cc50/61e965c1-e946-4500-a63b-fb711a3a2ae7"
+          (reference "#PWR0607") (unit 1)
+        )
+        (path "/44bc1157-6d68-4ab3-afc0-b8d9f089cc50/064703a1-ee1f-4a0b-949a-89ec1ae8066a"
+          (reference "#PWR0408") (unit 1)
+        )
+      )
+    )
+  )
   (symbol (lib_id "Device:D_TVS") (at 246.38 142.24 90) (mirror x) (unit 1)
     (in_bom yes) (on_board yes) (dnp no)
@@
         (path "/44bc1157-6d68-4ab3-afc0-b8d9f089cc50/064703a1-ee1f-4a0b-949a-89ec1ae8066a"
           (reference "D403") (unit 1)
+        )
+      )
+    )
+  )
+  (symbol (lib_id "power:+5VD") (at 81.28 63.5 0) (unit 1)
+    (in_bom yes) (on_board yes) (dnp no)
+    (property "Reference" "#PWR0607" (at 81.28 67.31 0)
+      (effects (font (size 1.27 1.27)) hide)
+    )
+    (property "Value" "+5VD" (at 81.28 59.055 0)
+      (effects (font (size 1.27 1.27)))
+    )
+    (property "Footprint" "" (at 81.28 63.5 0)
+      (effects (font (size 1.27 1.27)) hide)
+    )
+    (property "Datasheet" "" (at 81.28 63.5 0)
+      (effects (font (size 1.27 1.27)) hide)
+    )
+    (pin "1")
+    (instances
+      (project "ETH1CFGEN1"
+        (path "/44bc1157-6d68-4ab3-afc0-b8d9f089cc50/61e965c1-e946-4500-a63b-fb711a3a2ae7"
+          (reference "#PWR0607") (unit 1)
+        )
+        (path "/44bc1157-6d68-4ab3-afc0-b8d9f089cc50/064703a1-ee1f-4a0b-949a-89ec1ae8066a"
+          (reference "#PWR0432") (unit 1)
         )
       )
@@
         )
       )
+    )
+  )
+  (symbol (lib_id "power:+5VD") (at 82.55 21.59 0) (unit 1)
+    (in_bom yes) (on_board yes) (dnp no)
+    (property "Reference" "#PWR0607" (at 82.55 25.4 0)
+      (effects (font (size 1.27 1.27)) hide)
+    )
+    (property "Value" "+5VD" (at 82.55 17.145 0)
+      (effects (font (size 1.27 1.27)))
+    )
+    (property "Footprint" "" (at 82.55 21.59 0)
+      (effects (font (size 1.27 1.27)) hide)
+    )
+    (property "Datasheet" "" (at 82.55 21.59 0)
+      (effects (font (size 1.27 1.27)) hide)
+    )
+    (pin "1")
+    (instances
+      (project "ETH1CFGEN1"
+        (path "/44bc1157-6d68-4ab3-afc0-b8d9f089cc50/61e965c1-e946-4500-a63b-fb711a3a2ae7"
+          (reference "#PWR0607") (unit 1)
+        )
+        (path "/44bc1157-6d68-4ab3-afc0-b8d9f089cc50/064703a1-ee1f-4a0b-949a-89ec1ae8066a"
+          (reference "#PWR0409") (unit 1)
+        )
+      )
