File: hardware/ETH1CFGEN1/MCU.kicad_sch (KiCad schematic)
At the start: 42 parts, among them J1001 Conn_02x01, J1002 20021111-00010T4LF, U1001 HDC1080, U1002 STM32F746ZG, U1003 24LC08B-E/MS, Y1001 NX5032GA-16.000M

Commit message: Development
Parts:
- removed C1001, C1002, C1004, C1007, C1009, C1011, C1012, C1013, C1014, C1015, C1016, C1017, C1018, C1019, C1020: 100n, Capacitor_SMD:C_0603_1608Metric_Pad1.08x0.95mm_HandSolder, symbol Device:C
- removed C1010: 1u, Capacitor_SMD:C_0603_1608Metric_Pad1.08x0.95mm_HandSolder, symbol Device:C
- removed R1009: 10k, Resistor_SMD:R_0603_1608Metric_Pad0.98x0.95mm_HandSolder, symbol Device:R
- removed U1002: STM32F746ZG, ETH1CFGEN1:TQFP-144_20x20mm_P0.5mm, symbol ETH1CFGEN1:STM32F746ZG
- added C1021 (x12), C221, C222: 100n, Capacitor_SMD:C_0603_1608Metric_Pad1.08x0.95mm_HandSolder, symbol Device:C
- added C1021 (x2): 1u, Capacitor_SMD:C_0603_1608Metric_Pad1.08x0.95mm_HandSolder, symbol Device:C
- added R206: 10k, Resistor_SMD:R_0603_1608Metric_Pad0.98x0.95mm_HandSolder, symbol Device:R
- added U201: STM32H723ZGTx, Package_QFP:LQFP-144_20x20mm_P0.5mm, symbol MCU_ST_STM32H7:STM32H723ZGTx
Connections:
- net SENS_SCL is gone; now on net I2C1_SCL: R1004.2, U1001.6 (SCL)
- net SENS_SDA is gone; now on net I2C1_SDA: R1006.2, U1001.1 (SDA)
- net +3.3V: now also C1021.1, C1021.1, C1021.1, C1021.1, C1021.1, C1021.1, C1021.1, C1021.1, C1021.1, C1021.1, C1021.1, C1021.1, C1021.1, C221.2, C222.2, U201.108 (VDD), U201.121 (VDD), U201.131 (VDD), U201.143 (PDR_ON), U201.144 (VDD), U201.17 (VDD), U201.30 (VDD), U201.39 (VDD), U201.52 (VDD), U201.6 (VBAT), U201.62 (VDD), U201.72 (VDD), U201.84 (VDD), U201.95 (VDD33USB)
- net CXN_REL1: now also U201.88 (PG3)
- net CXN_REL2: now also U201.89 (PG4)
- net CXN_REL3: now also U201.90 (PG5)
- net CXN_REL4: now also U201.91 (PG6)
- net CXN_REL5: now also U201.92 (PG7)
- net CXN_REL6: now also U201.93 (PG8)
- net EEPROM_WP: now also U201.135 (PB5)
- net GNDD: now also C1021.2, C1021.2, C1021.2, C1021.2, C1021.2, C1021.2, C1021.2, C1021.2, C1021.2, C1021.2, C1021.2, C1021.2, C1021.2, C1021.2, C221.1, C222.1, R206.1, U201.107 (VSS), U201.120 (VSS), U201.130 (VSS), U201.16 (VSS), U201.31 (VSSA), U201.38 (VSS), U201.51 (VSS), U201.61 (VSS), U201.83 (VSS), U201.94 (VSS)
- net LED_BLUE: now also U201.142 (PE1)
- net LED_GREEN: now also U201.46 (PB0)
- net LED_RED: now also U201.75 (PB14)
- net MCU_DEFAULT: now also U201.76 (PB15)
- net NRST: now also U201.25 (NRST)
- net REF_CLK: now also U201.35 (PA1)
- net RMII_CRS_DV: now also U201.43 (PA7)
- net RMII_MDC: now also U201.27 (PC1)
- net RMII_MDIO: now also U201.36 (PA2)
- net RMII_RXD0: now also U201.44 (PC4)
- net RMII_RXD1: now also U201.45 (PC5)
- net RMII_TXD0: now also U201.128 (PG13)
- net RMII_TXD1: now also U201.74 (PB13)
- net RMII_TXEN: now also U201.126 (PG11)
- net TCK_SWCLK: now also U201.109 (PA14(JTCK)
- net TMS_SWDIO: now also U201.105 (PA13(JTMS)
- net TRIG_EN: now also U201.102 (PA10)
- net TRIG_IN: now also U201.100 (PA8)
- net TRIG_OUT: now also U201.101 (PA9)
- net at C1003.1, Y1001.1: now also U201.23 (PH0)
- net at C1005.1, Y1001.2: now also U201.24 (PH1)
- net at C1006.1: now also U201.71 (VCAP)
- net at C1008.1: now also U201.106 (VCAP)
- net I2C_SCL renamed I2C1_SCL
- net I2C1_SCL: now also U201.136 (PB6)
- net I2C_SDA renamed I2C1_SDA
- net I2C1_SDA: now also U201.137 (PB7)
- net MCU_VDDA renamed VDDA
- net VDDA: now also C1021.1, U201.32 (VREF+), U201.33 (VDDA)
- new net: R206.2, U201.138 (BOOT0)
- new net I2C2_SCL: U201.11 (PF1)
- new net I2C2_SDA: U201.10 (PF0)
- new net SPI2_CLK: U201.79 (PD10)
- new net SPI2_CS: U201.73 (PB12)
- new net SPI2_MISO: U201.28 (PC2_C)
- new net SPI2_MOSI: U201.29 (PC3_C)
- no-connect marks 83 -> 7
Other:
- note added: "Connect to VBAT"
- moved on the sheet: C1021, D1001, D1002, D1003, FB1001, J1002, R1001, R1003, R1004, R1005, R1006, R1007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

Commit message: PCB design
Parts:
- U201: footprint Package_QFP:LQFP-144_20x20mm_P0.5mm -> ETH1CFGEN1:TQFP-144_20x20mm_P0.5mm

Commit message: PCB design
Parts:
- C1021: value 1u -> 100n

Commit message: PCB design
Parts:
- C1021: value 100n -> 1u
Connections:
- net SPI2_CLK renamed MCU_SPI2_CLK
- net SPI2_CS renamed MCU_SPI2_CS
- net SPI2_MISO renamed MCU_SPI2_MISO
- net SPI2_MOSI renamed MCU_SPI2_MOSI

Commit message: PCB design
Connections:
- net CXN_REL1: now also U201.90 (PG5); no longer U201.88 (PG3)
- net CXN_REL3: now also U201.88 (PG3); no longer U201.90 (PG5)
- net CXN_REL4: now also U201.87 (PG2); no longer U201.91 (PG6)
- net CXN_REL5: now also U201.86 (PD15); no longer U201.92 (PG7)
- net CXN_REL6: now also U201.85 (PD14); no longer U201.93 (PG8)
- net LED_BLUE: now also U201.15 (PF5); no longer U201.142 (PE1)
- net LED_GREEN: now also U201.13 (PF3); no longer U201.46 (PB0)
- net LED_RED: now also U201.14 (PF4); no longer U201.75 (PB14)
- net TRIG_EN: now also U201.82 (PD13); no longer U201.102 (PA10)
- net TRIG_IN: now also U201.80 (PD11); no longer U201.100 (PA8)
- net TRIG_OUT: now also U201.81 (PD12); no longer U201.101 (PA9)

Commit message: PCB design
Connections:
- net MCU_DEFAULT: now also U201.66 (PE13); no longer U201.76 (PB15)
- net RMII_TXD1: now also U201.129 (PG14); no longer U201.74 (PB13)
- net MCU_SPI_CLK: now reaches U201.111 (PC10)
- net MCU_SPI_MISO: now reaches U201.112 (PC11)
- net MCU_SPI_MOSI: now reaches U201.113 (PC12)
- net MCU_SPI_NSS: now reaches U201.114 (PD0)
- net MCU_SPI2_CLK: no longer names the net of U201.79 (PD10)
- net MCU_SPI2_CS: no longer names the net of U201.73 (PB12)
- net MCU_SPI2_MISO: no longer names the net of U201.28 (PC2_C)
- net MCU_SPI2_MOSI: no longer names the net of U201.29 (PC3_C)

Commit message: Schematic and PCB design
Connections:
- net MCU_GPIO1: now reaches U201.117 (PD3)
- net MCU_GPIO2: now reaches U201.118 (PD4)

Commit message: FPGA code
Connections:
- no-connect marks 7 -> 81
