File: hardware/AD9744_Test/AD9744_Test.kicad_sch (KiCad schematic)
At the start: 35 parts, among them J1 71764-0012, J2 71764-0012, J3 Conn_01x01, J4 Conn_01x01, U1 AD9744, U2 AD8041, X1 SG5032CAN 50.000000M-TJGA3

Commit message: Development
Parts:
- FB1, FB2: value MMZ1005S800HTD25 -> 80
Changed lines of the file:
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@@
   (symbol (lib_id "Device:FerriteBead_Small") (at 102.235 29.21 90) (unit 1)
     (in_bom yes) (on_board yes) (dnp no) (fields_autoplaced)
-    (property "Reference" "FB2" (at 102.1969 22.225 90)
-      (effects (font (size 1.27 1.27)))
-    )
-    (property "Value" "MMZ1005S800HTD25" (at 102.1969 24.765 90)
+    (property "Reference" "FB2" (at 102.1969 22.86 90)
+      (effects (font (size 1.27 1.27)))
+    )
+    (property "Value" "80" (at 102.1969 25.4 90)
       (effects (font (size 1.27 1.27)))
     )
@@
       (effects (font (size 1.27 1.27)))
     )
-    (property "Value" "MMZ1005S800HTD25" (at 44.4119 35.56 90)
-      (effects (font (size 1.27 1.27)))
-    )
+    (property "Value" "80" (at 44.4119 35.56 90)
+      (effects (font (size 1.27 1.27)))
+    )
