File: hardware/ETH1CFGEN1A/WaveformDAC.kicad_sch (KiCad schematic)
At the start: 155 parts, among them K601 G6SU-2F-DC3, K602 G6SU-2F-DC3, Q601 MMBT5087LT1G, U601 AD9744, U602 TL072CD, U603 LT1016CS8, U604 THS3001CD, X1 SG5032CAN 50.000000M-TJGA3

Commit message: Development
Parts:
- renumbered U602 to U601, U601 to U602
