File: hardware/ETH1CFGEN1A/Connector.kicad_sch (KiCad schematic)
At the start: 9 parts, among them J301 C64AC, K301 HE3621A0510, K302 HE3621A0510, K303 HE3621A0510, K304 HE3621A0510, K305 HE3621A0510, K306 HE3621A0510, U301 ULN2003AIDE4

Commit message: Development
Connections:
- net GND_TRIG renamed GND1
Changed lines of the file:
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@@
       (effects (font (size 1.27 1.27)) hide)
     )
-    (property "Value" "+24V" (at 112.395 178.0342 0)
+    (property "Value" "+24V" (at 112.395 178.054 0)
       (effects (font (size 1.27 1.27)))
     )
@@
       (effects (font (size 1.27 1.27)) hide)
     )
-    (property "Value" "+24V" (at 83.7438 179.959 90)
-      (effects (font (size 1.27 1.27)) (justify left))
+    (property "Value" "+24V" (at 81.28 180.34 90)
+      (effects (font (size 1.27 1.27)))
     )
     (property "Footprint" "" (at 86.995 180.34 0)
@@
     )
   )
-  (symbol (lib_id "ETH1CSMU2:GND_TRIG") (at 88.265 102.87 270) (unit 1)
+  (symbol (lib_id "power:GND1") (at 88.265 102.87 270) (unit 1)
     (in_bom yes) (on_board yes) (dnp no)
     (property "Reference" "#PWR0307" (at 81.915 102.87 0)
       (effects (font (size 1.27 1.27)) hide)
     )
-    (property "Value" "GND_TRIG" (at 85.0138 102.997 90)
-      (effects (font (size 1.27 1.27)) (justify right))
+    (property "Value" "GND1" (at 82.55 102.87 90)
+      (effects (font (size 1.27 1.27)))
     )
     (property "Footprint" "" (at 88.265 102.87 0)
@@
       (effects (font (size 1.27 1.27)) hide)
     )
-    (property "Value" "PWR_FLAG" (at 112.395 186.0534 0)
-      (effects (font (size 1.27 1.27)))
-    )
+    (property "Value" "PWR_FLAG" (at 112.395 185.42 0)
+      (effects (font (size 1.27 1.27)))
+    )

Commit message: Development
Parts:
- C301: footprint (none) -> Capacitor_SMD:C_0603_1608Metric_Pad1.08x0.95mm_HandSolder
- J301: footprint (none) -> ETH1CFGEN1:Socket_DIN41612-CaseC1-AC-Male-64Pin-2rows
- K301, K302, K303, K304, K305, K306: footprint (none) -> ETH1CFGEN1:HE360_x-5050462-8
- U301: value ULN2003AIDE4 -> ULN2003AIPWR; footprint (none) -> Package_SO:TSSOP-16_4.4x5mm_P0.65mm
Changed lines of the file:
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@@
       (effects (font (size 1.27 1.27)) (justify left))
     )
-    (property "Footprint" "" (at 120.015 45.72 0)
+    (property "Footprint" "ETH1CFGEN1:HE360_x-5050462-8" (at 120.015 45.72 0)
       (effects (font (size 1.27 1.27)) hide)
     )
@@
       (effects (font (size 1.27 1.27)) (justify left))
     )
-    (property "Footprint" "" (at 97.155 104.14 0)
+    (property "Footprint" "ETH1CFGEN1:Socket_DIN41612-CaseC1-AC-Male-64Pin-2rows" (at 97.155 104.14 0)
       (effects (font (size 1.27 1.27)) hide)
     )
@@
       (effects (font (size 1.27 1.27)) (justify left))
     )
-    (property "Footprint" "" (at 156.845 45.72 0)
+    (property "Footprint" "ETH1CFGEN1:HE360_x-5050462-8" (at 156.845 45.72 0)
       (effects (font (size 1.27 1.27)) hide)
     )
@@
       (effects (font (size 1.27 1.27)) (justify left))
     )
-    (property "Footprint" "" (at 210.185 45.72 0)
+    (property "Footprint" "ETH1CFGEN1:HE360_x-5050462-8" (at 210.185 45.72 0)
       (effects (font (size 1.27 1.27)) hide)
     )
@@
       (effects (font (size 1.27 1.27)))
     )
-    (property "Footprint" "" (at 52.705 50.8 0)
+    (property "Footprint" "ETH1CFGEN1:HE360_x-5050462-8" (at 52.705 50.8 0)
       (effects (font (size 1.27 1.27)) hide)
     )
@@
       (effects (font (size 1.27 1.27)) (justify left))
     )
-    (property "Footprint" "" (at 139.065 45.72 0)
+    (property "Footprint" "ETH1CFGEN1:HE360_x-5050462-8" (at 139.065 45.72 0)
       (effects (font (size 1.27 1.27)) hide)
     )
@@
       (effects (font (size 1.27 1.27)))
     )
-    (property "Footprint" "" (at 52.705 24.13 0)
+    (property "Footprint" "ETH1CFGEN1:HE360_x-5050462-8" (at 52.705 24.13 0)
       (effects (font (size 1.27 1.27)) hide)
     )
@@
       (effects (font (size 1.27 1.27)) (justify left))
     )
-    (property "Footprint" "" (at 192.405 45.72 0)
+    (property "Footprint" "ETH1CFGEN1:HE360_x-5050462-8" (at 192.405 45.72 0)
       (effects (font (size 1.27 1.27)) hide)
     )
@@
       (effects (font (size 1.27 1.27)))
     )
-    (property "Footprint" "" (at 52.705 68.58 0)
+    (property "Footprint" "ETH1CFGEN1:HE360_x-5050462-8" (at 52.705 68.58 0)
       (effects (font (size 1.27 1.27)) hide)
     )
@@
       (effects (font (size 1.27 1.27)))
     )
-    (property "Footprint" "" (at 52.705 33.02 0)
+    (property "Footprint" "ETH1CFGEN1:HE360_x-5050462-8" (at 52.705 33.02 0)
       (effects (font (size 1.27 1.27)) hide)
     )
@@
       (effects (font (size 1.27 1.27)))
     )
-    (property "Footprint" "" (at 52.705 59.69 0)
+    (property "Footprint" "ETH1CFGEN1:HE360_x-5050462-8" (at 52.705 59.69 0)
       (effects (font (size 1.27 1.27)) hide)
     )
@@
       (effects (font (size 1.27 1.27)) (justify left))
     )
-    (property "Footprint" "" (at 174.625 45.72 0)
+    (property "Footprint" "ETH1CFGEN1:HE360_x-5050462-8" (at 174.625 45.72 0)
       (effects (font (size 1.27 1.27)) hide)
     )
@@
       (effects (font (size 1.27 1.27)))
     )
-    (property "Footprint" "" (at 52.705 41.91 0)
+    (property "Footprint" "ETH1CFGEN1:HE360_x-5050462-8" (at 52.705 41.91 0)
       (effects (font (size 1.27 1.27)) hide)
     )
@@
       (effects (font (size 1.27 1.27)) (justify left))
     )
-    (property "Footprint" "" (at 273.3802 57.15 0)
+    (property "Footprint" "Capacitor_SMD:C_0603_1608Metric_Pad1.08x0.95mm_HandSolder" (at 273.3802 57.15 0)
       (effects (font (size 1.27 1.27)) hide)
     )
@@
       (effects (font (size 1.27 1.27)))
     )
-    (property "Value" "ULN2003AIDE4" (at 239.395 39.9796 0)
-      (effects (font (size 1.27 1.27)))
-    )
-    (property "Footprint" "" (at 238.125 68.58 0)
+    (property "Value" "ULN2003AIPWR" (at 239.395 39.9796 0)
+      (effects (font (size 1.27 1.27)))
+    )
+    (property "Footprint" "Package_SO:TSSOP-16_4.4x5mm_P0.65mm" (at 238.125 68.58 0)
       (effects (font (size 1.27 1.27)) (justify left) hide)
     )
