File: hardware/ETH1CFGEN1A/Ethernet.kicad_sch (KiCad schematic)
At the start: 43 parts, among them U201 LAN8742A, U202 LC03-3.3, U203 LC03-3.3, Y201 NX5032GA-25.000000MHZ-LN-CD-1

Commit message: Development
Parts:
- C206, C207: footprint Capacitor_SMD:C_0603_1608Metric_Pad1.08x0.95mm_HandSolder -> (none)
- C213, C214: footprint Capacitor_SMD:C_1206_3216Metric_Pad1.33x1.80mm_HandSolder -> (none)
- FB201: footprint Inductor_SMD:L_0805_2012Metric_Pad1.15x1.40mm_HandSolder -> (none)
- L201: footprint ETH1CSMU2:749010012A -> (none); symbol ETH1CSMU2:749010012A -> ETH1CFGEN1:749010012A
- R219: footprint Resistor_SMD:R_1206_3216Metric_Pad1.30x1.75mm_HandSolder -> (none)
- U201: footprint Package_DFN_QFN:QFN-24-1EP_4x4mm_P0.5mm_EP2.6x2.6mm_ThermalVias -> (none)
- U202, U203: footprint ETH1CSMU2:SO8E -> (none); symbol ETH1CSMU2:LC03-3.3 -> ETH1CFGEN1:LC03-3.3
- Y201: footprint ETH1CSMU2:NX5032GA -> (none)
Connections:
- net GND renamed GNDD

Commit message: Development
Parts:
- FB201: symbol Device:Ferrite_Bead -> Device:FerriteBead
- U201: value LAN8742A -> LAN8742; footprint (none) -> Package_DFN_QFN:QFN-24-1EP_4x4mm_P0.5mm_EP2.6x2.6mm; symbol ETH1CSMU2:LAN8742 -> ETH1CFGEN1:LAN8742
Changed lines of the file:
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@@
       (effects (font (size 1.27 1.27)) hide)
     )
-    (property "Value" "PWR_FLAG" (at 21.59 191.0842 0)
+    (property "Value" "PWR_FLAG" (at 21.59 190.5 0)
       (effects (font (size 1.27 1.27)))
     )
@@
       (effects (font (size 1.27 1.27)) hide)
     )
-    (property "Value" "PWR_FLAG" (at 33.02 191.0842 0)
+    (property "Value" "PWR_FLAG" (at 33.02 190.5 0)
       (effects (font (size 1.27 1.27)))
     )
@@
       (effects (font (size 1.27 1.27)) hide)
     )
-    (property "Value" "VCCQ" (at 22.0218 182.2958 0)
+    (property "Value" "VCCQ" (at 21.59 182.88 0)
       (effects (font (size 1.27 1.27)))
     )
@@
       (effects (font (size 1.27 1.27)) hide)
     )
-    (property "Value" "+3.3V" (at 53.34 21.8242 0)
+    (property "Value" "+3.3V" (at 53.34 21.844 0)
       (effects (font (size 1.27 1.27)))
     )
@@
     )
   )
-  (symbol (lib_id "ETH1CSMU2:LAN8742") (at 86.36 86.36 0) (unit 1)
-    (in_bom yes) (on_board yes) (dnp no)
-    (property "Reference" "U201" (at 69.85 57.15 0)
-      (effects (font (size 1.27 1.27)))
-    )
-    (property "Value" "LAN8742A" (at 96.52 57.15 0)
-      (effects (font (size 1.27 1.27)))
-    )
-    (property "Footprint" "" (at 87.63 113.03 0)
+  (symbol (lib_id "ETH1CFGEN1:LAN8742") (at 86.36 86.36 0) (unit 1)
+    (in_bom yes) (on_board yes) (dnp no)
+    (property "Reference" "U201" (at 99.695 54.61 0)
+      (effects (font (size 1.27 1.27)) (justify right))
+    )
+    (property "Value" "LAN8742" (at 101.6 57.15 0)
+      (effects (font (size 1.27 1.27)) (justify right))
+    )
+    (property "Footprint" "Package_DFN_QFN:QFN-24-1EP_4x4mm_P0.5mm_EP2.6x2.6mm" (at 87.63 113.03 0)
       (effects (font (size 1.27 1.27)) (justify left) hide)
     )
@@
     )
   )
-  (symbol (lib_id "Device:Ferrite_Bead") (at 86.36 26.67 270) (unit 1)
-    (in_bom yes) (on_board yes) (dnp no)
-    (property "Reference" "FB201" (at 86.36 19.7104 90)
-      (effects (font (size 1.27 1.27)))
-    )
-    (property "Value" "742792031" (at 86.36 22.0218 90)
+  (symbol (lib_id "Device:FerriteBead") (at 86.36 26.67 270) (unit 1)
+    (in_bom yes) (on_board yes) (dnp no)
+    (property "Reference" "FB201" (at 86.36 19.685 90)
+      (effects (font (size 1.27 1.27)))
+    )
+    (property "Value" "742792031" (at 86.36 22.225 90)
       (effects (font (size 1.27 1.27)))
     )
@@
       (effects (font (size 1.27 1.27)) hide)
     )
-    (property "Value" "PWR_FLAG" (at 47.5742 44.45 90)
-      (effects (font (size 1.27 1.27)) (justify left))
+    (property "Value" "PWR_FLAG" (at 46.99 44.45 0)
+      (effects (font (size 1.27 1.27)))
     )
     (property "Footprint" "" (at 50.8 44.45 0)
@@
       (effects (font (size 1.27 1.27)) hide)
     )
-    (property "Value" "VCCQ" (at 197.2818 21.0058 0)
+    (property "Value" "VCCQ" (at 196.85 21.59 0)
       (effects (font (size 1.27 1.27)))
     )
@@
       (effects (font (size 1.27 1.27)) hide)
     )
-    (property "Value" "+3.3V" (at 71.501 164.5158 0)
-      (effects (font (size 1.27 1.27)))
-    )
+    (property "Value" "+3.3V" (at 71.12 165.354 0)
+      (effects (font (size 1.27 1.27)))
+    )

Commit message: Development
Parts:
- C206, C207: footprint (none) -> Capacitor_SMD:C_0603_1608Metric_Pad1.08x0.95mm_HandSolder
- C213, C214: footprint (none) -> Capacitor_SMD:C_1206_3216Metric_Pad1.33x1.80mm_HandSolder
- FB201: footprint (none) -> Inductor_SMD:L_0805_2012Metric_Pad1.05x1.20mm_HandSolder
- L201: footprint (none) -> ETH1CFGEN1:749010012A
- R219: footprint (none) -> Resistor_SMD:R_1206_3216Metric_Pad1.30x1.75mm_HandSolder
- U202, U203: value LC03-3.3 -> LC03-3.3BTG; footprint (none) -> Package_SO:SOIC-8_3.9x4.9mm_P1.27mm
- Y201: footprint (none) -> ETH1CFGEN1:NX5032GA
Changed lines of the file:
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@@
       (effects (font (size 1.27 1.27)))
     )
-    (property "Footprint" "" (at 234.95 74.93 0)
+    (property "Footprint" "ETH1CFGEN1:749010012A" (at 234.95 74.93 0)
       (effects (font (size 1.27 1.27)) hide)
     )
@@
       (effects (font (size 1.27 1.27)))
     )
-    (property "Footprint" "" (at 209.55 112.522 90)
+    (property "Footprint" "Resistor_SMD:R_1206_3216Metric_Pad1.30x1.75mm_HandSolder" (at 209.55 112.522 90)
       (effects (font (size 1.27 1.27)) hide)
     )
@@
       (effects (font (size 1.27 1.27)))
     )
-    (property "Footprint" "" (at 205.74 125.4252 0)
+    (property "Footprint" "Capacitor_SMD:C_1206_3216Metric_Pad1.33x1.80mm_HandSolder" (at 205.74 125.4252 0)
       (effects (font (size 1.27 1.27)) hide)
     )
@@
       (effects (font (size 1.27 1.27)) (justify left))
     )
-    (property "Footprint" "" (at 93.6752 35.56 0)
+    (property "Footprint" "Capacitor_SMD:C_0603_1608Metric_Pad1.08x0.95mm_HandSolder" (at 93.6752 35.56 0)
       (effects (font (size 1.27 1.27)) hide)
     )
@@
       (effects (font (size 1.524 1.524)))
     )
-    (property "Value" "LC03-3.3" (at 262.89 63.9826 0)
+    (property "Value" "LC03-3.3BTG" (at 262.89 63.9826 0)
       (effects (font (size 1.524 1.524)))
     )
-    (property "Footprint" "" (at 262.89 72.39 0)
+    (property "Footprint" "Package_SO:SOIC-8_3.9x4.9mm_P1.27mm" (at 262.89 72.39 0)
       (effects (font (size 1.524 1.524)) hide)
     )
@@
       (effects (font (size 1.524 1.524)))
     )
-    (property "Value" "LC03-3.3" (at 262.89 84.3026 0)
+    (property "Value" "LC03-3.3BTG" (at 262.89 84.3026 0)
       (effects (font (size 1.524 1.524)))
     )
-    (property "Footprint" "" (at 262.89 92.71 0)
+    (property "Footprint" "Package_SO:SOIC-8_3.9x4.9mm_P1.27mm" (at 262.89 92.71 0)
       (effects (font (size 1.524 1.524)) hide)
     )
@@
       (effects (font (size 1.27 1.27)))
     )
-    (property "Footprint" "" (at 86.36 24.892 90)
+    (property "Footprint" "Inductor_SMD:L_0805_2012Metric_Pad1.05x1.20mm_HandSolder" (at 86.36 24.892 90)
       (effects (font (size 1.27 1.27)) hide)
     )
@@
       (effects (font (size 1.27 1.27)) (justify left))
     )
-    (property "Footprint" "" (at 65.7352 53.34 0)
+    (property "Footprint" "Capacitor_SMD:C_0603_1608Metric_Pad1.08x0.95mm_HandSolder" (at 65.7352 53.34 0)
       (effects (font (size 1.27 1.27)) hide)
     )
@@
       (effects (font (size 1.27 1.27)) (justify left))
     )
-    (property "Footprint" "" (at 229.5652 111.76 0)
+    (property "Footprint" "Capacitor_SMD:C_1206_3216Metric_Pad1.33x1.80mm_HandSolder" (at 229.5652 111.76 0)
       (effects (font (size 1.27 1.27)) hide)
     )
@@
       (effects (font (size 1.27 1.27)))
     )
-    (property "Footprint" "" (at 44.45 120.65 0)
-      (effects (font (size 1.27 1.27)) hide)
-    )
+    (property "Footprint" "ETH1CFGEN1:NX5032GA" (at 44.45 120.65 0)
+      (effects (font (size 1.27 1.27)) hide)
+    )
