File: hardware/ETH1CFGEN1A/FPGA.kicad_sch (KiCad schematic)
At the start: 46 parts, among them J501 Conn_01x06, J502 Conn_02x07_Odd_Even, U503 XC6SLX9-TQG144, U504 W25Q64JV, X501 ASFL1-100.000MHZ-L-T

Commit message: Development
Parts:
- C501, C502, C503, C504, C505, C507, C508, C509, C510, C511, C512, C514, C515, C516, C517, C518, C519, C520, C521, C522, C523, C524, C525, C526, C527, C528, C529: value 0.1u -> 100n; footprint (none) -> Capacitor_SMD:C_0603_1608Metric_Pad1.08x0.95mm_HandSolder
- D501: footprint (none) -> LED_SMD:LED_0603_1608Metric_Pad1.05x0.95mm_HandSolder
- R501, R502, R503, R504, R505, R506, R507, R508, R509: footprint (none) -> Resistor_SMD:R_0603_1608Metric_Pad0.98x0.95mm_HandSolder
- U503: value XC6SLX9-TQG144 -> XC6SLX9-3TQG144I; footprint (none) -> ETH1CFGEN1:TQFP-144_20x20mm_P0.5mm
