File: hardware/ETH1CFGEN1A/MCU.kicad_sch (KiCad schematic)
At the start: 42 parts, among them J1001 Conn_02x01, J1002 20021111-00010T4LF, U1001 HDC1080, U1002 STM32F746ZG, U1003 24LC08B-E/MS, Y1001 NX5032GA-16.000M

Commit message: Development
Parts:
- C1006, C1008, C1010, C1021: footprint Capacitor_SMD:C_0603_1608Metric_Pad1.08x0.95mm_HandSolder -> (none)
- FB1001: footprint Inductor_SMD:L_0805_2012Metric_Pad1.15x1.40mm_HandSolder -> (none)
- J1001: footprint Connector_PinHeader_2.54mm:PinHeader_1x02_P2.54mm_Vertical -> (none)
- J1002: footprint Connector_PinHeader_1.27mm:PinHeader_2x05_P1.27mm_Vertical -> (none)
- U1001: footprint Package_SON:Texas_PWSON-N6 -> (none)
- U1002: value STM32F746ZG -> STM32H743ZI; footprint ETH1CSMU2:TQFP-144_20x20mm_P0.5mm -> (none)
- U1003: footprint Package_SO:MSOP-8_3x3mm_P0.65mm -> (none)
- Y1001: footprint ETH1CSMU2:NX3225GD -> (none)
Connections:
- net SPI2_MISO is gone; now on net TRIG_OUT: U1002.75 (PB14,TIM1_CH2N,TIM8_CH2N,USART1_TX,SPI2_MISO,DFSDM1_DATIN2,USART3_RTS,UART4_RTS,TIM12_CH1,SDMMC2_D0,OTG_HS_DM,EVENTOUT)
- net SPI2_MOSI is gone; now on net TRIG_EN: U1002.76 (PB15,RTC_REFIN,TIM1_CH3N,TIM8_CH3N,USART1_RX,SPI2_MOSI,I2S2_SD,DFSDM1_CKIN2,UART4_CTS,TIM12_CH2,SDMMC2_D1,OTG_HS_DP,EVENTOUT)
- net SPI2_SCK is gone; now on net TRIG_IN: U1002.74 (PB13,TIM1_CH1N,SPI2_SCK,I2S2_CK,DFSDM1_CKIN1,USART3_CTS,UART5_TX,CAN2_TX,OTG_HS_ULPI_D6,ETH_MII_TXD1,ETH_RMII_TXD1,EVENTOUT,OTG_HS_VBUS)
- net TRIG_EN: no longer U1002.60 (PE9,TIM1_CH1,DFSDM1_CKOUT,UART7_RTS,QUADSPI_BK2_IO2,FMC_D6,EVENTOUT)
- net TRIG_IN: no longer U1002.58 (PE7,TIM1_ETR,DFSDM1_DATIN2,UART7_RX,QUADSPI_BK2_IO0,FMC_D4,EVENTOUT)
- net TRIG_OUT: no longer U1002.59 (PE8,TIM1_CH1N,DFSDM1_CKIN2,UART7_TX,QUADSPI_BK2_IO1,FMC_D5,EVENTOUT)
- net GPIO1: now reaches U1002.133 (PB3,JTDO,TRACESWO,TIM2_CH2,SPI1_SCK,I2S1_CK,SPI3_SCK,I2S3_CK,SPI6_SCK,SDMMC2_D2,CAN3_RX,UART7_RX,EVENTOUT)
- net GPIO2: now reaches U1002.134 (PB4,NJTRST,TIM3_CH1,SPI1_MISO,SPI3_MISO,SPI2_NSS,I2S2_WS,SPI6_MISO,SDMMC2_D3,CAN3_TX,UART7_TX,EVENTOUT)
- net ADC1_RVS1: no longer names the net of U1002.114 (PD0,DFSDM1_CKIN6,DFSDM1_DATIN7,UART4_RX,CAN1_RX,FMC_D2,EVENTOUT)
- net ADC1_RVS2: no longer names the net of U1002.115 (PD1,DFSDM1_DATIN6,DFSDM1_CKIN7,UART4_TX,CAN1_TX,FMC_D3,EVENTOUT)
- net DAC1_LDAC: no longer names the net of U1002.104 (PA12,TIM1_ETR,SPI2_SCK,I2S2_CK,UART4_TX,USART1_RTS,SAI2_FS_B,CAN1_TX,OTG_FS_DP,LCD_R5,EVENTOUT)
- net DAC1_~{RST}: no longer names the net of U1002.103 (PA11,TIM1_CH4,SPI2_NSS,I2S2_WS,UART4_RX,USART1_CTS,CAN1_RX,OTG_FS_DM,LCD_R4,EVENTOUT)
- net DAC2_~{LDAC}: no longer names the net of U1002.127 (PG12,LPTIM1_IN1,SPI6_MISO,SPDIF_RX1,USART6_RTS,LCD_B4,SDMMC2_D3,FMC_NE4,LCD_B1,EVENTOUT)
- net DAC_OFFS_SCL renamed SENS_SCL
- net SENS_SCL: no longer U1002.100 (PA8,MCO1,TIM1_CH1,TIM8_BKIN2,I2C3_SCL,USART1_CK,OTG_FS_SOF,CAN3_RX,UART7_RX,LCD_B3,LCD_R6,EVENTOUT)
- net DAC_OFFS_SDA renamed SENS_SDA
- net SENS_SDA: no longer U1002.99 (PC9,MCO2,TIM3_CH4,TIM8_CH4,I2C3_SDA,I2S_CKIN,UART5_CTS,QUADSPI_BK1_IO0,LCD_G3,SDMMC1_D1,DCMI_D3,LCD_B2,EVENTOUT)
- net FGEN_DIV2: no longer names the net of U1002.10 (PF0,I2C2_SDA,FMC_A0,EVENTOUT)
- net FGEN_DIV4: no longer names the net of U1002.9 (PC15,EVENTOUT,OSC32_OUT)
- net FGEN_DIV8: no longer names the net of U1002.8 (PC14,EVENTOUT,OSC32_IN)
- net GND renamed GNDD
- net MCU_CURR_SENS_100R: no longer names the net of U1002.91 (PG6,FMC_NE3,DCMI_D12,LCD_R7,EVENTOUT)
- net MCU_CURR_SENS_10R: no longer names the net of U1002.92 (PG7,SAI1_MCLK_A,USART6_CK,FMC_INT,DCMI_D13,LCD_CLK,EVENTOUT)
- net MCU_CURR_SENS_1R: no longer names the net of U1002.93 (PG8,SPI6_NSS,SPDIF_RX2,USART6_RTS,ETH_PPS_OUT,FMC_SDCLK,LCD_G7,EVENTOUT)
- net MCU_CURR_SENS_1kR: no longer names the net of U1002.90 (PG5,FMC_A15,FMC_BA1,EVENTOUT)
- net MCU_nISNK: no longer names the net of U1002.79 (PD10,DFSDM1_CKOUT,USART3_CK,FMC_D15,LCD_B3,EVENTOUT)
- net MCU_nISRC: no longer names the net of U1002.80 (PD11,I2C4_SMBA,USART3_CTS,QUADSPI_BK1_IO0,SAI2_SD_A,FMC_A16,FMC_CLE,EVENTOUT)
- net MCU_nTDS: no longer names the net of U1002.78 (PD9,DFSDM1_DATIN3,USART3_RX,FMC_D14,EVENTOUT)
- net SPI1_NSS renamed SPI1_CS
- net SPI1_SCK renamed SPI1_CLK
- net SPI2_NSS: no longer names the net of U1002.73 (PB12,TIM1_BKIN,I2C2_SMBA,SPI2_NSS,I2S2_WS,DFSDM1_DATIN1,USART3_CK,UART5_RX,CAN2_RX,OTG_HS_ULPI_D5,ETH_MII_TXD0,ETH_RMII_TXD0,OTG_HS_ID,EVENTOUT)
- net SPI3_MISO: no longer names the net of U1002.112 (PC11,DFSDM1_DATIN5,SPI3_MISO,USART3_RX,UART4_RX,QUADSPI_BK2_NCS,SDMMC1_D3,DCMI_D4,EVENTOUT)
- net SPI3_MOSI: no longer names the net of U1002.113 (PC12,TRACED3,SPI3_MOSI,I2S3_SD,USART3_CK,UART5_TX,SDMMC1_CK,DCMI_D9,EVENTOUT)
- net SPI3_NSS: no longer names the net of U1002.110 (PA15,JTDI,TIM2_CH1,TIM2_ETR,HDMI_CEC,SPI1_NSS,I2S1_WS,SPI3_NSS,I2S3_WS,SPI6_NSS,UART4_RTS,CAN3_TX,UART7_TX,EVENTOUT)
- net SPI3_SCK: no longer names the net of U1002.111 (PC10,DFSDM1_CKIN5,SPI3_SCK,I2S3_CK,USART3_TX,UART4_TX,QUADSPI_BK1_IO1,SDMMC1_D2,DCMI_D8,LCD_R2,EVENTOUT)
- net SPI4_MISO: no longer names the net of U1002.4 (PE5,TRACED2,TIM9_CH1,SPI4_MISO,SAI1_SCK_A,DFSDM1_CKIN3,FMC_A21,DCMI_D6,LCD_G0,EVENTOUT)
- net SPI4_MOSI: no longer names the net of U1002.5 (PE6,TRACED3,TIM1_BKIN2,TIM9_CH2,SPI4_MOSI,SAI1_SD_A,SAI2_MCLK_B,FMC_A22,DCMI_D7,LCD_G1,EVENTOUT)
- net SPI4_NSS: no longer names the net of U1002.3 (PE4,TRACED1,SPI4_NSS,SAI1_FS_A,DFSDM1_DATIN3,FMC_A20,DCMI_D4,LCD_B0,EVENTOUT)
- net SPI4_SCK: no longer names the net of U1002.1 (PE2,TRACECLK,SPI4_SCK,SAI1_MCLK_A,QUADSPI_BK1_IO2,ETH_MII_TXD3,FMC_A23,EVENTOUT)
- net SPI5_MISO: no longer names the net of U1002.20 (PF8,SPI5_MISO,SAI1_SCK_B,UART7_RTS,TIM13_CH1,QUADSPI_BK1_IO0,EVENTOUT,ADC3_IN6)
- net SPI5_MOSI: no longer names the net of U1002.21 (PF9,SPI5_MOSI,SAI1_FS_B,UART7_CTS,TIM14_CH1,QUADSPI_BK1_IO1,EVENTOUT,ADC3_IN7)
- net SPI5_NSS: no longer names the net of U1002.18 (PF6,TIM10_CH1,SPI5_NSS,SAI1_SD_B,UART7_RX,QUADSPI_BK1_IO3,EVENTOUT,ADC3_IN4)
- net SPI5_SCK: no longer names the net of U1002.19 (PF7,TIM11_CH1,SPI5_SCK,SAI1_MCLK_B,UART7_TX,QUADSPI_BK1_IO2,EVENTOUT,ADC3_IN5)
- net SR_CLK: no longer names the net of U1002.87 (PG2,FMC_A12,EVENTOUT)
- net SR_DAT: no longer names the net of U1002.88 (PG3,FMC_A13,EVENTOUT)
- net SR_LAT: no longer names the net of U1002.86 (PD15,TIM4_CH4,UART8_RTS,FMC_D1,EVENTOUT)
- net SR_OUT: no longer names the net of U1002.85 (PD14,TIM4_CH3,UART8_CTS,FMC_D0,EVENTOUT)
- net ~{FGEN_DIV10}: no longer names the net of U1002.7 (PC13,EVENTOUT,RTC_TAMP2,RTC_TS,WKUP5)
- no-connect marks 47 -> 83

Commit message: Development
Parts:
- FB1001: symbol Device:Ferrite_Bead -> Device:FerriteBead
- U1001: footprint (none) -> Package_SON:Texas_PWSON-N6
- U1002: value STM32H743ZI -> STM32F746ZG; symbol ETH1CSMU2:STM32F746ZG -> ETH1CFGEN1:STM32F746ZG
Connections:
- net EEPROM_SCL renamed I2C_SCL
- net EEPROM_SDA renamed I2C_SDA
Changed lines of the file:
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@@
     (stroke (width 0) (type default))
   )
-  (wire (pts (xy 372.11 106.68) (xy 398.78 106.68))
+  (wire (pts (xy 372.11 106.68) (xy 391.16 106.68))
     (stroke (width 0) (type default))
   )
@@
     (stroke (width 0) (type default))
   )
-  (wire (pts (xy 372.11 104.14) (xy 398.78 104.14))
+  (wire (pts (xy 372.11 104.14) (xy 391.16 104.14))
     (stroke (width 0) (type default))
   )
@@
     (effects (font (size 1.27 1.27)) (justify right bottom))
   )
-  (label "EEPROM_SCL" (at 398.78 104.14 180) (fields_autoplaced)
+  (label "EEPROM_SCL" (at 391.16 104.14 180) (fields_autoplaced)
     (effects (font (size 1.27 1.27)) (justify right bottom))
   )
@@
     (effects (font (size 1.27 1.27)) (justify right bottom))
   )
-  (label "EEPROM_SDA" (at 398.78 106.68 180) (fields_autoplaced)
+  (label "EEPROM_SDA" (at 391.16 106.68 180) (fields_autoplaced)
     (effects (font (size 1.27 1.27)) (justify right bottom))
+  )
+  (hierarchical_label "I2C_SDA" (shape bidirectional) (at 391.16 106.68 0) (fields_autoplaced)
+    (effects (font (size 1.27 1.27)) (justify left))
   )
   (hierarchical_label "RMII_MDIO" (shape bidirectional) (at 81.28 86.36 180) (fields_autoplaced)
@@
   )
   (hierarchical_label "RMII_TXEN" (shape bidirectional) (at 373.38 58.42 0) (fields_autoplaced)
+    (effects (font (size 1.27 1.27)) (justify left))
+  )
+  (hierarchical_label "I2C_SCL" (shape bidirectional) (at 391.16 104.14 0) (fields_autoplaced)
     (effects (font (size 1.27 1.27)) (justify left))
   )
@@
       (effects (font (size 1.27 1.27)) hide)
     )
-    (property "Value" "+3.3V" (at 227.33 16.7442 0)
+    (property "Value" "+3.3V" (at 227.33 16.764 0)
       (effects (font (size 1.27 1.27)))
     )
@@
       (effects (font (size 1.27 1.27)) hide)
     )
-    (property "Value" "+3.3V" (at 246.761 255.9558 0)
+    (property "Value" "+3.3V" (at 246.38 256.794 0)
       (effects (font (size 1.27 1.27)))
     )
@@
       (effects (font (size 1.27 1.27)) hide)
     )
-    (property "Value" "+3.3V" (at 282.321 249.6058 0)
+    (property "Value" "+3.3V" (at 281.94 250.444 0)
       (effects (font (size 1.27 1.27)))
     )
@@
       (effects (font (size 1.27 1.27)) hide)
     )
-    (property "Value" "+3.3V" (at 94.361 261.0358 0)
+    (property "Value" "+3.3V" (at 93.98 261.874 0)
       (effects (font (size 1.27 1.27)))
     )
@@
       (effects (font (size 1.27 1.27)) hide)
     )
-    (property "Value" "+3.3V" (at 20.701 186.1058 0)
+    (property "Value" "+3.3V" (at 20.32 186.944 0)
       (effects (font (size 1.27 1.27)))
     )
@@
       (effects (font (size 1.27 1.27)) hide)
     )
-    (property "Value" "+3.3V" (at 73.66 220.98 90)
+    (property "Value" "+3.3V" (at 76.454 220.98 0)
       (effects (font (size 1.27 1.27)))
     )
@@
       (effects (font (size 1.27 1.27)) hide)
     )
-    (property "Value" "+3.3V" (at 38.481 146.7358 0)
+    (property "Value" "+3.3V" (at 38.1 147.574 0)
       (effects (font (size 1.27 1.27)))
     )
@@
     )
   )
-  (symbol (lib_id "Device:Ferrite_Bead") (at 175.26 266.7 270) (unit 1)
-    (in_bom yes) (on_board yes) (dnp no)
-    (property "Reference" "FB1001" (at 175.26 259.7404 90)
-      (effects (font (size 1.27 1.27)))
-    )
-    (property "Value" "742792031" (at 175.26 262.0518 90)
+  (symbol (lib_id "Device:FerriteBead") (at 175.26 266.7 270) (unit 1)
+    (in_bom yes) (on_board yes) (dnp no)
+    (property "Reference" "FB1001" (at 175.26 259.715 90)
+      (effects (font (size 1.27 1.27)))
+    )
+    (property "Value" "742792031" (at 175.26 262.255 90)
       (effects (font (size 1.27 1.27)))
     )
@@
       (effects (font (size 1.27 1.27)) hide)
     )
-    (property "Value" "+3.3V" (at 157.861 241.9858 0)
+    (property "Value" "+3.3V" (at 157.48 242.824 0)
       (effects (font (size 1.27 1.27)))
     )
@@
   (symbol (lib_id "Sensor_Humidity:HDC1080") (at 22.86 165.1 0) (unit 1)
     (in_bom yes) (on_board yes) (dnp no)
-    (property "Reference" "U1001" (at 27.94 156.21 0)
-      (effects (font (size 1.27 1.27)) (justify right))
-    )
-    (property "Value" "HDC1080" (at 30.48 158.75 0)
-      (effects (font (size 1.27 1.27)) (justify right))
-    )
-    (property "Footprint" "" (at 21.59 171.45 0)
+    (property "Reference" "U1001" (at 25.4 156.845 0)
+      (effects (font (size 1.27 1.27)))
+    )
+    (property "Value" "HDC1080" (at 25.4 158.75 0)
+      (effects (font (size 1.27 1.27)))
+    )
+    (property "Footprint" "Package_SON:Texas_PWSON-N6" (at 21.59 171.45 0)
       (effects (font (size 1.27 1.27)) (justify left) hide)
     )
@@
       (effects (font (size 1.27 1.27)) hide)
     )
-    (property "Value" "+3.3V" (at 383.921 207.6958 0)
+    (property "Value" "+3.3V" (at 383.54 208.534 0)
       (effects (font (size 1.27 1.27)))
     )
@@
       (effects (font (size 1.27 1.27)) hide)
     )
-    (property "Value" "+3.3V" (at 20.701 150.5458 0)
+    (property "Value" "+3.3V" (at 20.32 151.384 0)
       (effects (font (size 1.27 1.27)))
     )
@@
       (effects (font (size 1.27 1.27)) hide)
     )
-    (property "Value" "+3.3V" (at 199.771 255.9558 0)
+    (property "Value" "+3.3V" (at 199.39 256.794 0)
       (effects (font (size 1.27 1.27)))
     )
@@
     )
   )
-  (symbol (lib_id "ETH1CSMU2:STM32F746ZG") (at 227.33 125.73 0) (unit 1)
-    (in_bom yes) (on_board yes) (dnp no)
-    (property "Reference" "U1002" (at 88.9 26.67 0)
-      (effects (font (size 1.27 1.27)) (justify left))
-    )
-    (property "Value" "STM32H743ZI" (at 353.06 26.67 0)
-      (effects (font (size 1.27 1.27)) (justify left))
+  (symbol (lib_id "ETH1CFGEN1:STM32F746ZG") (at 227.33 125.73 0) (unit 1)
+    (in_bom yes) (on_board yes) (dnp no)
+    (property "Reference" "U1002" (at 90.17 26.67 0)
+      (effects (font (size 1.27 1.27)))
+    )
+    (property "Value" "STM32F746ZG" (at 358.14 26.67 0)
+      (effects (font (size 1.27 1.27)))
     )
     (property "Footprint" "" (at 631.19 87.63 0)
@@
       (effects (font (size 1.27 1.27)) hide)
     )
-    (property "Value" "+3.3V" (at 29.591 228.0158 0)
+    (property "Value" "+3.3V" (at 29.21 228.854 0)
       (effects (font (size 1.27 1.27)))
     )
@@
       (effects (font (size 1.27 1.27)) hide)
     )
-    (property "Value" "+3.3V" (at 145.161 241.9858 0)
-      (effects (font (size 1.27 1.27)))
-    )
+    (property "Value" "+3.3V" (at 144.78 242.824 0)
+      (effects (font (size 1.27 1.27)))
+    )

Commit message: Development
Parts:
- C1006, C1008, C1010, C1021: footprint (none) -> Capacitor_SMD:C_0603_1608Metric_Pad1.08x0.95mm_HandSolder
- FB1001: footprint (none) -> Inductor_SMD:L_0805_2012Metric_Pad1.05x1.20mm_HandSolder
- J1001: footprint (none) -> Connector_PinHeader_2.54mm:PinHeader_1x02_P2.54mm_Vertical
- J1002: footprint (none) -> Connector_PinHeader_1.27mm:PinHeader_2x05_P1.27mm_Vertical
- U1002: footprint (none) -> ETH1CFGEN1:TQFP-144_20x20mm_P0.5mm
- U1003: footprint (none) -> Package_SO:MSOP-8_3x3mm_P0.65mm
- Y1001: footprint (none) -> ETH1CFGEN1:NX5032GA
Changed lines of the file:
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@@
       (effects (font (size 1.27 1.27)) (justify left))
     )
-    (property "Footprint" "" (at 49.53 27.94 0)
+    (property "Footprint" "ETH1CFGEN1:NX5032GA" (at 49.53 27.94 0)
       (effects (font (size 1.27 1.27)) hide)
     )
@@
       (effects (font (size 1.27 1.27)))
     )
-    (property "Footprint" "" (at 246.38 267.97 0)
+    (property "Footprint" "Package_SO:MSOP-8_3x3mm_P0.65mm" (at 246.38 267.97 0)
       (effects (font (size 1.27 1.27)) hide)
     )
@@
       (effects (font (size 1.27 1.27)) (justify left))
     )
-    (property "Footprint" "" (at 53.0352 209.55 0)
+    (property "Footprint" "Capacitor_SMD:C_0603_1608Metric_Pad1.08x0.95mm_HandSolder" (at 53.0352 209.55 0)
       (effects (font (size 1.27 1.27)) hide)
     )
@@
       (effects (font (size 1.27 1.27)))
     )
-    (property "Footprint" "" (at 175.26 264.922 90)
+    (property "Footprint" "Inductor_SMD:L_0805_2012Metric_Pad1.05x1.20mm_HandSolder" (at 175.26 264.922 90)
       (effects (font (size 1.27 1.27)) hide)
     )
@@
       (effects (font (size 1.27 1.27)))
     )
-    (property "Footprint" "" (at 631.19 87.63 0)
+    (property "Footprint" "ETH1CFGEN1:TQFP-144_20x20mm_P0.5mm" (at 631.19 87.63 0)
       (effects (font (size 1.27 1.27)) hide)
     )
@@
       (effects (font (size 1.27 1.27)) (justify left))
     )
-    (property "Footprint" "" (at 82.2452 231.14 0)
+    (property "Footprint" "Capacitor_SMD:C_0603_1608Metric_Pad1.08x0.95mm_HandSolder" (at 82.2452 231.14 0)
       (effects (font (size 1.27 1.27)) hide)
     )
@@
       (effects (font (size 1.27 1.27)) (justify left))
     )
-    (property "Footprint" "" (at 182.5752 275.59 0)
+    (property "Footprint" "Capacitor_SMD:C_0603_1608Metric_Pad1.08x0.95mm_HandSolder" (at 182.5752 275.59 0)
       (effects (font (size 1.27 1.27)) hide)
     )
@@
       (effects (font (size 1.27 1.27)))
     )
-    (property "Footprint" "" (at 210.82 267.97 0)
+    (property "Footprint" "Connector_PinHeader_1.27mm:PinHeader_2x05_P1.27mm_Vertical" (at 210.82 267.97 0)
       (effects (font (size 1.27 1.27)) hide)
     )
@@
       (effects (font (size 1.27 1.27)) (justify left))
     )
-    (property "Footprint" "" (at 64.4652 209.55 0)
+    (property "Footprint" "Capacitor_SMD:C_0603_1608Metric_Pad1.08x0.95mm_HandSolder" (at 64.4652 209.55 0)
       (effects (font (size 1.27 1.27)) hide)
     )
@@
       (effects (font (size 1.27 1.27)) (justify left))
     )
-    (property "Footprint" "" (at 20.32 205.74 0)
-      (effects (font (size 1.27 1.27)) hide)
-    )
+    (property "Footprint" "Connector_PinHeader_2.54mm:PinHeader_1x02_P2.54mm_Vertical" (at 20.32 205.74 0)
+      (effects (font (size 1.27 1.27)) hide)
+    )
