File: hardware/ETH1CFGEN1A/Power.kicad_sch (KiCad schematic)
At the start: 89 parts, among them Q701 IRFR5410, U701 TSR 1-2450, U702 LT8330_S6, U703 LT8330_S6, U704 TSR 1-2433, U705 MAX5902, U706 MC7815BD2TR4G, U707 MC7915ACD2TG, U708 LT8330_S6, U709 LT8330_S6, U710 THL15WI_Single, U711 MC7805CD2TG, U712 L7905CD2T-TR

Commit message: Development
Parts:
- C721, C722: value 10u/50V -> 10u/35V
- L703: symbol ETH1CDMM1:7448014501 -> ETH1CFGEN1:7448014501
- U701: value TSR 1-2450 -> TSR1
- U704: value TSR 1-2433 -> TSR1
- U705: symbol ETH1CDMM1:MAX5902 -> ETH1CFGEN1:MAX5902
- U710: value THL15WI_Single -> THL15-2415WI
Connections:
- net +24VF renamed VPP
Other:
- moved on the sheet: C914, C915, U701, U704

Commit message: Development
Parts:
- C702, C703, C711, C712, C717, C718, C719, C720, C721, C722, C723, C724, C725, C726, C727, C728, C733, C734, C737, C738, C739, C740, C741, C742: footprint (none) -> Capacitor_SMD:C_1206_3216Metric_Pad1.33x1.80mm_HandSolder
- C705: renamed from C704; footprint (none) -> Capacitor_SMD:C_1206_3216Metric_Pad1.33x1.80mm_HandSolder
- C706: renamed from C705; footprint (none) -> Capacitor_SMD:C_1206_3216Metric_Pad1.33x1.80mm_HandSolder
- C708, C709, C729, C730, C914: footprint (none) -> Capacitor_SMD:C_0603_1608Metric_Pad1.08x0.95mm_HandSolder
- C731, C732: footprint (none) -> Capacitor_SMD:C_1210_3225Metric_Pad1.33x2.70mm_HandSolder
- C914: value 1u -> 1u/50V; footprint (none) -> Capacitor_SMD:C_1206_3216Metric_Pad1.33x1.80mm_HandSolder
- D701, D702, D706, D707: footprint (none) -> Diode_SMD:D_SOD-128
- D703: footprint (none) -> ETH1CFGEN1:DO_214AA_REV
- D704: footprint (none) -> LED_SMD:LED_0603_1608Metric_Pad1.05x0.95mm_HandSolder
- D705: footprint (none) -> Diode_SMD:D_SOD-123
- F701: footprint (none) -> ETH1CFGEN1:Fuse_SMD2920
- L701, L702, L704, L705: footprint (none) -> ETH1CFGEN1:74489440068
- L703: footprint (none) -> ETH1CFGEN1:7448014501
- Q701: footprint (none) -> ETH1CFGEN1:TO-252-2_Rectifier
- U701: value TSR1 -> TSR1-2450; footprint (none) -> ETH1CFGEN1:TSR1
- U702, U703, U708, U709: value LT8330_S6 -> LT8330ES6#TRMPBF; footprint (none) -> Package_TO_SOT_SMD:TSOT-23-6_HandSoldering
- U704: value TSR1 -> TSR1-2433; footprint (none) -> ETH1CFGEN1:TSR1
- U705: value MAX5902 -> MAX5902AAEUT+T; footprint (none) -> Package_TO_SOT_SMD:SOT-23-6_Handsoldering
- U706, U707, U711, U712: footprint (none) -> Package_TO_SOT_SMD:TO-263-2
- U710: footprint (none) -> ETH1CFGEN1:THL15
Other:
- moved on the sheet: C914, C915, U704
