File: hardware/ETH1CFGEN1A/SelftTest.kicad_sch (KiCad schematic)
At the start: 30 parts, among them U801 TL074, U802 TL074, U803 TLA2528

Commit message: Development
Parts:
- removed U803: TLA2528, Package_DFN_QFN:WQFN-16-1EP_3x3mm_P0.5mm_EP1.6x1.6mm_ThermalVias, symbol ETH3CDAQ1:TLA2528
- added U803: TLA2528, symbol ETH1CFGEN1:TLA2528
Connections:
- net +5V: now also U803.7 (AVDD)
- net AIN0: now also U803.15 (AIN0/GPIO0)
- net AIN1: now also U803.16 (AIN1/GPIO1)
- net AIN2: now also U803.1 (AIN2/GPIO2)
- net AIN3: now also U803.2 (AIN3/GPIO3)
- net AIN4: now also U803.3 (AIN4/GPIO4)
- net AIN5: now also U803.4 (AIN5/GPIO5)
- net GNDA: now also U803.17 (PAD), U803.9 (GND)
- net at R815.2, R816.2: now also U803.11 (ADDR)
- net at C809.2, R815.1: now also U803.8 (DECAP)
- net +3V3 renamed +3.3V
- net +3.3V: now also U803.10 (DVDD)
- net ADC_SCL renamed I2C_SCL
- net I2C_SCL: now also U803.13 (SCL)
- net ADC_SDA renamed I2C_SDA
- net I2C_SDA: now also U803.14 (SDA)
- no-connect marks 1 -> 2
Other:
- moved on the sheet: R817, R818

Commit message: Development
Parts:
- U801, U802: value TL074 -> TL074HIPWR
- U803: value TLA2528 -> TLA2528IRTER; footprint (none) -> Package_DFN_QFN:WQFN-16-1EP_3x3mm_P0.5mm_EP1.6x1.6mm_ThermalVias
Changed lines of the file:
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@@
       (effects (font (size 1.27 1.27)))
     )
-    (property "Value" "TL074" (at 101.6 93.9546 0)
+    (property "Value" "TL074HIPWR" (at 101.6 93.9546 0)
       (effects (font (size 1.27 1.27)))
     )
@@
       (effects (font (size 1.27 1.27)))
     )
-    (property "Value" "TL074" (at 129.54 73.6346 0)
+    (property "Value" "TL074HIPWR" (at 129.54 73.6346 0)
       (effects (font (size 1.27 1.27)))
     )
@@
       (effects (font (size 1.27 1.27)))
     )
-    (property "Value" "TL074" (at 129.54 46.9646 0)
+    (property "Value" "TL074HIPWR" (at 129.54 46.9646 0)
       (effects (font (size 1.27 1.27)))
     )
@@
       (effects (font (size 1.27 1.27)))
     )
-    (property "Value" "TL074" (at 129.54 20.2946 0)
+    (property "Value" "TL074HIPWR" (at 129.54 20.2946 0)
       (effects (font (size 1.27 1.27)))
     )
@@
       (effects (font (size 1.27 1.27)) (justify left))
     )
-    (property "Value" "TL074" (at 25.6032 180.848 0)
+    (property "Value" "TL074HIPWR" (at 25.6032 180.848 0)
       (effects (font (size 1.27 1.27)) (justify left))
     )
@@
       (effects (font (size 1.27 1.27)) (justify left))
     )
-    (property "Value" "TL074" (at 39.5732 180.848 0)
+    (property "Value" "TL074HIPWR" (at 39.5732 180.848 0)
       (effects (font (size 1.27 1.27)) (justify left))
     )
@@
       (effects (font (size 1.27 1.27)))
     )
-    (property "Value" "TL074" (at 184.785 20.2946 0)
+    (property "Value" "TL074HIPWR" (at 184.785 20.2946 0)
       (effects (font (size 1.27 1.27)))
     )
@@
   )
   (symbol (lib_id "ETH1CFGEN1:TLA2528") (at 198.12 108.585 0) (unit 1)
-    (in_bom yes) (on_board yes) (dnp no) (fields_autoplaced)
-    (property "Reference" "U803" (at 208.915 86.995 0)
-      (effects (font (size 1.27 1.27)))
-    )
-    (property "Value" "TLA2528" (at 208.915 89.535 0)
-      (effects (font (size 1.27 1.27)))
-    )
-    (property "Footprint" "" (at 198.12 107.315 0)
+    (in_bom yes) (on_board yes) (dnp no)
+    (property "Reference" "U803" (at 208.915 125.73 0)
+      (effects (font (size 1.27 1.27)) (justify left))
+    )
+    (property "Value" "TLA2528IRTER" (at 205.3941 128.27 0)
+      (effects (font (size 1.27 1.27)) (justify left))
+    )
+    (property "Footprint" "Package_DFN_QFN:WQFN-16-1EP_3x3mm_P0.5mm_EP1.6x1.6mm_ThermalVias" (at 198.12 107.315 0)
       (effects (font (size 1.27 1.27)) hide)
     )
@@
       (effects (font (size 1.27 1.27)))
     )
-    (property "Value" "TL074" (at 101.6 137.1346 0)
+    (property "Value" "TL074HIPWR" (at 101.6 137.1346 0)
       (effects (font (size 1.27 1.27)))
     )
@@
       (effects (font (size 1.27 1.27)))
     )
-    (property "Value" "TL074" (at 184.785 46.9646 0)
+    (property "Value" "TL074HIPWR" (at 184.785 46.9646 0)
       (effects (font (size 1.27 1.27)))
     )
@@
       (effects (font (size 1.27 1.27)))
     )
-    (property "Value" "TL074" (at 129.54 116.8146 0)
-      (effects (font (size 1.27 1.27)))
-    )
+    (property "Value" "TL074HIPWR" (at 129.54 116.8146 0)
+      (effects (font (size 1.27 1.27)))
+    )
