File: hardware/ETH1CFGEN1A/Trigger.kicad_sch (KiCad schematic)
At the start: 22 parts, among them U701 TXB0104PW, U702 ADuM5402, U703 74AC125

Commit message: Development
Parts:
- C702, C705, C707: footprint Capacitor_SMD:C_0603_1608Metric_Pad1.08x0.95mm_HandSolder -> (none)
- D701: footprint Package_TO_SOT_SMD:SOT-23 -> (none)
- D702: footprint Diode_SMD:D_SMB -> (none)
- D703: footprint Diode_SMD:D_SOD-323_HandSoldering -> (none)
- L701: footprint ETH1CSMU2:CW252016 -> (none)
- U701: footprint Package_SO:TSSOP-14_4.4x5mm_P0.65mm -> (none)
- U702: footprint Package_SO:SOIC-16W_7.5x10.3mm_P1.27mm -> (none)
- U703: footprint Package_SO:TSSOP-14_4.4x5mm_P0.65mm -> (none); symbol ETH1CSMU2:74AC125 -> ETH1CFGEN1:74AC125
Connections:
- net GND renamed GNDD

Commit message: Development
Parts:
- U701: footprint (none) -> Package_SO:TSSOP-14_4.4x5mm_P0.65mm
Connections:
- net +5V_TRIG renamed +5VP
- net GND_TRIG renamed GND1

Commit message: Development
Parts:
- C702, C705, C707: footprint (none) -> Capacitor_SMD:C_0603_1608Metric_Pad1.08x0.95mm_HandSolder
- D701: footprint (none) -> Package_TO_SOT_SMD:SOT-23
- D702: footprint (none) -> Diode_SMD:D_SMB
- D703: footprint (none) -> Diode_SMD:D_SOD-323_HandSoldering
- L701: footprint (none) -> ETH1CFGEN1:CW252016
- U702: footprint (none) -> Package_SO:SOIC-16W_7.5x10.3mm_P1.27mm
- U703: footprint (none) -> Package_SO:TSSOP-14_4.4x5mm_P0.65mm
Changed lines of the file:
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@@
       (effects (font (size 1.27 1.27)) (justify left))
     )
-    (property "Footprint" "" (at 213.36 120.65 0)
+    (property "Footprint" "Diode_SMD:D_SMB" (at 213.36 120.65 0)
       (effects (font (size 1.27 1.27)) hide)
     )
@@
       (effects (font (size 1.27 1.27)) (justify left))
     )
-    (property "Footprint" "" (at 136.8552 31.75 0)
+    (property "Footprint" "Capacitor_SMD:C_0603_1608Metric_Pad1.08x0.95mm_HandSolder" (at 136.8552 31.75 0)
       (effects (font (size 1.27 1.27)) hide)
     )
@@
       (effects (font (size 1.27 1.27)))
     )
-    (property "Footprint" "" (at 127 179.07 0)
+    (property "Footprint" "Package_SO:TSSOP-14_4.4x5mm_P0.65mm" (at 127 179.07 0)
       (effects (font (size 1.27 1.27)) hide)
     )
@@
       (effects (font (size 1.27 1.27)))
     )
-    (property "Footprint" "" (at 196.85 59.69 0)
+    (property "Footprint" "Package_SO:TSSOP-14_4.4x5mm_P0.65mm" (at 196.85 59.69 0)
       (effects (font (size 1.27 1.27)) hide)
     )
@@
       (effects (font (size 1.27 1.27)))
     )
-    (property "Footprint" "" (at 219.71 137.16 0)
+    (property "Footprint" "ETH1CFGEN1:CW252016" (at 219.71 137.16 0)
       (effects (font (size 1.27 1.27)) hide)
     )
@@
       (effects (font (size 1.27 1.27)))
     )
-    (property "Footprint" "" (at 115.57 107.95 0)
+    (property "Footprint" "Package_SO:SOIC-16W_7.5x10.3mm_P1.27mm" (at 115.57 107.95 0)
       (effects (font (size 1.27 1.27) italic) hide)
     )
@@
       (effects (font (size 1.27 1.27)) (justify left))
     )
-    (property "Footprint" "" (at 70.8152 31.75 0)
+    (property "Footprint" "Capacitor_SMD:C_0603_1608Metric_Pad1.08x0.95mm_HandSolder" (at 70.8152 31.75 0)
       (effects (font (size 1.27 1.27)) hide)
     )
@@
       (effects (font (size 1.27 1.27)) (justify left))
     )
-    (property "Footprint" "" (at 185.42 137.16 0)
+    (property "Footprint" "Package_TO_SOT_SMD:SOT-23" (at 185.42 137.16 0)
       (effects (font (size 1.27 1.27)) hide)
     )
@@
       (effects (font (size 1.27 1.27)) (justify left))
     )
-    (property "Footprint" "" (at 107.6452 31.75 0)
+    (property "Footprint" "Capacitor_SMD:C_0603_1608Metric_Pad1.08x0.95mm_HandSolder" (at 107.6452 31.75 0)
       (effects (font (size 1.27 1.27)) hide)
     )
@@
       (effects (font (size 1.27 1.27)) (justify left))
     )
-    (property "Footprint" "" (at 246.38 142.24 0)
+    (property "Footprint" "Diode_SMD:D_SOD-323_HandSoldering" (at 246.38 142.24 0)
       (effects (font (size 1.27 1.27)) hide)
     )
@@
       (effects (font (size 1.27 1.27)))
     )
-    (property "Footprint" "" (at 196.85 81.28 0)
+    (property "Footprint" "Package_SO:TSSOP-14_4.4x5mm_P0.65mm" (at 196.85 81.28 0)
       (effects (font (size 1.27 1.27)) hide)
     )
@@
       (effects (font (size 1.27 1.27)))
     )
-    (property "Footprint" "" (at 151.13 115.57 0)
+    (property "Footprint" "Package_SO:TSSOP-14_4.4x5mm_P0.65mm" (at 151.13 115.57 0)
       (effects (font (size 1.27 1.27)) hide)
     )
@@
       (effects (font (size 1.27 1.27)))
     )
-    (property "Footprint" "" (at 196.85 38.1 0)
-      (effects (font (size 1.27 1.27)) hide)
-    )
+    (property "Footprint" "Package_SO:TSSOP-14_4.4x5mm_P0.65mm" (at 196.85 38.1 0)
+      (effects (font (size 1.27 1.27)) hide)
+    )
