File: hardware/ETH1CFGEN1A/ETH1CFGEN1A.kicad_pcb (KiCad board)
At the start: 4 copper layers, 160 x 100 mm, 280 parts, among them J201 Conn_02x01, J202 20021111-00010T4LF, J501 C64AC, J601 Conn_02x04_Odd_Even, J602 Conn_02x04_Odd_Even, J603 Conn_Coaxial, K501 HE3621A0510, K502 HE3621A0510, K503 HE3621A0510, K504 HE3621A0510, K505 HE3621A0510, K506 HE3621A0510, Q701 IRFR5410, U201 HDC1080, U202 STM32F746ZG, U203 24LC08B-E/MS, U301 LAN8742, U302 LC03-3.3BTG, U303 LC03-3.3BTG, U401 TXB0104PW, U402 ADuM5402, U403 74AC125, U501 ULN2003AIPWR, U701 TSR1-2450, U702 LT8330ES6#TRMPBF, U703 LT8330ES6#TRMPBF, U704 TSR1-2433, U705 MAX5902AAEUT+T, U706 MC7815BD2TR4G, U707 MC7915ACD2TG, U708 LT8330ES6#TRMPBF, U709 LT8330ES6#TRMPBF, U710 THL15-2415WI, U711 MC7805CD2TG, U712 L7905CD2T-TR, U801 TL074HIPWR, U802 TL074HIPWR, U803 TLA2528IRTER, U903 XC6SLX9-3TQG144I, U904 W25Q64JV, Y201 NX5032GA-16.000M, Y301 NX5032GA-25.000000MHZ-LN-CD-1

Commit message: Hardware development
Parts:
- added C1001: 33p, Capacitor_SMD:C_0603_1608Metric_Pad1.08x0.95mm_HandSolder, F.Cu at (54.4, -6.01)
- added C1002: 33p, Capacitor_SMD:C_0603_1608Metric_Pad1.08x0.95mm_HandSolder, F.Cu at (54.4, -3.50)
- added C1003: 100n, Capacitor_SMD:C_0603_1608Metric_Pad1.08x0.95mm_HandSolder, F.Cu at (54.4, -0.99)
- added C1005: 100n, Capacitor_SMD:C_0603_1608Metric_Pad1.08x0.95mm_HandSolder, F.Cu at (54.4, 1.52)
- added C1006: 100n, Capacitor_SMD:C_0603_1608Metric_Pad1.08x0.95mm_HandSolder, F.Cu at (54.4, 4.03)
- added C1010: 100p, Capacitor_SMD:C_0603_1608Metric_Pad1.08x0.95mm_HandSolder, F.Cu at (54.4, 6.54)
- added C1011: 100p, Capacitor_SMD:C_0603_1608Metric_Pad1.08x0.95mm_HandSolder, F.Cu at (54.4, 9.05)
- added C1012: 100n, Capacitor_SMD:C_0603_1608Metric_Pad1.08x0.95mm_HandSolder, F.Cu at (54.4, 11.6)
- added C1013: 33p, Capacitor_SMD:C_0603_1608Metric_Pad1.08x0.95mm_HandSolder, F.Cu at (54.4, 14.1)
- added C1014: 33p, Capacitor_SMD:C_0603_1608Metric_Pad1.08x0.95mm_HandSolder, F.Cu at (54.4, 16.6)
- added C1015: 30p, Capacitor_SMD:C_0603_1608Metric_Pad1.08x0.95mm_HandSolder, F.Cu at (54.4, 19.1)
- added C1016: 30p, Capacitor_SMD:C_0603_1608Metric_Pad1.08x0.95mm_HandSolder, F.Cu at (54.4, 21.6)
- added C1017: 100n, Capacitor_SMD:C_0603_1608Metric_Pad1.08x0.95mm_HandSolder, F.Cu at (54.4, 24.1)
- added C1018: 33p, Capacitor_SMD:C_0603_1608Metric_Pad1.08x0.95mm_HandSolder, F.Cu at (54.4, 26.6)
- added C1019: 33p, Capacitor_SMD:C_0603_1608Metric_Pad1.08x0.95mm_HandSolder, F.Cu at (58.8, -6.01)
- added C1021: 56p, Capacitor_SMD:C_0603_1608Metric_Pad1.08x0.95mm_HandSolder, F.Cu at (58.8, -3.50)
- added C1022: 56p, Capacitor_SMD:C_0603_1608Metric_Pad1.08x0.95mm_HandSolder, F.Cu at (58.8, -0.99)
- added C1023: 3p3, Capacitor_SMD:C_0603_1608Metric_Pad1.08x0.95mm_HandSolder, F.Cu at (58.8, 1.52)
- added C1024: 3p3, Capacitor_SMD:C_0603_1608Metric_Pad1.08x0.95mm_HandSolder, F.Cu at (58.8, 4.03)
- added C1027: 56p, Capacitor_SMD:C_0603_1608Metric_Pad1.08x0.95mm_HandSolder, F.Cu at (58.8, 6.54)
- added C1028: 56p, Capacitor_SMD:C_0603_1608Metric_Pad1.08x0.95mm_HandSolder, F.Cu at (58.8, 9.05)
- added C1029: 120p, Capacitor_SMD:C_0603_1608Metric_Pad1.08x0.95mm_HandSolder, F.Cu at (58.8, 11.6)
- added C1030: 120p, Capacitor_SMD:C_0603_1608Metric_Pad1.08x0.95mm_HandSolder, F.Cu at (58.8, 14.1)
- added C1031: 33p, Capacitor_SMD:C_0603_1608Metric_Pad1.08x0.95mm_HandSolder, F.Cu at (58.8, 16.6)
- added C1032: 33p, Capacitor_SMD:C_0603_1608Metric_Pad1.08x0.95mm_HandSolder, F.Cu at (58.8, 19.1)
- added C1033: 56p, Capacitor_SMD:C_0603_1608Metric_Pad1.08x0.95mm_HandSolder, F.Cu at (58.8, 21.6)
- added C1034: 56p, Capacitor_SMD:C_0603_1608Metric_Pad1.08x0.95mm_HandSolder, F.Cu at (58.8, 24.1)
- added C1035: 150p, Capacitor_SMD:C_0603_1608Metric_Pad1.08x0.95mm_HandSolder, F.Cu at (58.8, 26.6)
- added C1036: 150p, Capacitor_SMD:C_0603_1608Metric_Pad1.08x0.95mm_HandSolder, F.Cu at (63.1, -6.01)
- added C1037: 62p, Capacitor_SMD:C_0603_1608Metric_Pad1.08x0.95mm_HandSolder, F.Cu at (63.1, -3.50)
- added C1038: 62p, Capacitor_SMD:C_0603_1608Metric_Pad1.08x0.95mm_HandSolder, F.Cu at (63.1, -0.99)
- added C1039: 8p2, Capacitor_SMD:C_0603_1608Metric_Pad1.08x0.95mm_HandSolder, F.Cu at (63.1, 1.52)
- added C1040: 8p2, Capacitor_SMD:C_0603_1608Metric_Pad1.08x0.95mm_HandSolder, F.Cu at (63.1, 4.03)
- added C1041: 100n, Capacitor_SMD:C_0603_1608Metric_Pad1.08x0.95mm_HandSolder, F.Cu at (63.1, 6.54)
- added C1042: 33p, Capacitor_SMD:C_0603_1608Metric_Pad1.08x0.95mm_HandSolder, F.Cu at (63.1, 9.05)
- added C1043: 33p, Capacitor_SMD:C_0603_1608Metric_Pad1.08x0.95mm_HandSolder, F.Cu at (63.1, 11.6)
- added C1044: 100n, Capacitor_SMD:C_0603_1608Metric_Pad1.08x0.95mm_HandSolder, F.Cu at (63.1, 14.1)
- added C1045: 100n, Capacitor_SMD:C_0603_1608Metric_Pad1.08x0.95mm_HandSolder, F.Cu at (63.1, 16.6)
- added C1046: 130p, Capacitor_SMD:C_0603_1608Metric_Pad1.08x0.95mm_HandSolder, F.Cu at (63.1, 19.1)
- added C1047: 130p, Capacitor_SMD:C_0603_1608Metric_Pad1.08x0.95mm_HandSolder, F.Cu at (63.1, 21.6)
- added C1048: 330p, Capacitor_SMD:C_0603_1608Metric_Pad1.08x0.95mm_HandSolder, F.Cu at (63.1, 24.1)
- added C1049: 330p, Capacitor_SMD:C_0603_1608Metric_Pad1.08x0.95mm_HandSolder, F.Cu at (63.1, 26.6)
- added C1051: 100n, Capacitor_SMD:C_0603_1608Metric_Pad1.08x0.95mm_HandSolder, F.Cu at (67.5, -6.01)
- added C1053: 15p, Capacitor_SMD:C_0603_1608Metric_Pad1.08x0.95mm_HandSolder, F.Cu at (67.5, -3.50)
- added C1054: 15p, Capacitor_SMD:C_0603_1608Metric_Pad1.08x0.95mm_HandSolder, F.Cu at (67.5, -0.99)
- added C1055: 56p, Capacitor_SMD:C_0603_1608Metric_Pad1.08x0.95mm_HandSolder, F.Cu at (67.5, 1.52)
- added C1056: 56p, Capacitor_SMD:C_0603_1608Metric_Pad1.08x0.95mm_HandSolder, F.Cu at (67.5, 4.03)
- added C1058: 33p, Capacitor_SMD:C_0603_1608Metric_Pad1.08x0.95mm_HandSolder, F.Cu at (67.5, 6.54)
- added C1059: 33p, Capacitor_SMD:C_0603_1608Metric_Pad1.08x0.95mm_HandSolder, F.Cu at (67.5, 9.05)
- added C1060: 220n, Capacitor_SMD:C_0603_1608Metric_Pad1.08x0.95mm_HandSolder, F.Cu at (67.5, 11.6)
- added C1061: 100p, Capacitor_SMD:C_0603_1608Metric_Pad1.08x0.95mm_HandSolder, F.Cu at (67.5, 14.1)
- added C1062: 100p, Capacitor_SMD:C_0603_1608Metric_Pad1.08x0.95mm_HandSolder, F.Cu at (67.5, 16.6)
- added C1063: 5p6, Capacitor_SMD:C_0603_1608Metric_Pad1.08x0.95mm_HandSolder, F.Cu at (67.5, 19.1)
- added C1064: 5p6, Capacitor_SMD:C_0603_1608Metric_Pad1.08x0.95mm_HandSolder, F.Cu at (67.5, 21.6)
- added C1065: 100n, Capacitor_SMD:C_0603_1608Metric_Pad1.08x0.95mm_HandSolder, F.Cu at (67.5, 24.1)
- added C1066: 100n, Capacitor_SMD:C_0603_1608Metric_Pad1.08x0.95mm_HandSolder, F.Cu at (67.5, 26.6)
- added C1067: 47p, Capacitor_SMD:C_0603_1608Metric_Pad1.08x0.95mm_HandSolder, F.Cu at (71.8, -6.01)
- added C1068: 47p, Capacitor_SMD:C_0603_1608Metric_Pad1.08x0.95mm_HandSolder, F.Cu at (71.8, -3.50)
- added C1071: 220n, Capacitor_SMD:C_0603_1608Metric_Pad1.08x0.95mm_HandSolder, F.Cu at (71.8, -0.99)
- added C1072: 22p, Capacitor_SMD:C_0603_1608Metric_Pad1.08x0.95mm_HandSolder, F.Cu at (71.8, 1.52)
- added C1073: 22p, Capacitor_SMD:C_0603_1608Metric_Pad1.08x0.95mm_HandSolder, F.Cu at (71.8, 4.03)
- added C1074: 10p, Capacitor_SMD:C_0603_1608Metric_Pad1.08x0.95mm_HandSolder, F.Cu at (71.8, 6.54)
- added C1075: 100p, Capacitor_SMD:C_0603_1608Metric_Pad1.08x0.95mm_HandSolder, F.Cu at (71.8, 9.05)
- added C1076: 1p, Capacitor_SMD:C_0603_1608Metric_Pad1.08x0.95mm_HandSolder, F.Cu at (71.8, 11.6)
- added C1077: 100p, Capacitor_SMD:C_0603_1608Metric_Pad1.08x0.95mm_HandSolder, F.Cu at (71.8, 14.1)
- added C1078: 10p, Capacitor_SMD:C_0603_1608Metric_Pad1.08x0.95mm_HandSolder, F.Cu at (71.8, 16.6)
- added C1079: 10p, Capacitor_SMD:C_0603_1608Metric_Pad1.08x0.95mm_HandSolder, F.Cu at (71.8, 19.1)
- added C1080: 47p, Capacitor_SMD:C_0603_1608Metric_Pad1.08x0.95mm_HandSolder, F.Cu at (71.8, 21.6)
- added C1081: 15p, Capacitor_SMD:C_0603_1608Metric_Pad1.08x0.95mm_HandSolder, F.Cu at (71.8, 24.1)
- added C1082: 33p, Capacitor_SMD:C_0603_1608Metric_Pad1.08x0.95mm_HandSolder, F.Cu at (71.8, 26.6)
- added C1083: 150p, Capacitor_SMD:C_0603_1608Metric_Pad1.08x0.95mm_HandSolder, F.Cu at (76.2, -6.01)
- added D1001: BAS40-04, Package_TO_SOT_SMD:SOT-23, F.Cu at (89.5, 17.9)
- added J901: Conn_01x06, Connector_PinHeader_2.54mm:PinHeader_1x06_P2.54mm_Vertical, F.Cu at (145.9, 73.7)
- added R1001: 1k, Resistor_SMD:R_0603_1608Metric_Pad0.98x0.95mm_HandSolder, F.Cu at (76.2, -3.50)
- added R1002: 10k, Resistor_SMD:R_0603_1608Metric_Pad0.98x0.95mm_HandSolder, F.Cu at (76.2, -0.99)
- added R1003: 51R1, Resistor_SMD:R_0603_1608Metric_Pad0.98x0.95mm_HandSolder, F.Cu at (76.2, 1.52)
- added R1004: 51R1, Resistor_SMD:R_0603_1608Metric_Pad0.98x0.95mm_HandSolder, F.Cu at (76.2, 4.03)
- added R1005: 100, Resistor_SMD:R_0603_1608Metric_Pad0.98x0.95mm_HandSolder, F.Cu at (76.2, 6.54)
- added R1006: 82k5, Resistor_SMD:R_0603_1608Metric_Pad0.98x0.95mm_HandSolder, F.Cu at (76.2, 9.05)
- added R1007: 1k, Resistor_SMD:R_0603_1608Metric_Pad0.98x0.95mm_HandSolder, F.Cu at (76.2, 11.6)
- added R1008: 2k, Resistor_SMD:R_0603_1608Metric_Pad0.98x0.95mm_HandSolder, F.Cu at (76.2, 14.1)
- added R1009: 69, Resistor_SMD:R_0603_1608Metric_Pad0.98x0.95mm_HandSolder, F.Cu at (76.2, 16.6)
- added R1010: 261, Resistor_SMD:R_0603_1608Metric_Pad0.98x0.95mm_HandSolder, F.Cu at (76.2, 19.1)
- added R1011: 261, Resistor_SMD:R_0603_1608Metric_Pad0.98x0.95mm_HandSolder, F.Cu at (76.2, 21.6)
- added R1012: 21k5, Resistor_SMD:R_0603_1608Metric_Pad0.98x0.95mm_HandSolder, F.Cu at (76.2, 24.1)
- added R1013: 69, Resistor_SMD:R_0603_1608Metric_Pad0.98x0.95mm_HandSolder, F.Cu at (76.2, 26.6)
- added R1014: 1k, Resistor_SMD:R_0603_1608Metric_Pad0.98x0.95mm_HandSolder, F.Cu at (80.5, -6.01)
- added R1015: 100, Resistor_SMD:R_0603_1608Metric_Pad0.98x0.95mm_HandSolder, F.Cu at (80.5, -3.50)
- added R1016: 100, Resistor_SMD:R_0603_1608Metric_Pad0.98x0.95mm_HandSolder, F.Cu at (80.5, -0.99)
- added R1017: 10k, Resistor_SMD:R_0603_1608Metric_Pad0.98x0.95mm_HandSolder, F.Cu at (80.5, 1.52)
- added R1018: 1k78, Resistor_SMD:R_0603_1608Metric_Pad0.98x0.95mm_HandSolder, F.Cu at (80.5, 4.03)
- added R1019: 100, Resistor_SMD:R_0603_1608Metric_Pad0.98x0.95mm_HandSolder, F.Cu at (80.5, 6.54)
- added R1020: 511, Resistor_SMD:R_0603_1608Metric_Pad0.98x0.95mm_HandSolder, F.Cu at (80.5, 9.05)
- added R1021: 511, Resistor_SMD:R_0603_1608Metric_Pad0.98x0.95mm_HandSolder, F.Cu at (80.5, 11.6)
- added R1022: 100, Resistor_SMD:R_0603_1608Metric_Pad0.98x0.95mm_HandSolder, F.Cu at (80.5, 14.1)
- added R1023: 10k, Resistor_SMD:R_0603_1608Metric_Pad0.98x0.95mm_HandSolder, F.Cu at (80.5, 16.6)
- added R1024: 21R5, Resistor_SMD:R_0603_1608Metric_Pad0.98x0.95mm_HandSolder, F.Cu at (80.5, 19.1)
- added R1025: 100, Resistor_SMD:R_0603_1608Metric_Pad0.98x0.95mm_HandSolder, F.Cu at (80.5, 21.6)
- added R1026: 1k78, Resistor_SMD:R_0603_1608Metric_Pad0.98x0.95mm_HandSolder, F.Cu at (80.5, 24.1)
- added R1027: 10k, Resistor_SMD:R_0603_1608Metric_Pad0.98x0.95mm_HandSolder, F.Cu at (80.5, 26.6)
- added R1028: 51R1, Resistor_SMD:R_0603_1608Metric_Pad0.98x0.95mm_HandSolder, F.Cu at (84.9, -6.01)
- added R1029: 200, Resistor_SMD:R_0603_1608Metric_Pad0.98x0.95mm_HandSolder, F.Cu at (84.9, -3.50)
- added R1030: 200, Resistor_SMD:R_0603_1608Metric_Pad0.98x0.95mm_HandSolder, F.Cu at (84.9, -0.99)
- added R1031: 100k, Resistor_SMD:R_0603_1608Metric_Pad0.98x0.95mm_HandSolder, F.Cu at (84.9, 1.52)
- added R1032: 953, Resistor_SMD:R_0603_1608Metric_Pad0.98x0.95mm_HandSolder, F.Cu at (84.9, 4.03)
- added R1033: 953, Resistor_SMD:R_0603_1608Metric_Pad0.98x0.95mm_HandSolder, F.Cu at (84.9, 6.54)
- added R1034: 100k, Resistor_SMD:R_0603_1608Metric_Pad0.98x0.95mm_HandSolder, F.Cu at (84.9, 9.05)
- added R1035: 51R1, Resistor_SMD:R_0603_1608Metric_Pad0.98x0.95mm_HandSolder, F.Cu at (84.9, 11.6)
- added R1036: 34R8, Resistor_SMD:R_0603_1608Metric_Pad0.98x0.95mm_HandSolder, F.Cu at (84.9, 14.1)
- added R1037: 196, Resistor_SMD:R_0603_1608Metric_Pad0.98x0.95mm_HandSolder, F.Cu at (84.9, 16.6)
- added U1002: AD9744, Package_SO:TSSOP-28_4.4x9.7mm_P0.65mm, F.Cu at (119.3, 78.0)
- added U1004: THS3001CD, Package_SO:SOIC-8_3.9x4.9mm_P1.27mm, F.Cu at (91.3, 7.21)
- added U901: TLV1117LV33DCYR, Package_TO_SOT_SMD:SOT-223-3_TabPin2, F.Cu at (103.4, 96.6)
- added U902: TLV1117LV12DCYR, Package_TO_SOT_SMD:SOT-223-3_TabPin2, F.Cu at (115.7, 95.4)
- added X1001: SG5032CAN 50.000000M-TJGA3, Oscillator:Oscillator_SMD_SeikoEpson_SG8002LB-4Pin_5.0x3.2mm, F.Cu at (90.4, 13.1)
- moved L701 10.5 mm to (107.8, 126.6)
- moved L702 10.5 mm to (108.1, 113.6)
- moved U706 10.5 mm to (92.6, 126.5)
- moved U707 10.5 mm to (92.8, 113.4)
- moved L704 5.09 mm to (146.6, 126.7)
- moved L705 5.09 mm to (146.6, 113.4)
- moved U711 5.09 mm to (131.3, 126.7)
- moved U712 5.09 mm to (131.3, 113.4)
- moved U701 2.65 mm to (165.6, 128.4)
- moved U704 2.63 mm to (165.6, 113.3)
- moved U903 1.68 mm to (138.4, 89.8)
- moved U301 0.12 mm to (185.6, 98.5), turned to -90 degrees
