File: hardware/ETH1CFGEN1A/ETH1CFGEN1A.kicad_sch (KiCad schematic)
At the start: 4 parts

Commit message: Development
Other:
- sheet MCU ports: added I2C_SCL, I2C_SDA; removed none
- sheet Self test ports: added I2C_SCL, I2C_SDA; removed ADC_SCL, ADC_SDA
Changed lines of the file:
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@@
+    (stroke (width 0) (type default))
+  )
+  (wire (pts (xy 104.14 100.33) (xy 111.76 100.33))
     (stroke (width 0) (type default))
   )
@@
   )
   (wire (pts (xy 150.495 99.06) (xy 156.21 99.06))
+    (stroke (width 0) (type default))
+  )
+  (wire (pts (xy 104.14 102.235) (xy 111.76 102.235))
     (stroke (width 0) (type default))
   )
@@
       (effects (font (size 1.27 1.27)) (justify left))
     )
+    (pin "I2C_SDA" bidirectional (at 111.76 102.235 180)
+      (effects (font (size 1.27 1.27)) (justify left))
+    )
+    (pin "I2C_SCL" bidirectional (at 111.76 100.33 180)
+      (effects (font (size 1.27 1.27)) (justify left))
+    )
     (instances
       (project "ETH1CFGEN1A"
@@
       (effects (font (size 1.27 1.27)) (justify left top))
     )
-    (pin "ADC_SCL" bidirectional (at 104.14 100.965 0)
-      (effects (font (size 1.27 1.27)) (justify right))
-    )
-    (pin "ADC_SDA" bidirectional (at 104.14 102.87 0)
-      (effects (font (size 1.27 1.27)) (justify right))
-    )
+    (pin "I2C_SCL" bidirectional (at 104.14 100.33 0)
+      (effects (font (size 1.27 1.27)) (justify right))
+    )
+    (pin "I2C_SDA" bidirectional (at 104.14 102.235 0)
+      (effects (font (size 1.27 1.27)) (justify right))
+    )

Commit message: Development
Parts:
- removed H104: MountingHole, symbol Mechanical:MountingHole
- H101, H102, H103: footprint (none) -> MountingHole:MountingHole_3.2mm_M3_DIN965_Pad
Other:
- added sheet FPGA (FPGA.kicad_sch)
Changed lines of the file:
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@@
       (effects (font (size 1.27 1.27)) (justify left))
     )
-    (property "Footprint" "" (at 18.415 184.785 0)
+    (property "Footprint" "MountingHole:MountingHole_3.2mm_M3_DIN965_Pad" (at 18.415 184.785 0)
       (effects (font (size 1.27 1.27)) hide)
     )
@@
       (effects (font (size 1.27 1.27)) (justify left))
     )
-    (property "Footprint" "" (at 18.415 178.435 0)
+    (property "Footprint" "MountingHole:MountingHole_3.2mm_M3_DIN965_Pad" (at 18.415 178.435 0)
       (effects (font (size 1.27 1.27)) hide)
     )
@@
     )
   )
-  (symbol (lib_id "Mechanical:MountingHole") (at 18.415 191.135 0) (unit 1)
-    (in_bom yes) (on_board yes) (dnp no) (fields_autoplaced)
-    (property "Reference" "H104" (at 20.955 189.865 0)
-      (effects (font (size 1.27 1.27)) (justify left))
-    )
-    (property "Value" "MountingHole" (at 20.955 192.405 0)
-      (effects (font (size 1.27 1.27)) (justify left))
-    )
-    (property "Footprint" "" (at 18.415 191.135 0)
-      (effects (font (size 1.27 1.27)) hide)
-    )
-    (property "Datasheet" "~" (at 18.415 191.135 0)
-      (effects (font (size 1.27 1.27)) hide)
-    )
-    (instances
-      (project "ETH1CFGEN1A"
-        (path "/44bc1157-6d68-4ab3-afc0-b8d9f089cc50"
-          (reference "H104") (unit 1)
-        )
-      )
-    )
-  )
   (symbol (lib_id "Mechanical:MountingHole") (at 18.415 172.085 0) (unit 1)
     (in_bom yes) (on_board yes) (dnp no) (fields_autoplaced)
@@
       (effects (font (size 1.27 1.27)) (justify left))
     )
-    (property "Footprint" "" (at 18.415 172.085 0)
+    (property "Footprint" "MountingHole:MountingHole_3.2mm_M3_DIN965_Pad" (at 18.415 172.085 0)
       (effects (font (size 1.27 1.27)) hide)
     )
@@
       )
     )
+  )
+  (sheet (at 22.225 43.815) (size 41.91 43.815) (fields_autoplaced)
+    (stroke (width 0.1524) (type solid))
+    (fill (color 0 0 0 0.0000))
+    (property "Sheetname" "FPGA" (at 22.225 43.1034 0)
+      (effects (font (size 1.27 1.27)) (justify left bottom))
+    )
+    (property "Sheetfile" "FPGA.kicad_sch" (at 22.225 88.2146 0)
+      (effects (font (size 1.27 1.27)) (justify left top))
+    )
+    (instances
+      (project "ETH1CFGEN1A"
+        (path "/44bc1157-6d68-4ab3-afc0-b8d9f089cc50" (page "9"))
+      )
+    )

Commit message: Hardware development
Other:
- removed sheet FPGA
Changed lines of the file:
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@@
-    )
-  )
-  (sheet (at 22.225 43.815) (size 41.91 43.815) (fields_autoplaced)
-    (stroke (width 0.1524) (type solid))
-    (fill (color 0 0 0 0.0000))
-    (property "Sheetname" "FPGA" (at 22.225 43.1034 0)
-      (effects (font (size 1.27 1.27)) (justify left bottom))
-    )
-    (property "Sheetfile" "FPGA.kicad_sch" (at 22.225 88.2146 0)
-      (effects (font (size 1.27 1.27)) (justify left top))
-    )
-    (instances
-      (project "ETH1CFGEN1A"
-        (path "/44bc1157-6d68-4ab3-afc0-b8d9f089cc50" (page "9"))
-      )
     )
   )
