File: hardware/ETH1CFGEN1B/FPGA.kicad_sch (KiCad schematic)
At the start: 46 parts, among them J501 Conn_01x06, J502 Conn_02x07_Odd_Even, U503 XC6SLX9-3TQG144I, U504 W25Q64JV, X501 ASFL1-100.000MHZ-L-T

Commit message: Hardware development
Parts:
- C206: renamed from C506; footprint (none) -> Capacitor_SMD:C_1206_3216Metric_Pad1.33x1.80mm_HandSolder
- C213: renamed from C513; footprint (none) -> Capacitor_SMD:C_1206_3216Metric_Pad1.33x1.80mm_HandSolder
- J201: renamed from J501; footprint (none) -> Connector_PinHeader_2.54mm:PinHeader_1x06_P2.54mm_Vertical
- U201, U202: renamed from U?; footprint (none) -> Package_TO_SOT_SMD:SOT-223-3_TabPin2
- renumbered C501 to C201, C502 to C202, C503 to C203, C504 to C204, C505 to C205, C507 to C207, C508 to C208, C509 to C209, C510 to C210, C511 to C211, C512 to C212, C514 to C214, C515 to C215, C516 to C216, C517 to C217, C518 to C218, C519 to C219, C520 to C220, C521 to C221, C522 to C222, C523 to C223, C524 to C224, C525 to C225, C526 to C226, C527 to C227, C528 to C228, C529 to C229, D501 to D201, J502 to J202, R501 to R201, R502 to R202, R503 to R203, R504 to R204, R505 to R205, R506 to R206, R507 to R207, R508 to R208, R509 to R209, U503 to U203, U504 to U204, X501 to X201
